File: IMU.sch (KiCad schematic (older format))
At the start: 11 parts, among them U3 MPU60X0, U4 HMC5883L, U5 MS5611-01BA03

Commit message: improved version
Parts:
- C16, C17, C18, C20, C21, C22, C23, C24: footprint SM0603_Capa -> ESP32-footprints-Lib:0603_new_new
Changed lines of the file:
@@
 	3900 4900 4100 4900
 Wire Wire Line
-	4100 4900 4100 5100
+	4100 4900 4100 5000
 Connection ~ 4000 5600
 Wire Wire Line
-	4000 5700 4000 5400
+	4000 5700 4000 5600
 Wire Wire Line
 	4000 5400 4200 5400
@@
 	6900 2800 6900 3000
 Wire Wire Line
-	6900 3000 7300 3000
+	6900 3000 7050 3000
 Wire Wire Line
 	5500 2400 7300 2400
@@
 Connection ~ 7050 3000
 Wire Wire Line
-	7050 3100 7050 2700
+	7050 3100 7050 3000
 Wire Wire Line
 	7050 2700 7300 2700
@@
 Connection ~ 2900 2800
 Wire Wire Line
-	4100 2800 2900 2800
+	4100 2800 3900 2800
 Wire Wire Line
 	3850 3850 3850 3950
 Connection ~ 3200 3950
 Wire Wire Line
-	3850 3950 2900 3950
+	3850 3950 3500 3950
 Wire Wire Line
 	2900 3950 2900 3850
@@
 	5500 2200 6050 2200
 Wire Wire Line
-	1750 2500 4100 2500
-Wire Wire Line
-	3850 3150 3850 3450
+	1750 2500 2300 2500
+Wire Wire Line
+	3850 3150 3850 3200
 Wire Wire Line
 	3200 3450 3200 2900
@@
 	3200 2900 4100 2900
 Wire Wire Line
-	1750 2400 4100 2400
-Wire Wire Line
-	3200 4050 3200 3850
-Wire Wire Line
-	2900 3450 2900 2650
+	1750 2400 2400 2400
+Wire Wire Line
+	3200 4050 3200 3950
+Wire Wire Line
+	2900 3450 2900 2800
 Wire Wire Line
 	4100 2200 3500 2200
@@
 	8600 2900 8750 2900
 Wire Wire Line
-	8750 2900 8750 3600
-Wire Wire Line
-	7050 3500 7050 3600
+	8750 2900 8750 3000
+Wire Wire Line
+	7050 3500 7050 3550
 Wire Wire Line
 	8600 2600 8950 2600
@@
 	4200 5000 4100 5000
 Wire Wire Line
-	4200 5600 3800 5600
+	4200 5600 4000 5600
 Wire Wire Line
 	3800 5600 3800 5550
@@
 F 0 "C24" H 4050 6000 50  0000 L CNN
 F 1 "100nF" H 4050 5800 50  0000 L CNN
-F 2 "SM0603_Capa" H 4000 5900 60  0001 C CNN
+F 2 "ESP32-footprints-Lib:0603_new_new" H 4000 5900 60  0001 C CNN
 F 3 "" H 4000 5900 50  0001 C CNN
 	1    4000 5900
@@
 F 0 "C22" H 6700 3400 50  0000 L CNN
 F 1 "4.7uF" H 6700 3200 50  0000 L CNN
-F 2 "SM0603_Capa" H 6650 3300 60  0001 C CNN
+F 2 "ESP32-footprints-Lib:0603_new_new" H 6650 3300 60  0001 C CNN
 F 3 "" H 6650 3300 50  0001 C CNN
 	1    6650 3300
@@
 F 0 "C21" H 9200 2800 50  0000 L CNN
 F 1 "0.22uF" H 9200 2600 50  0000 L CNN
-F 2 "SM0603_Capa" H 9150 2700 60  0001 C CNN
+F 2 "ESP32-footprints-Lib:0603_new_new" H 9150 2700 60  0001 C CNN
 F 3 "" H 9150 2700 50  0001 C CNN
 	1    9150 2700
@@
 F 0 "C23" H 7100 3400 50  0000 L CNN
 F 1 "100nF" H 7100 3200 50  0000 L CNN
-F 2 "SM0603_Capa" H 7050 3300 60  0001 C CNN
+F 2 "ESP32-footprints-Lib:0603_new_new" H 7050 3300 60  0001 C CNN
 F 3 "" H 7050 3300 50  0001 C CNN
 	1    7050 3300
@@
 F 0 "C18" H 3550 3750 50  0000 L CNN
 F 1 "100nF" H 3550 3550 50  0000 L CNN
-F 2 "SM0603_Capa" H 3500 3650 60  0001 C CNN
+F 2 "ESP32-footprints-Lib:0603_new_new" H 3500 3650 60  0001 C CNN
 F 3 "" H 3500 3650 50  0001 C CNN
 	1    3500 3650
@@
 F 0 "C16" H 2950 3750 50  0000 L CNN
 F 1 "10nF" H 2950 3550 50  0000 L CNN
-F 2 "SM0603_Capa" H 2900 3650 60  0001 C CNN
+F 2 "ESP32-footprints-Lib:0603_new_new" H 2900 3650 60  0001 C CNN
 F 3 "" H 2900 3650 50  0001 C CNN
 	1    2900 3650
@@
 F 0 "C17" H 3250 3750 50  0000 L CNN
 F 1 "2.2nF" H 3250 3550 50  0000 L CNN
-F 2 "SM0603_Capa" H 3200 3650 60  0001 C CNN
+F 2 "ESP32-footprints-Lib:0603_new_new" H 3200 3650 60  0001 C CNN
 F 3 "" H 3200 3650 50  0001 C CNN
 	1    3200 3650
@@
 F 0 "C20" H 3900 3750 50  0000 L CNN
 F 1 "100nF" H 3900 3550 50  0000 L CNN
-F 2 "SM0603_Capa" H 3850 3650 60  0001 C CNN
+F 2 "ESP32-footprints-Lib:0603_new_new" H 3850 3650 60  0001 C CNN
 F 3 "" H 3850 3650 50  0001 C CNN
 	1    3850 3650
@@
 	1    0    0    -1
 $EndComp
+Wire Wire Line
+	4100 5000 4100 5100
+Wire Wire Line
+	4000 5600 4000 5400
+Wire Wire Line
+	4000 5600 3800 5600
+Wire Wire Line
+	2400 2400 4100 2400
+Wire Wire Line
+	7050 3000 7300 3000
+Wire Wire Line
+	7050 3000 7050 2900
+Wire Wire Line
+	8750 3000 8750 3600
+Wire Wire Line
+	3500 3950 3200 3950
+Wire Wire Line
+	2900 2800 2900 2650
+Wire Wire Line
+	3200 3950 3200 3850
+Wire Wire Line
+	3200 3950 2900 3950
+Wire Wire Line
+	3850 3200 3850 3450
+Wire Wire Line
+	3900 2800 2900 2800
+Wire Wire Line
+	7050 2900 7050 2700
+Wire Wire Line
+	7050 3550 7050 3600
+Wire Wire Line
+	2300 2500 4100 2500
 $EndSCHEMATC

Commit message: version 2.0
Parts:
- removed C16: 10nF, ESP32-footprints-Lib:0603_new_new, symbol Crazyflie-contol-board-rescue:C
- removed C17: 2.2nF, ESP32-footprints-Lib:0603_new_new, symbol Crazyflie-contol-board-rescue:C
- removed C21: 0.22uF, ESP32-footprints-Lib:0603_new_new, symbol Crazyflie-contol-board-rescue:C
- removed C22: 4.7uF, ESP32-footprints-Lib:0603_new_new, symbol Crazyflie-contol-board-rescue:C
- removed C23: 100nF, ESP32-footprints-Lib:0603_new_new, symbol Crazyflie-contol-board-rescue:C
- removed U3: MPU60X0, MPU60X0, symbol Crazyflie-contol-board-rescue:MPU60X0
- removed U4: HMC5883L, QFN16_HMC5883L, symbol Crazyflie-contol-board-rescue:HMC5883L
- added U1: BMX160, digikey-footprints:LGA-14L_2.5x3mm__LSM6DS3, symbol Crazyflie-contol-board-rescue:BMX160-SensorMotion
- C18: renamed from C20; symbol Crazyflie-contol-board-rescue:C -> Crazyflie-contol-board-rescue:C-Crazyflie-contol-board-rescue
- C20: renamed from C18; symbol Crazyflie-contol-board-rescue:C -> Crazyflie-contol-board-rescue:C-Crazyflie-contol-board-rescue
- C24: symbol Crazyflie-contol-board-rescue:C -> Crazyflie-contol-board-rescue:C-Crazyflie-contol-board-rescue
- U5: symbol Crazyflie-contol-board-rescue:MS5611-01BA01 -> Crazyflie-contol-board-rescue:MS5611-01BA01-Crazyflie-contol-board-rescue
Connections:
- net AGND: now also U1.1 (AD0/SDO), U1.2 (GND), U1.3 (GND), U1.6 (GNDIO), U1.7 (GND)
- net I2C_SCL_VCCA: now also U1.13 (SCL/SCLK)
- net I2C_SDA_VCCA: now also U1.14 (SDA/SDI)
- net INT_GA: now also U1.4 (INT1)
- net VCCA: now also C20.1, U1.12 (CSB), U1.5 (VDDIO), U1.8 (VDD)
- no-connect marks 8 -> 1
Other:
- note added: "U5 not mounted on 9-DOF version"
- note removed: "U4 not mounted on 6-DOF version"
- note removed: "U5 not mounted on 6-DOF version"
- moved on the sheet: C18, C20, C24, U5
