File: Power.sch (KiCad schematic (older format))
At the start: 47 parts, among them P7 MICRO-B-USB, P9 CONN_1, Q5 2N7002, Q6 2N7002, SW1 PUSH ON/OFF, U10 MAX16054, U6 NUF2221, U7 TPS79301, U8 BQ24075, U9 TPS79301

Commit message: improved version
Parts:
- C29, C30, C31, C32, C33, C34, C35, C36, C37, C38, C39, C40, C41: footprint SM0603_Capa -> ESP32-footprints-Lib:0603_new_new
- R16, R17, R18, R19, R20, R21, R22, R23, R24, R25, R26, R27, R28, R29, R30, R31, R32, R33, R36, R37, R38: footprint SM0603 -> ESP32-footprints-Lib:0603_new_new
Changed lines of the file:
@@
 	5350 3500 5050 3500
 Connection ~ 3250 4000
-Wire Wire Line
-	3450 3200 1850 3200
 Connection ~ 1850 3200
 Connection ~ 2550 4600
@@
 F 0 "R38" V 10730 3650 50  0000 C CNN
 F 1 "1k" V 10650 3650 50  0000 C CNN
-F 2 "SM0603" H 10650 3650 60  0001 C CNN
+F 2 "ESP32-footprints-Lib:0603_new_new" H 10650 3650 60  0001 C CNN
 F 3 "" H 10650 3650 50  0001 C CNN
 F 4 "General" V 10650 3650 60  0001 C CNN "Field4"
@@
 F 0 "R37" V 4480 5750 50  0000 C CNN
 F 1 "10k" V 4400 5750 50  0000 C CNN
-F 2 "SM0603" H 4400 5750 60  0001 C CNN
+F 2 "ESP32-footprints-Lib:0603_new_new" H 4400 5750 60  0001 C CNN
 F 3 "" H 4400 5750 50  0001 C CNN
 F 4 "Genaral" V 4400 5750 60  0001 C CNN "Field4"
@@
 F 0 "R36" V 5730 6800 50  0000 C CNN
 F 1 "10k" V 5650 6800 50  0000 C CNN
-F 2 "SM0603" H 5650 6800 60  0001 C CNN
+F 2 "ESP32-footprints-Lib:0603_new_new" H 5650 6800 60  0001 C CNN
 F 3 "" H 5650 6800 50  0001 C CNN
 F 4 "Genaral" V 5650 6800 60  0001 C CNN "Field4"
@@
 F 0 "R33" V 5430 5450 50  0000 C CNN
 F 1 "10k" V 5350 5450 50  0000 C CNN
-F 2 "SM0603" H 5350 5450 60  0001 C CNN
+F 2 "ESP32-footprints-Lib:0603_new_new" H 5350 5450 60  0001 C CNN
 F 3 "" H 5350 5450 50  0001 C CNN
 F 4 "Genaral" V 5350 5450 60  0001 C CNN "Field4"
@@
 F 0 "R25" V 2430 4050 50  0000 C CNN
 F 1 "10k" V 2350 4050 50  0000 C CNN
-F 2 "SM0603" H 2350 4050 60  0001 C CNN
+F 2 "ESP32-footprints-Lib:0603_new_new" H 2350 4050 60  0001 C CNN
 F 3 "" H 2350 4050 50  0001 C CNN
 	1    2350 4050
@@
 F 0 "C33" H 4500 2600 50  0000 L CNN
 F 1 "100nF" H 4500 2400 50  0000 L CNN
-F 2 "SM0603_Capa" H 4450 2500 60  0001 C CNN
+F 2 "ESP32-footprints-Lib:0603_new_new" H 4450 2500 60  0001 C CNN
 F 3 "" H 4450 2500 50  0001 C CNN
 F 4 "General" H 4450 2500 60  0001 C CNN "Field4"
@@
 F 0 "R29" V 7680 4400 50  0000 C CNN
 F 1 "0R" V 7600 4400 50  0000 C CNN
-F 2 "SM0603" H 7600 4400 60  0001 C CNN
+F 2 "ESP32-footprints-Lib:0603_new_new" H 7600 4400 60  0001 C CNN
 F 3 "" H 7600 4400 50  0001 C CNN
 F 4 "General" V 7600 4400 60  0001 C CNN "Field4"
@@
 F 0 "R19" V 7630 2450 50  0000 C CNN
 F 1 "0R" V 7550 2450 50  0000 C CNN
-F 2 "SM0603" H 7550 2450 60  0001 C CNN
+F 2 "ESP32-footprints-Lib:0603_new_new" H 7550 2450 60  0001 C CNN
 F 3 "" H 7550 2450 50  0001 C CNN
 	1    7550 2450
@@
 F 0 "R21" V 9680 3600 50  0000 C CNN
 F 1 "300k" V 9600 3600 50  0000 C CNN
-F 2 "SM0603" H 9600 3600 60  0001 C CNN
+F 2 "ESP32-footprints-Lib:0603_new_new" H 9600 3600 60  0001 C CNN
 F 3 "" H 9600 3600 50  0001 C CNN
 F 4 "General" V 9600 3600 60  0001 C CNN "Field4"
@@
 F 0 "C29" H 8950 1800 50  0000 L CNN
 F 1 "15pF" H 8950 1600 50  0000 L CNN
-F 2 "SM0603_Capa" H 8900 1700 60  0001 C CNN
+F 2 "ESP32-footprints-Lib:0603_new_new" H 8900 1700 60  0001 C CNN
 F 3 "" H 8900 1700 50  0001 C CNN
 	1    8900 1700
@@
 F 0 "R16" V 8730 1650 50  0000 C CNN
 F 1 "39k" V 8650 1650 50  0000 C CNN
-F 2 "SM0603" H 8650 1650 60  0001 C CNN
+F 2 "ESP32-footprints-Lib:0603_new_new" H 8650 1650 60  0001 C CNN
 F 3 "" H 8650 1650 50  0001 C CNN
 F 4 "General" V 8650 1650 60  0001 C CNN "Field4"
@@
 F 0 "R18" V 8730 2350 50  0000 C CNN
 F 1 "30k" V 8650 2350 50  0000 C CNN
-F 2 "SM0603" H 8650 2350 60  0001 C CNN
+F 2 "ESP32-footprints-Lib:0603_new_new" H 8650 2350 60  0001 C CNN
 F 3 "" H 8650 2350 50  0001 C CNN
 F 4 "General" V 8650 2350 60  0001 C CNN "Field4"
@@
 F 0 "C35" H 8950 3700 50  0000 L CNN
 F 1 "15pF" H 8950 3500 50  0000 L CNN
-F 2 "SM0603_Capa" H 8900 3600 60  0001 C CNN
+F 2 "ESP32-footprints-Lib:0603_new_new" H 8900 3600 60  0001 C CNN
 F 3 "" H 8900 3600 50  0001 C CNN
 	1    8900 3600
@@
 F 0 "R23" V 9330 3900 50  0000 C CNN
 F 1 "150k" V 9250 3900 50  0000 C CNN
-F 2 "SM0603" H 9250 3900 60  0001 C CNN
+F 2 "ESP32-footprints-Lib:0603_new_new" H 9250 3900 60  0001 C CNN
 F 3 "" H 9250 3900 50  0001 C CNN
 F 4 "General" V 9250 3900 60  0001 C CNN "Field4"
@@
 F 0 "R28" V 8730 4250 50  0000 C CNN
 F 1 "30k" V 8650 4250 50  0000 C CNN
-F 2 "SM0603" H 8650 4250 60  0001 C CNN
+F 2 "ESP32-footprints-Lib:0603_new_new" H 8650 4250 60  0001 C CNN
 F 3 "" H 8650 4250 50  0001 C CNN
 	1    8650 4250
@@
 F 0 "R20" V 8730 3600 50  0000 C CNN
 F 1 "42.2k" V 8650 3600 50  0000 C CNN
-F 2 "SM0603" H 8650 3600 60  0001 C CNN
+F 2 "ESP32-footprints-Lib:0603_new_new" H 8650 3600 60  0001 C CNN
 F 3 "" H 8650 3600 50  0001 C CNN
 F 4 "General" V 8650 3600 60  0001 C CNN "Field4"
@@
 F 0 "R31" V 2380 6950 50  0000 C CNN
 F 1 "100k" V 2300 6950 50  0000 C CNN
-F 2 "SM0603" H 2300 6950 60  0001 C CNN
+F 2 "ESP32-footprints-Lib:0603_new_new" H 2300 6950 60  0001 C CNN
 F 3 "" H 2300 6950 50  0001 C CNN
 F 4 "General" V 2300 6950 60  0001 C CNN "Field4"
@@
 F 0 "R22" V 10480 3650 50  0000 C CNN
 F 1 "1k" V 10400 3650 50  0000 C CNN
-F 2 "SM0603" H 10400 3650 60  0001 C CNN
+F 2 "ESP32-footprints-Lib:0603_new_new" H 10400 3650 60  0001 C CNN
 F 3 "" H 10400 3650 50  0001 C CNN
 F 4 "General" V 10400 3650 60  0001 C CNN "Field4"
@@
 F 0 "C34" H 4850 2600 50  0000 L CNN
 F 1 "4.7uF" H 4850 2400 50  0000 L CNN
-F 2 "SM0603_Capa" H 4800 2500 60  0001 C CNN
+F 2 "ESP32-footprints-Lib:0603_new_new" H 4800 2500 60  0001 C CNN
 F 3 "" H 4800 2500 50  0001 C CNN
 F 4 "General" H 4800 2500 60  0001 C CNN "Field4"
@@
 F 0 "C41" H 6700 6850 50  0000 L CNN
 F 1 "100nF" H 6700 6650 50  0000 L CNN
-F 2 "SM0603_Capa" H 6650 6750 60  0001 C CNN
+F 2 "ESP32-footprints-Lib:0603_new_new" H 6650 6750 60  0001 C CNN
 F 3 "" H 6650 6750 50  0001 C CNN
 	1    6650 6750
@@
 F 0 "R32" V 6430 6800 50  0000 C CNN
 F 1 "10k" V 6350 6800 50  0000 C CNN
-F 2 "SM0603" H 6350 6800 60  0001 C CNN
+F 2 "ESP32-footprints-Lib:0603_new_new" H 6350 6800 60  0001 C CNN
 F 3 "" H 6350 6800 50  0001 C CNN
 	1    6350 6800
@@
 F 0 "R30" V 6430 5550 50  0000 C CNN
 F 1 "20k" V 6350 5550 50  0000 C CNN
-F 2 "SM0603" H 6350 5550 60  0001 C CNN
+F 2 "ESP32-footprints-Lib:0603_new_new" H 6350 5550 60  0001 C CNN
 F 3 "" H 6350 5550 50  0001 C CNN
 	1    6350 5550
@@
 F 0 "R27" V 2830 4050 50  0000 C CNN
 F 1 "10k" V 2750 4050 50  0000 C CNN
-F 2 "SM0603" H 2750 4050 60  0001 C CNN
+F 2 "ESP32-footprints-Lib:0603_new_new" H 2750 4050 60  0001 C CNN
 F 3 "" H 2750 4050 50  0001 C CNN
 F 4 "Genaral" V 2750 4050 60  0001 C CNN "Field4"
@@
 F 0 "R26" V 2630 4050 50  0000 C CNN
 F 1 "1.2K" V 2550 4050 50  0000 C CNN
-F 2 "SM0603" H 2550 4050 60  0001 C CNN
+F 2 "ESP32-footprints-Lib:0603_new_new" H 2550 4050 60  0001 C CNN
 F 3 "" H 2550 4050 50  0001 C CNN
 	1    2550 4050
@@
 F 0 "R24" V 2230 4050 50  0000 C CNN
 F 1 "1.2k" V 2150 4050 50  0000 C CNN
-F 2 "SM0603" H 2150 4050 60  0001 C CNN
+F 2 "ESP32-footprints-Lib:0603_new_new" H 2150 4050 60  0001 C CNN
 F 3 "" H 2150 4050 50  0001 C CNN
 F 4 "General" V 2150 4050 60  0001 C CNN "Field4"
@@
 F 0 "C36" H 1900 4400 50  0000 L CNN
 F 1 "100nF" H 1900 4200 50  0000 L CNN
-F 2 "SM0603_Capa" H 1850 4300 60  0001 C CNN
+F 2 "ESP32-footprints-Lib:0603_new_new" H 1850 4300 60  0001 C CNN
 F 3 "" H 1850 4300 50  0001 C CNN
 	1    1850 4300
@@
 F 0 "C39" H 3050 4400 50  0000 L CNN
 F 1 "10uF" H 3050 4200 50  0000 L CNN
-F 2 "SM0603_Capa" H 3000 4300 60  0001 C CNN
+F 2 "ESP32-footprints-Lib:0603_new_new" H 3000 4300 60  0001 C CNN
 F 3 "" H 3000 4300 50  0001 C CNN
 F 4 "General" H 3000 4300 60  0001 C CNN "Field4"
@@
 F 0 "R17" V 6280 1900 50  0000 C CNN
 F 1 "10R" V 6200 1900 50  0000 C CNN
-F 2 "SM0603" H 6200 1900 60  0001 C CNN
+F 2 "ESP32-footprints-Lib:0603_new_new" H 6200 1900 60  0001 C CNN
 F 3 "" H 6200 1900 50  0001 C CNN
 F 4 "General" V 6200 1900 60  0001 C CNN "Field4"
@@
 F 0 "C30" H 9250 2100 50  0000 L CNN
 F 1 "4.7uF" H 9250 1900 50  0000 L CNN
-F 2 "SM0603_Capa" H 9200 2000 60  0001 C CNN
+F 2 "ESP32-footprints-Lib:0603_new_new" H 9200 2000 60  0001 C CNN
 F 3 "" H 9200 2000 50  0001 C CNN
 	1    9200 2000
@@
 F 0 "C32" H 8350 2500 50  0000 L CNN
 F 1 "10nF" H 8350 2300 50  0000 L CNN
-F 2 "SM0603_Capa" H 8300 2400 60  0001 C CNN
+F 2 "ESP32-footprints-Lib:0603_new_new" H 8300 2400 60  0001 C CNN
 F 3 "" H 8300 2400 50  0001 C CNN
 F 4 "General" H 8300 2400 60  0001 C CNN "Field4"
@@
 F 0 "C40" H 8350 4400 50  0000 L CNN
 F 1 "10nF" H 8350 4200 50  0000 L CNN
-F 2 "SM0603_Capa" H 8300 4300 60  0001 C CNN
+F 2 "ESP32-footprints-Lib:0603_new_new" H 8300 4300 60  0001 C CNN
 F 3 "" H 8300 4300 50  0001 C CNN
 F 4 "General" H 8300 4300 60  0001 C CNN "Field4"
@@
 F 0 "C37" H 10000 4050 50  0000 L CNN
 F 1 "4.7uF" H 10000 3850 50  0000 L CNN
-F 2 "SM0603_Capa" H 9950 3950 60  0001 C CNN
+F 2 "ESP32-footprints-Lib:0603_new_new" H 9950 3950 60  0001 C CNN
 F 3 "" H 9950 3950 50  0001 C CNN
 	1    9950 3950
@@
 F 0 "C38" H 6550 4200 50  0000 L CNN
 F 1 "100nF" H 6550 4000 50  0000 L CNN
-F 2 "SM0603_Capa" H 6500 4100 60  0001 C CNN
+F 2 "ESP32-footprints-Lib:0603_new_new" H 6500 4100 60  0001 C CNN
 F 3 "" H 6500 4100 50  0001 C CNN
 	1    6500 4100
@@
 F 0 "C31" H 6600 2300 50  0000 L CNN
 F 1 "4.7uF" H 6600 2100 50  0000 L CNN
-F 2 "SM0603_Capa" H 6550 2200 60  0001 C CNN
+F 2 "ESP32-footprints-Lib:0603_new_new" H 6550 2200 60  0001 C CNN
 F 3 "" H 6550 2200 50  0001 C CNN
 	1    6550 2200
@@
 Wire Wire Line
 	1850 3200 1850 4100
+Wire Wire Line
+	1850 3200 2700 3200
+Wire Wire Line
+	2700 3200 2700 2900
+Text HLabel 2700 2900 1    60   Output ~ 0
+VUSB
+Connection ~ 2700 3200
+Wire Wire Line
+	2700 3200 3450 3200
 $EndSCHEMATC

Commit message: version 2.0
Parts:
- BT1: symbol Crazyflie-contol-board-rescue:BATTERY -> Crazyflie-contol-board-rescue:BATTERY-Crazyflie-contol-board-rescue
- C29, C30, C31, C32, C33, C34, C35, C36, C37, C38, C39, C40, C41: symbol Crazyflie-contol-board-rescue:C -> Crazyflie-contol-board-rescue:C-Crazyflie-contol-board-rescue
- D7, D8: symbol Crazyflie-contol-board-rescue:LED -> Crazyflie-contol-board-rescue:LED-Crazyflie-contol-board-rescue
- P7: symbol Crazyflie-contol-board-rescue:MICRO-B-USB -> Crazyflie-contol-board-rescue:MICRO-B-USB-Crazyflie-contol-board-rescue
- P9: symbol Crazyflie-contol-board-rescue:CONN_1 -> Crazyflie-contol-board-rescue:CONN_1-Crazyflie-contol-board-rescue
- Q5, Q6: symbol Crazyflie-contol-board-rescue:MOSFET_N -> Crazyflie-contol-board-rescue:MOSFET_N-Crazyflie-contol-board-rescue
- R16, R17, R18, R19, R20, R21, R22, R23, R24, R25, R26, R27, R28, R29, R30, R31, R32, R33, R36, R37, R38: symbol Crazyflie-contol-board-rescue:R -> Crazyflie-contol-board-rescue:R-Crazyflie-contol-board-rescue
- SW1: symbol Crazyflie-contol-board-rescue:SW_PUSH -> Crazyflie-contol-board-rescue:SW_PUSH-Crazyflie-contol-board-rescue
- U10: symbol Crazyflie-contol-board-rescue:MAX16054 -> Crazyflie-contol-board-rescue:MAX16054-Crazyflie-contol-board-rescue
- U6: symbol Crazyflie-contol-board-rescue:NUF2221 -> Crazyflie-contol-board-rescue:NUF2221-Crazyflie-contol-board-rescue
- U7, U9: symbol Crazyflie-contol-board-rescue:TPS79301 -> Crazyflie-contol-board-rescue:TPS79301-Crazyflie-contol-board-rescue
- U8: symbol Crazyflie-contol-board-rescue:BQ24075 -> Crazyflie-contol-board-rescue:BQ24075-Crazyflie-contol-board-rescue
Connections:
- net USB_CON is gone; now on net VCC: U6.5 (VBUS)
