File: Crazyflie contol board.kicad_pcb (KiCad board)
At the start: 4 copper layers, 40.1 x 38.1 mm, 98 parts, among them P1 CONN_2, P2 CONN_2, P3 CONN_2, P4 CONN_2, P7 MICRO-B-USB, P9 CONN_1, Q1 PMV31XN, Q2 PMV31XN, Q3 PMV31XN, Q4 PMV31XN, Q5 2N7002, Q6 2N7002, Q7 SS8050-G, Q8 SS8050-G, SW1 PUSH ON/OFF, SW2 BOOT, U1 BMX160, U10 MAX16054, U11 ESP32-WROOM, U12 CP2102N-A01-GQFN24, U5 MS5611-01BA03, U6 NUF2221, U7 TPS79301, U8 BQ24075, U9 TPS79301

Commit message: jlpcb fix
Connections:
- net /Red renamed /RED
Changed lines of the file:
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@@
     (visible_elements 7FFFFFFF)
     (pcbplotparams
-      (layerselection 0x00030_ffffffff)
+      (layerselection 0x010f0_ffffffff)
       (usegerberextensions true)
       (usegerberattributes false)
@@
   (net 60 /USBD+)
   (net 61 /USBD-)
-  (net 62 /Red)
+  (net 62 /RED)
   (net_class Default "This is the default net class."
     (clearance 0.1524)
@@
     (add_net /PGOOD)
     (add_net /POWER/VUSB)
-    (add_net /Red)
+    (add_net /RED)
     (add_net /SYSOFF)
     (add_net /USBD+)
@@
     (fp_line (start -1.143 0.635) (end -1.143 -0.635) (layer F.SilkS) (width 0.127))
     (pad 1 smd rect (at -0.762 0) (size 0.635 1.143) (layers Front_L1 F.Paste F.Mask)
-      (net 62 /Red))
+      (net 62 /RED))
     (pad 2 smd rect (at 0.762 0) (size 0.635 1.143) (layers Front_L1 F.Paste F.Mask)
       (net 24 "Net-(D5-Pad2)"))
@@
       (effects (font (size 0.8001 0.8001) (thickness 0.20066)))
     )
-    (fp_text value "BLUE LED" (at 0.249651 -1.298545 225) (layer F.SilkS) hide
+    (fp_text value "BLUE LED" (at -0.084414 -2.717426 225) (layer F.SilkS) hide
       (effects (font (size 0.8001 0.8001) (thickness 0.20066)))
     )
@@
     (pad 32 smd oval (at -9 2.37 180) (size 2.5 0.9) (layers Back_L4 B.Paste B.Mask))
     (pad 31 smd oval (at -9 3.64 180) (size 2.5 0.9) (layers Back_L4 B.Paste B.Mask)
-      (net 62 /Red))
+      (net 62 /RED))
     (pad 30 smd oval (at -9 4.91 180) (size 2.5 0.9) (layers Back_L4 B.Paste B.Mask)
       (net 36 /PGOOD))
