File: Crazyflie contol board.sch (KiCad schematic (older format))
At the start: 40 parts, among them P1 CONN_2, P2 CONN_2, P3 CONN_2, P4 CONN_2, Q1 PMV31XN, Q2 PMV31XN, Q3 PMV31XN, Q4 PMV31XN, Q7 SS8050-G, Q8 SS8050-G, SW2 BOOT, U11 ESP32-WROOM, U12 CP2102N-A01-GQFN24

Commit message: jlpcb fix
Connections:
- net Red renamed RED
Changed lines of the file:
@@
 	1050 1800 650  1800
-Wire Wire Line
-	9050 5200 9500 5200
 Wire Wire Line
 	1250 3550 1250 3850
@@
 	1950 2000 1950 2400
 Wire Wire Line
-	9050 4300 9700 4300
-Wire Wire Line
 	7800 6000 7800 6450
 Wire Wire Line
 	2200 5400 1700 5400
-Wire Wire Line
-	3500 5650 3900 5650
 Connection ~ 10950 6150
 Wire Wire Line
@@
 	10600 6150 10950 6150
 Wire Wire Line
-	3500 5550 3900 5550
-Wire Wire Line
 	2200 5300 1700 5300
 Wire Wire Line
@@
 Wire Wire Line
 	10950 6350 10950 6150
-Wire Wire Line
-	9050 4600 9700 4600
 Wire Wire Line
 	1650 1000 1650 900
@@
 Wire Wire Line
 	1450 3750 2200 3750
-Wire Wire Line
-	9050 5300 9500 5300
 Wire Wire Line
 	2450 1800 2850 1800
@@
 F4 "I2C_SCL_VCCA" I L 2200 3750 60
 $EndSheet
-Text Label 5300 4850 0    60   ~ 0
+Text Label 5350 5050 0    60   ~ 0
 INT_GA
-Text Label 9700 4600 2    60   ~ 0
+Text Label 10600 4600 2    60   ~ 0
 I2C_SCK_VCCA
-Text Label 9700 4300 2    60   ~ 0
+Text Label 10600 4300 2    60   ~ 0
 I2C_SCL_VCCA
 Text Notes 650  7600 1    60   ~ 0
@@
 	1    0    0    -1
 $EndComp
-Text Label 9500 5300 2    60   ~ 0
+Text Label 10600 5300 2    60   ~ 0
 MOTOR3
-Text Label 9500 5200 2    60   ~ 0
+Text Label 10600 5200 2    60   ~ 0
 MOTOR4
 Text Label 10600 4200 2    60   ~ 0
@@
 Text Label 7800 6450 1    60   ~ 0
 MOTOR1
-Text Label 5300 5150 0    60   ~ 0
+Text Label 5350 5350 0    60   ~ 0
 EN2
-Text Label 5300 4950 0    60   ~ 0
+Text Label 5350 5150 0    60   ~ 0
 EN1
-Text Label 5300 5050 0    60   ~ 0
+Text Label 5350 5250 0    60   ~ 0
 TDO
-Text Label 5300 4700 0    60   ~ 0
+Text Label 5350 4950 0    60   ~ 0
 SYSOFF
-Text Label 10050 4900 2    60   ~ 0
+Text Label 10600 4900 2    60   ~ 0
 PGOOD
-Text Label 10050 5100 2    60   ~ 0
+Text Label 10600 5100 2    60   ~ 0
 CHG
-Text Label 3900 5650 2    60   ~ 0
+Text Label 4200 5650 2    60   ~ 0
 PGOOD
-Text Label 3900 5550 2    60   ~ 0
+Text Label 4200 5550 2    60   ~ 0
 CHG
 Text Label 1700 5500 0    60   ~ 0
@@
 	0    -1   -1   0
 $EndComp
-Wire Wire Line
-	6750 5250 7200 5250
-Wire Wire Line
-	6850 5150 7200 5150
-Wire Wire Line
-	7000 5050 7200 5050
-Wire Wire Line
-	10050 4900 9050 4900
 $Comp
 L Crazyflie-contol-board-rescue:VCC-power #PWR0113
@@
 Wire Wire Line
 	4550 6950 4650 6950
-Wire Wire Line
-	5300 4700 7100 4700
 Text Label 7900 2200 0    50   ~ 0
 USBD-
 Wire Wire Line
 	3500 5300 4200 5300
-Text Label 4200 5300 0    50   ~ 0
+Text Label 4200 5300 2    50   ~ 0
 USBD-
-Text Label 4200 5400 0    50   ~ 0
+Text Label 4200 5400 2    50   ~ 0
 USBD+
 Text Label 7900 2100 0    50   ~ 0
@@
 Wire Wire Line
 	9650 1700 9550 1700
-Wire Wire Line
-	9050 5100 10050 5100
-Wire Wire Line
-	7000 4850 7000 5050
-Wire Wire Line
-	5300 4850 7000 4850
-Wire Wire Line
-	6850 4950 6850 5150
-Wire Wire Line
-	5300 4950 6850 4950
-Wire Wire Line
-	6750 5050 6750 5250
-Wire Wire Line
-	5300 5050 6750 5050
 Connection ~ 7100 4350
 Wire Wire Line
@@
 Connection ~ 7200 6000
 Wire Wire Line
-	7100 4950 7200 4950
-Wire Wire Line
-	7100 4700 7100 4950
-Wire Wire Line
-	5300 5150 6650 5150
-Wire Wire Line
-	6650 5150 6650 5350
-Wire Wire Line
-	6650 5350 7200 5350
-Wire Wire Line
 	9450 6350 8600 6350
 Wire Wire Line
 	9050 4200 10600 4200
-Wire Wire Line
-	9050 4800 9150 4800
 Wire Wire Line
 	9150 6150 9450 6150
@@
 	6900 3500 9650 3500
 Text Label 9150 6150 0    50   ~ 0
-Red
-Text Label 9150 4800 0    50   ~ 0
-Red
+RED
+Text Label 10600 4800 2    50   ~ 0
+RED
 Wire Wire Line
 	10000 3200 5950 3200
@@
 Wire Wire Line
 	8600 6350 8600 6000
+Wire Wire Line
+	9050 4600 10600 4600
+Wire Wire Line
+	9050 4800 10600 4800
+Wire Wire Line
+	9050 4900 10600 4900
+Wire Wire Line
+	9050 5100 10600 5100
+Wire Wire Line
+	9050 5200 10600 5200
+Wire Wire Line
+	9050 5300 10600 5300
+Wire Wire Line
+	3500 5550 4200 5550
+Wire Wire Line
+	3500 5650 4200 5650
+Wire Wire Line
+	9050 4300 10600 4300
+Wire Wire Line
+	5350 4950 7200 4950
+Wire Wire Line
+	5350 5050 7200 5050
+Wire Wire Line
+	5350 5250 7200 5250
+Wire Wire Line
+	5350 5150 7200 5150
+Wire Wire Line
+	5350 5350 7200 5350
 $EndSCHEMATC
