File: esp32_mine.kicad_sch (KiCad schematic)
At the start: 75 parts, among them J1 USB_C_Receptacle_USB2.0_14P, J2 Conn_01x02_Pin, J3 Conn_01x18_Pin, J5 Conn_01x18_Pin, Q1 AO3401A, U1 ESP32-S3, U2 W25Q128JVS, U3 MCP73831-2-OT, U4 AMS1117-3.3, Y1 32.768 kHz, Y2 40MHz(10ppm)

Commit message: save
Parts:
- removed BTN1: BTN, Button_Switch_SMD:SW_Push_1P1T_XKB_TS-1187A, symbol Switch:SW_Push
- removed Flash1: Flash, Button_Switch_SMD:SW_Push_1P1T_XKB_TS-1187A, symbol Switch:SW_Push
- removed J2: Conn_01x02_Pin, Connector_PinSocket_2.54mm:PinSocket_1x02_P2.54mm_Vertical, symbol Connector:Conn_01x02_Pin
- removed J3, J5: Conn_01x18_Pin, Connector_PinHeader_2.54mm:PinHeader_1x18_P2.54mm_Vertical, symbol Connector:Conn_01x18_Pin
- removed R21: 10K, Resistor_SMD:R_0402_1005Metric, symbol Device:R
- removed Reset1: Reset, Button_Switch_SMD:SW_Push_1P1T_XKB_TS-1187A, symbol Switch:SW_Push
- removed U4: AMS1117-3.3, Package_TO_SOT_SMD:SOT-223-3_TabPin2, symbol Regulator_Linear:AMS1117-3.3
- added C1, C5: 12pF, Capacitor_SMD:C_0402_1005Metric, symbol Device:C
- added C9: C, Capacitor_SMD:C_0603_1608Metric, symbol Device:C
- added J3: GPIO, Connector_PinHeader_2.54mm:PinHeader_2x05_P2.54mm_Vertical, symbol Connector_Generic:Conn_02x05_Odd_Even
- added R3, R6, R7, R8, R9: 10k, Resistor_SMD:R_0402_1005Metric, symbol Device:R
- added R5: R, Resistor_SMD:R_0402_1005Metric, symbol Device:R
- added U4: BNO055, Package_LGA:LGA-28_5.2x3.8mm_P0.5mm, symbol Sensor_Motion:BNO055
- added U5: BMP280, Package_LGA:Bosch_LGA-8_2x2.5mm_P0.65mm_ClockwisePinNumbering, symbol Sensor_Pressure:BMP280
- added Y3: 32.768 kHz, Crystal:Crystal_SMD_3215-2Pin_3.2x1.5mm, symbol Device:Crystal
- R4: value 10K -> R; LCSC C25744 -> (none); MNF PART NUMBER C25744 -> (none)
Connections:
- net +3V3: now also R3.1, R5.1, R7.1, U4.28 (VDDIO), U4.3 (VDD), U4.4 (~{BOOT_LOAD_PIN}), U5.2 (CSB), U5.6 (VDDIO), U5.8 (VDD)
- net GND: now also C1.2, C5.2, C9.2, J3.1 (Pin_1), J3.4 (Pin_4), R6.2, R8.2, R9.2, U4.18 (COM2), U4.2 (GND), U4.25 (GNDIO), U5.1 (GND), U5.7 (GND)
- net IO0: now also J3.6 (Pin_6)
- net IO12: now also R12.2, R19.1
- net IO14: no longer R4.2
- net IO5: now also R4.2, U4.20 (COM0), U5.3 (SDI)
- net IO6: now also R5.2, U4.19 (COM1), U5.4 (SCK)
- net RX: now also J3.3 (Pin_3)
- net TX: now also J3.5 (Pin_5)
- net VBAT: now also J3.2 (Pin_2)
- removed net IO4/BAT: R12.2, R19.1, U1.9 (GPIO4)
- new net: C1.1, U4.27 (XIN32), Y3.1
- new net: C5.1, U4.26 (XOUT32), Y3.2
- new net: R8.1, U4.6 (PS0)
- new net: R3.2, U5.5 (SDO)
- new net: R7.2, U4.11 (~{RESET})
- new net: R6.1, U4.17 (COM3)
- new net: R9.1, U4.5 (PS1)
- new net: C9.1, U4.9 (CAP)
- new net IO4: U1.9 (GPIO4)

Commit message: save
Parts:
- added C12, C21, C23, C24: C, Capacitor_SMD:C_0603_1608Metric, symbol Device:C
- added C27: 0.1uF, Capacitor_SMD:C_0603_1608Metric, symbol Device:C
- added C28: 10uF, Capacitor_SMD:C_0603_1608Metric, symbol Device:C
- added D5, D6, D7, D8: D, symbol Device:D
- added Q2, Q3, Q4, Q5: Q_NMOS_GSD, symbol Transistor_FET:Q_NMOS_GSD
- added R10, R11, R13, R21: R, Resistor_SMD:R_0402_1005Metric, symbol Device:R
- added R32, R33, R34, R35: 10k, Resistor_SMD:R_0402_1005Metric, symbol Device:R
- added U7: RT9701, symbol Power_Management:RT9701
- C9: value C -> 0.1uF
Connections:
- net +3V3: now also C27.1, C28.1, U7.5 (VOUT)
- net GND: now also C27.2, C28.2, Q2.2 (S), Q3.2 (S), Q4.2 (S), Q5.2 (S), R32.2, R33.2, R34.2, R35.2, U7.2 (GND)
- net IO11: now also R21.1
- net IO21: now also R10.1
- net IO45: now also R13.1
- net IO9: now also R11.1
- net VBAT: now also C12.1, C21.1, C23.1, C24.1, D5.1 (K), D6.1 (K), D7.1 (K), D8.1 (K)
- net VSYS: now also U7.1 (VIN/EN), U7.3 (VIN)
- new net: C24.2, D6.2 (A), Q2.3 (D)
- new net: C21.2, D7.2 (A), Q5.3 (D)
- new net: Q2.1 (G), R10.2, R35.1
- new net: Q3.1 (G), R21.2, R32.1
- new net: C12.2, D8.2 (A), Q3.3 (D)
- new net: Q4.1 (G), R11.2, R33.1
- new net: Q5.1 (G), R13.2, R34.1
- new net: C23.2, D5.2 (A), Q4.3 (D)
Other:
- moved on the sheet: C17, C3, C39, D3, J3, R25

Commit message: save
Other:
- moved on the sheet: C12, C21, C23, C24, C27, C28, C37, C38, D5, D6, D7, D8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

Commit message: save
Parts:
- added U6: NUP2202, Package_TO_SOT_SMD:SOT-363_SC-70-6, symbol Power_Protection:NUP2202
- R4, R5: value R -> 1k
Connections:
- net 5V: now also U6.5
- net GND: now also U6.2
- net IO10: now also R11.1
- net IO38: now also R13.1
- net IO45: no longer R13.1
- net IO5: no longer R4.2, U4.20 (COM0), U5.3 (SDI)
- net IO6: no longer R5.2, U4.19 (COM1), U5.4 (SCK)
- net IO8: now also R4.2, U4.20 (COM0), U5.3 (SDI)
- net IO9: now also R5.2, U4.19 (COM1), U5.4 (SCK); no longer R11.1
- net USB_D+: now also U6.6
- net USB_D-: now also U6.1
