File: esp32_mine.kicad_pcb (KiCad board)
At the start: 2 copper layers, 36 x 68.8 mm, 76 parts, among them J1 USB_C_Receptacle_USB2.0_14P, J2 Conn_01x02_Pin, J3 Conn_01x18_Pin, J5 Conn_01x18_Pin, Q1 AO3401A, U1 ESP32-S3, U2 W25Q128JVS, U3 MCP73831-2-OT, U4 AMS1117-3.3, Y1 32.768 kHz, Y2 40MHz(10ppm)

Commit message: save
Parts:
- removed +3V3: +3V3, TestPoint:TestPoint_Pad_D1.0mm
- removed BTN1: BTN, Button_Switch_SMD:SW_Push_1P1T_XKB_TS-1187A
- removed Flash1: Flash, Button_Switch_SMD:SW_Push_1P1T_XKB_TS-1187A
- removed G***: LOGO, Library:logo
- removed GND1: GND, TestPoint:TestPoint_Pad_D1.0mm
- removed J2: Conn_01x02_Pin, Connector_PinSocket_2.54mm:PinSocket_1x02_P2.54mm_Vertical
- removed J5: Conn_01x18_Pin, Connector_PinHeader_2.54mm:PinHeader_1x18_P2.54mm_Vertical
- removed Reset1: Reset, Button_Switch_SMD:SW_Push_1P1T_XKB_TS-1187A
- added C1: 12pF, Capacitor_SMD:C_0402_1005Metric, B.Cu at (107.6, 101.5)
- added C15: 0.1uF, Capacitor_SMD:C_0603_1608Metric, F.Cu at (94.6, 106.5)
- added C16: 10uF, Capacitor_SMD:C_0603_1608Metric, F.Cu at (97.2, 82.7)
- added C17: 10uF, Capacitor_SMD:C_0603_1608Metric, F.Cu at (127.6, 87.7)
- added C18: 0.1uF, Capacitor_SMD:C_0603_1608Metric, F.Cu at (127.6, 107.4)
- added C5: 12pF, Capacitor_SMD:C_0402_1005Metric, B.Cu at (109.2, 103.0)
- added C9: C, Capacitor_SMD:C_0603_1608Metric, B.Cu at (110.5, 92.2)
- added D2: LED, Diode_SMD:D_SOD-323, F.Cu at (95.2, 109.8)
- added D3: LED, Diode_SMD:D_SOD-323, F.Cu at (96.0, 81.4)
- added D4: SS14, Diode_SMD:D_SOD-323, F.Cu at (128.8, 84.5)
- added D5: 1N4148W, Diode_SMD:D_SOD-323, F.Cu at (127.6, 110.0)
- added R18: 33R, Resistor_SMD:R_0603_1608Metric, F.Cu at (90.9, 104.4)
- added R19: 200K, Resistor_SMD:R_0603_1608Metric, F.Cu at (91.7, 87.9)
- added R20: 100K, Resistor_SMD:R_0603_1608Metric, F.Cu at (131.6, 87.6)
- added R3: 10k, Resistor_SMD:R_0402_1005Metric, F.Cu at (130.9, 95.9)
- added R5: R, Resistor_SMD:R_0402_1005Metric, F.Cu at (126.8, 94.1)
- added R6: 10k, Resistor_SMD:R_0402_1005Metric, B.Cu at (115.5, 96.4)
- added R7: 10k, Resistor_SMD:R_0402_1005Metric, B.Cu at (112.7, 93.5)
- added R8: 10k, Resistor_SMD:R_0402_1005Metric, B.Cu at (108.5, 93.2)
- added R9: 10k, Resistor_SMD:R_0402_1005Metric, B.Cu at (107.3, 95.6)
- added REF**: PinHeader_1x02_P2.54mm_Vertical, Connector_PinHeader_2.54mm:PinHeader_1x02_P2.54mm_Vertical, F.Cu at (132.0, 73.9)
- added REF**: PinHeader_1x02_P2.54mm_Vertical, Connector_PinHeader_2.54mm:PinHeader_1x02_P2.54mm_Vertical, F.Cu at (91.1, 74.1)
- added REF**: PinHeader_1x02_P2.54mm_Vertical, Connector_PinHeader_2.54mm:PinHeader_1x02_P2.54mm_Vertical, F.Cu at (89.4, 116.4)
- added REF**: PinHeader_1x02_P2.54mm_Vertical, Connector_PinHeader_2.54mm:PinHeader_1x02_P2.54mm_Vertical, F.Cu at (133.3, 116.8)
- added T1: SI2302DS-T1, SI2302DS-T1:SOT95P237X112-3N, F.Cu at (90.9, 107.3)
- added T2: SI2302DS-T1, SI2302DS-T1:SOT95P237X112-3N, F.Cu at (91.9, 85.1)
- added T3: SI2302DS-T1, SI2302DS-T1:SOT95P237X112-3N, F.Cu at (131.7, 84.7)
- added T4: SI2302DS-T1, SI2302DS-T1:SOT95P237X112-3N, F.Cu at (128.3, 104.3)
- added U3: MCP73831-2-OT, XIAO ESP32S3_v1.2_230725:BGA6-0.35-0.745X10.95X0.4MM, F.Cu at (102.9, 91.2)
- added U5: BMP280, Package_LGA:Bosch_LGA-8_2x2.5mm_P0.65mm_ClockwisePinNumbering, F.Cu at (129.0, 95.7)
- added Y3: 32.768 kHz, Crystal:Crystal_SMD_3215-2Pin_3.2x1.5mm, B.Cu at (110.2, 100.8)
- C16, C2, C22, C36, C6, C8, D1, D4, J1, Q1, R1, R12, R14, R15, R17, R18, R19, R2, R20, R27, U3: moved to B.Cu
- J3: value Conn_01x18_Pin -> GPIO; footprint Connector_PinHeader_2.54mm:PinHeader_1x18_P2.54mm_Vertical -> Connector_PinHeader_2.54mm:PinHeader_2x03_P2.54mm_Vertical
- R21: value 10K -> 10k; footprint Resistor_SMD:R_0402_1005Metric -> Resistor_SMD:R_0603_1608Metric
- R4: value 10K -> R
- U2: footprint Package_SO:SOIC-8_5.3x5.3mm_P1.27mm -> Ic:USON8-0.8-3X3X0.55MM
- U4: value AMS1117-3.3 -> BNO055; footprint Package_TO_SOT_SMD:SOT-223-3_TabPin2 -> Package_LGA:LGA-28_5.2x3.8mm_P0.5mm; moved to B.Cu
- moved AE1 85.9 mm to (113.0, 115.7), turned to 180 degrees
- moved C14 74.6 mm to (119.7, 111.3), turned to -135 degrees
- moved C33 73.9 mm to (112.8, 110.7), turned to -90 degrees
- moved Y2 73.5 mm to (115.3, 110.6), turned to 180 degrees
- moved C4 73.5 mm to (117.7, 110.6), turned to -90 degrees
- moved L5 72.7 mm to (121.1, 109.9), turned to 45 degrees
- moved R24 71.8 mm to (112.3, 109.1), turned to 180 degrees
- moved C31 70.6 mm to (122.0, 108.3), turned to 0 degrees
- moved C39 69.7 mm to (118.9, 107.9), turned to -90 degrees
- moved C40 69.7 mm to (117.9, 107.9), turned to -90 degrees
- moved U2 69.5 mm to (104.8, 105.3), turned to 90 degrees
- moved C11 69.3 mm to (112.4, 107.4), turned to 180 degrees
- moved R23 69.0 mm to (116.6, 107.4), turned to 90 degrees
- moved R31 68.7 mm to (114.9, 107.1), turned to 180 degrees
- moved L6 68.2 mm to (121.1, 106.7), turned to -45 degrees
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Connections:
- J3 pad 1: IO6 -> GND
- J3 pad 2: IO9 -> VBAT
- J3 pad 3: IO10 -> RX
- J3 pad 4: IO11 -> GND
- J3 pad 5: IO3 -> TX
- J3 pad 6: IO5 -> IO0
- R12 pad 2: IO4/BAT -> IO12
- R19 pad 1: IO4/BAT -> IO12
- R21 pad 1: VDD_CPU -> GND
- R21 pad 2: IO0 -> /MOT_4
- R4 pad 2: IO14 -> IO5
- U1 pad 14: IO9 -> /MOT_4
- U1 pad 9: IO4/BAT -> IO4
- U4 pad 1: GND -> unconnected-(U4-PIN1-Pad1)
- U4 pad 2: VDD_CPU -> GND
- U4 pad 3: VSYS -> VDD_CPU
Routing:
- net +BATT: track 0.00 -> 196.2 mm
- net IO14: track 71.9 -> 0.00 mm, vias 3 -> 0
- net IO4/BAT: track 58.3 -> 0.00 mm, vias 2 -> 0
- net /MOT_1: track 0.00 -> 36.7 mm
- net IO33: track 36.7 -> 0.79 mm
- net IO48: track 41.5 -> 6.74 mm
- net IO21: track 34.4 -> 0.00 mm, vias 3 -> 2
- net IO13: track 33.3 -> 0.00 mm, vias 3 -> 0
- net IO34: track 34.0 -> 0.76 mm
- net /MOT_2: track 0.00 -> 31.7 mm
- net IO35: track 31.3 -> 0.59 mm
- net IO18/SDA: track 34.2 -> 4.11 mm, vias 3 -> 0
- net IO17/SCL: track 33.3 -> 3.60 mm, vias 3 -> 0
- net IO36: track 30.1 -> 0.43 mm
- net IO8: track 28.9 -> 0.00 mm, vias 2 -> 0
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Other:
- board size 36 x 68.8 mm -> 100 x 100 mm
- copper layers 2 -> 6
- board text added: "100ohm SINGLE ENDED IMPEDANCE CONTROL +/-10%"
- board text added: "13 REF:L3"
- board text added: "4/4"
- board text added: "5.7"
- board text added: "50ohm SINGLE ENDED IMPEDANCE CONTROL +/-10%"
- board text added: "90ohm DIFFERENTIAL IMPEDANCE CONTROL +/-10%"
- board text added: "COPPER WEIGHT (OZ)"
- board text added: "HALF+PLATING=1OZ"
- board text added: "HALF=0.5OZ"
- board text added: "LAYER 1 - GTL"
- board text added: "LAYER 2 - GND"
- board text added: "LAYER 3 - SIG1"
- board text added: "LAYER 4 - SIG2"
- board text added: "LAYER 5 - GND"
- board text added: "LAYER 6 - GBL"
- board text added: "LAYER STACK-UP - ALL DIMENSIONS IN MIL"
- board text added: "LAYER#"
- board text added: "TRACE WIDTH"
- board text added: "TRACE WIDTH / SPACE"
- board text removed: "00"
- board text removed: "02"
- board text removed: "03"
- board text removed: "05"
- board text removed: "07"
- board text removed: "08"
- board text removed: "09"
- board text removed: "10"
- board text removed: "11"
- board text removed: "12"
- board text removed: "13"
- board text removed: "14"
- board text removed: "17"
- board text removed: "18"
- board text removed: "21"
- board text removed: "33"
- board text removed: "34"
- board text removed: "35"
- board text removed: "36"
- board text removed: "37"
- board text removed: "38"
- board text removed: "39"
- board text removed: "40"
- board text removed: "41"
- board text removed: "42"
- board text removed: "45"
- board text removed: "46"
- board text removed: "47"
- board text removed: "48"
- board text removed: "5V"
- board text removed: "O6"

Commit message: save
Parts:
- removed the U3 at (102.9, 91.2)
- added C27: 0.1uF, Capacitor_SMD:C_0603_1608Metric, F.Cu at (131.2, 97.6)
- added C28: 10uF, Capacitor_SMD:C_0603_1608Metric, B.Cu at (104.6, 97.5)
- added R10: R, Resistor_SMD:R_0402_1005Metric, F.Cu at (94.4, 89.5)
- added R11: R, Resistor_SMD:R_0402_1005Metric, F.Cu at (126.2, 99.3)
- added R13: R, Resistor_SMD:R_0402_1005Metric, F.Cu at (99.5, 108.3)
- added R21: R, Resistor_SMD:R_0402_1005Metric, F.Cu at (129.3, 89.9)
- added U7: RT9701, Package_TO_SOT_SMD:SOT-23-5, F.Cu at (103.6, 90.7)
- C12: renamed from C17; value 10uF -> C
- C21: renamed from C15; value 0.1uF -> C
- C23: renamed from C18; value 0.1uF -> C
- C24: renamed from C16; value 10uF -> C
- C9: value C -> 0.1uF
- D5: value 1N4148W -> D
- D6: renamed from D3; value LED -> D
- D7: renamed from D2; value LED -> D
- D8: renamed from D4; value SS14 -> D
- Q2: renamed from T2; value SI2302DS-T1 -> Q_NMOS_GSD
- Q3: renamed from T3; value SI2302DS-T1 -> Q_NMOS_GSD
- Q4: renamed from T4; value SI2302DS-T1 -> Q_NMOS_GSD
- Q5: renamed from T1; value SI2302DS-T1 -> Q_NMOS_GSD
- R32: renamed from R20; value 100K -> 10k
- R34: renamed from R18; value 33R -> 10k
- R35: renamed from R19; value 200K -> 10k
- moved R27 1.53 mm to (104.4, 99.3)
- moved R8 1.02 mm to (107.9, 94.0), turned to 180 degrees
- moved R4 0.91 mm to (126.0, 96.0), turned to 0 degrees
- moved C7 0.89 mm to (106.2, 93.0)
- moved R3 0.88 mm to (130.9, 95.0)
- moved R6 0.71 mm to (115.0, 95.9), turned to 90 degrees
- moved R28 0.13 mm to (105.9, 100.3)
- turned R32 to 0 degrees
- turned R33 to 180 degrees
- turned R34 to 180 degrees
- turned R35 to 0 degrees
- renumbered REF** to M1, REF** to M2, REF** to M3, REF** to M4, R21 to R33
Connections:
- C12 pad 1: VDD_CPU -> VBAT
- C12 pad 2: GND -> Net-(D8-A)
- C21 pad 1: EN -> VBAT
- C21 pad 2: GND -> Net-(D7-A)
- C23 pad 1: VDD_CPU -> VBAT
- C23 pad 2: GND -> Net-(D5-A)
- C24 pad 1: 5V -> VBAT
- C24 pad 2: GND -> Net-(D6-A)
- D5 pad 1: +BATT -> VBAT
- D6 pad 1: Net-(D3-K) -> VBAT
- D6 pad 2: IO1 -> Net-(D6-A)
- D7 pad 1: Net-(D2-K) -> VBAT
- D7 pad 2: VDD_CPU -> Net-(D7-A)
- D8 pad 1: VSYS -> VBAT
- D8 pad 2: 5V -> Net-(D8-A)
- M1 pad 1: (no net) -> Net-(D7-A)
- M1 pad 2: +BATT -> VBAT
- M2 pad 1: +BATT -> VBAT
- M2 pad 2: (no net) -> Net-(D6-A)
- M3 pad 1: +BATT -> VBAT
- M3 pad 2: (no net) -> Net-(D8-A)
- M4 pad 1: (no net) -> Net-(D5-A)
- M4 pad 2: +BATT -> VBAT
- Q2 pad 1: /MOT_2 -> Net-(Q2-G)
- Q2 pad 3: Net-(D3-A) -> Net-(D6-A)
- Q3 pad 1: /MOT_3 -> Net-(Q3-G)
- Q3 pad 3: Net-(D4-A) -> Net-(D8-A)
- Q4 pad 1: /MOT_4 -> Net-(Q4-G)
- Q5 pad 1: /MOT_1 -> Net-(Q5-G)
- Q5 pad 3: Net-(D2-A) -> Net-(D7-A)
- R32 pad 1: GND -> Net-(Q3-G)
- R32 pad 2: 5V -> GND
- R33 pad 1: GND -> Net-(Q4-G)
- R33 pad 2: /MOT_4 -> GND
- R34 pad 1: USB_D+ -> Net-(Q5-G)
- R34 pad 2: USB_D+ -> GND
- R35 pad 1: IO12 -> Net-(Q2-G)
- U1 pad 14: /MOT_4 -> IO9
Routing:
- net VBAT: track 10.1 -> 229.1 mm
- net +BATT: track 196.2 -> 0.00 mm
- net /MOT_1: track 36.7 -> 0.00 mm
- net /MOT_2: track 31.7 -> 0.00 mm
- net VDD_CPU: track 100.1 -> 129.1 mm, vias 7 -> 11
- net /MOT_3: track 27.8 -> 0.00 mm
- net IO21: track 0.00 -> 24.1 mm
- net /MOT_4: track 23.9 -> 0.00 mm, vias 2 -> 0
- net IO11: track 0.00 -> 22.2 mm
- net IO45: track 0.00 -> 22.1 mm
- net EN: track 24.6 -> 42.9 mm
- net Net-(D8-A): track 0.00 -> 16.8 mm
- net Net-(D7-A): track 0.00 -> 16.2 mm
- net Net-(D6-A): track 0.00 -> 14.5 mm
- net VSYS: track 15.3 -> 29.4 mm, vias 2 -> 3
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Other:
- board text removed: "3.3 V"

Commit message: save
Other:
- copper layers 6 -> 4

Commit message: save
Parts:
- added U6: NUP2202, Package_TO_SOT_SMD:SOT-363_SC-70-6, F.Cu at (102.3, 84.0)
- renumbered R2 to R18, R18 to R2
Connections:
- R11 pad 1: IO9 -> IO10
- R13 pad 1: IO45 -> IO38
- R18 pad 1: USB_D- -> USB_D+
- R18 pad 2: USB_D- -> USB_D+
- R2 pad 1: USB_D+ -> USB_D-
- R2 pad 2: USB_D+ -> USB_D-
- R4 pad 2: IO5 -> IO8
- R5 pad 2: IO6 -> IO9
- U4 pad 19: IO6 -> IO9
- U4 pad 20: IO5 -> IO8
- U5 pad 3: IO5 -> IO8
- U5 pad 4: IO6 -> IO9
Routing:
- net IO6: track 24.3 -> 0.00 mm, vias 2 -> 0
- net IO5: track 23.9 -> 0.00 mm, vias 2 -> 0
- net IO8: track 0.00 -> 22.6 mm, vias 0 -> 2
- net IO45: track 22.1 -> 1.75 mm, vias 2 -> 0
- net IO38: track 0.00 -> 15.9 mm, vias 0 -> 2
- net IO10: track 0.00 -> 11.5 mm, vias 0 -> 2
- net IO9: track 12.0 -> 22.7 mm
- net 5V: track 43.0 -> 50.9 mm
- net GND: track 7.54 -> 9.74 mm, vias 160 -> 208
- net USB_D-: track 26.5 -> 27.9 mm
- net USB_D+: track 27.8 -> 28.8 mm
- added copper zone on In1.Cu, net GND
- added copper zone on In2.Cu, net GND

Commit message: save
Routing:
- net GND: vias 208 -> 201
Changed lines of the file:
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@@
 		(filling no)
 		(pcbplotparams
-			(layerselection 0x00000000_00000000_55555555_5755f0af)
+			(layerselection 0x00000000_00000000_55555555_5755f5ff)
 			(plot_on_all_layers_selection 0x00000000_00000000_00000000_00000000)
 			(disableapertmacros no)
-			(usegerberextensions no)
+			(usegerberextensions yes)
 			(usegerberattributes yes)
 			(usegerberadvancedattributes yes)
-			(creategerberjobfile yes)
+			(creategerberjobfile no)
 			(dashed_line_dash_ratio 12)
 			(dashed_line_gap_ratio 3)
@@
 	)
 	(via
-		(at 105.5 115.15)
+		(at 105.4 115.5)
 		(size 0.6)
 		(drill 0.3)
@@
 	)
 	(via
-		(at 124.68 113.89)
+		(at 125.3 114.5)
 		(size 0.6)
 		(drill 0.3)
@@
 	)
 	(via
-		(at 106.6 114.55)
+		(at 106.7 114.7)
 		(size 0.6)
 		(drill 0.3)
@@
 	)
 	(via
-		(at 111.55 114.6)
+		(at 111.5 114.6)
 		(size 0.6)
 		(drill 0.3)
@@
 	)
 	(via
-		(at 102.9 115.65)
+		(at 102.8 115.5)
 		(size 0.6)
 		(drill 0.3)
@@
 	)
 	(via
-		(at 108 115.65)
+		(at 107.5 115.6)
 		(size 0.6)
 		(drill 0.3)
@@
 	)
 	(via
-		(at 117.35 114.4)
+		(at 117.1 114.6)
 		(size 0.6)
 		(drill 0.3)
@@
 	)
 	(via
-		(at 110.25 113.55)
-		(size 0.6)
-		(drill 0.3)
-		(layers "F.Cu" "B.Cu")
-		(free yes)
-		(capping no)
-		(covering
-			(front no)
-			(back no)
-		)
-		(plugging
-			(front no)
-			(back no)
-		)
-		(filling no)
-		(net "GND")
-	)
-	(via
 		(at 106.45 115.55)
 		(size 0.6)
@@
 	)
 	(via
-		(at 112.5 114.6)
+		(at 112.4 114.7)
 		(size 0.6)
 		(drill 0.3)
@@
 	)
 	(via
-		(at 112.05 113.35)
-		(size 0.6)
-		(drill 0.3)
-		(layers "F.Cu" "B.Cu")
-		(free yes)
-		(capping no)
-		(covering
-			(front no)
-			(back no)
-		)
-		(plugging
-			(front no)
-			(back no)
-		)
-		(filling no)
-		(net "GND")
-	)
-	(via
 		(at 124.68 100.489615)
 		(size 0.6)
@@
 	)
 	(via
-		(at 111.05 113.2)
-		(size 0.6)
-		(drill 0.3)
-		(layers "F.Cu" "B.Cu")
-		(free yes)
-		(capping no)
-		(covering
-			(front no)
-			(back no)
-		)
-		(plugging
-			(front no)
-			(back no)
-		)
-		(filling no)
-		(net "GND")
-	)
-	(via
-		(at 101.4 114.65)
+		(at 101.6 114.7)
 		(size 0.6)
 		(drill 0.3)
@@
 	)
 	(via
-		(at 100.4 114.6)
+		(at 100.7 114.6)
 		(size 0.6)
 		(drill 0.3)
@@
 	)
 	(via
-		(at 109.35 115.65)
-		(size 0.6)
-		(drill 0.3)
-		(layers "F.Cu" "B.Cu")
-		(free yes)
-		(capping no)
-		(covering
-			(front no)
-			(back no)
-		)
-		(plugging
-			(front no)
-			(back no)
-		)
-		(filling no)
-		(net "GND")
-	)
-	(via
-		(at 115.9 113.05)
+		(at 109.4 115.5)
 		(size 0.6)
 		(drill 0.3)
@@
 	)
 	(via
-		(at 104.1 114.55)
+		(at 104.5 115.5)
 		(size 0.6)
 		(drill 0.3)
@@
 	)
 	(via
-		(at 107.35 115.1)
+		(at 107.5 114.7)
 		(size 0.6)
 		(drill 0.3)
@@
 	)
 	(via
-		(at 129.8 114.7)
+		(at 129.6 114.8)
 		(size 0.6)
 		(drill 0.3)
@@
 	)
 	(via
-		(at 130.1 115.35)
+		(at 130.2 115.3)
 		(size 0.6)
 		(drill 0.3)
@@
 	)
 	(via
-		(at 110.5 114.55)
+		(at 110.4 114.6)
 		(size 0.6)
 		(drill 0.3)
@@
 	)
 	(via
-		(at 114.05 113.2)
+		(at 115.3 114.5)
 		(size 0.6)
 		(drill 0.3)
@@
 	)
 	(via
-		(at 103.55 115.1)
+		(at 103.8 114.8)
 		(size 0.6)
 		(drill 0.3)
@@
 	)
 	(via
-		(at 123.8 115.057693)
+		(at 123.4 114.8)
 		(size 0.6)
 		(drill 0.3)
@@
 	)
 	(via
-		(at 99.55 114.6)
+		(at 99.7 114.6)
 		(size 0.6)
 		(drill 0.3)
@@
 	)
 	(via
-		(at 105.8 114.5)
+		(at 105.8 114.7)
 		(size 0.6)
 		(drill 0.3)
@@
 	)
 	(via
-		(at 108.6 113.65)
-		(size 0.6)
-		(drill 0.3)
-		(layers "F.Cu" "B.Cu")
-		(free yes)
-		(capping no)
-		(covering
-			(front no)
-			(back no)
-		)
-		(plugging
-			(front no)
-			(back no)
-		)
-		(filling no)
-		(net "GND")
-	)
-	(via
-		(at 120.85 115.55)
+		(at 120.7 115.5)
 		(size 0.6)
 		(drill 0.3)
@@
 	)
 	(via
-		(at 104.45 115.65)
+		(at 103.7 115.5)
 		(size 0.6)
 		(drill 0.3)
@@
 	)
 	(via
-		(at 132.8 111.7)
+		(at 132.7 111.7)
 		(size 0.6)
 		(drill 0.3)
@@
 	)
 	(via
-		(at 117.25 112.8)
+		(at 118 114.7)
 		(size 0.6)
 		(drill 0.3)
@@
 	)
 	(via
-		(at 120.73 114.68)
+		(at 121.4 114.8)
 		(size 0.6)
 		(drill 0.3)
@@
 	)
 	(via
-		(at 105.2 113.7)
-		(size 0.6)
-		(drill 0.3)
-		(layers "F.Cu" "B.Cu")
-		(free yes)
-		(capping no)
-		(covering
-			(front no)
-			(back no)
-		)
-		(plugging
-			(front no)
-			(back no)
-		)
-		(filling no)
-		(net "GND")
-	)
-	(via
 		(at 110.5416 87.2233)
 		(size 0.6)
@@
 	)
 	(via
-		(at 119.73 114.38)
+		(at 119.9 114.7)
 		(size 0.6)
 		(drill 0.3)
@@
 	)
 	(via
-		(at 118.45 112.7)
+		(at 120.7 114.7)
 		(size 0.6)
 		(drill 0.3)
@@
 	)
 	(via
-		(at 118.7 114.3)
+		(at 118.9 114.7)
 		(size 0.6)
 		(drill 0.3)
@@
 	)
 	(via
-		(at 116.1 114.6)
+		(at 116.2 114.7)
 		(size 0.6)
 		(drill 0.3)
@@
 	)
 	(via
-		(at 124.68 114.795)
+		(at 124.4 114.8)
 		(size 0.6)
 		(drill 0.3)
@@
 	)
 	(via
-		(at 98.7 114.45)
+		(at 98.9 114.5)
 		(size 0.6)
 		(drill 0.3)
@@
 	)
 	(via
-		(at 108.45 115.1)
+		(at 108.5 115.5)
 		(size 0.6)
 		(drill 0.3)
@@
 	)
 	(via
-		(at 107.6 113.75)
-		(size 0.6)
-		(drill 0.3)
-		(layers "F.Cu" "B.Cu")
-		(free yes)
-		(capping no)
-		(covering
-			(front no)
-			(back no)
-		)
-		(plugging
-			(front no)
-			(back no)
-		)
-		(filling no)
-		(net "GND")
-	)
-	(via
 		(at 121.33 114.08)
 		(size 0.6)
@@
 	)
 	(via
-		(at 101.75 115.4)
+		(at 101.9 115.5)
 		(size 0.6)
 		(drill 0.3)
@@
 	)
 	(via
-		(at 130.65 114.9)
+		(at 130.8 114.8)
 		(size 0.6)
 		(drill 0.3)
@@
 	)
 	(via
-		(at 107.95 114.45)
+		(at 108.5 114.7)
 		(size 0.6)
 		(drill 0.3)
@@
 	)
 	(via
-		(at 102.65 114.85)
+		(at 102.7 114.7)
 		(size 0.6)
 		(drill 0.3)
@@
 	)
 	(via
-		(at 109.3 114.6)
+		(at 109.5 114.6)
 		(size 0.6)
 		(drill 0.3)
