File: Camera/spoel.kicad_pcb (KiCad board)
At the start: 4 copper layers, 48 x 25 mm, 7 parts, among them J2 HDMI, J3 header15, J4 header15, Q1 Q_NPN_BCE

Commit message: merge
Parts:
- removed J?: GPIOs, Connector_PinHeader_2.54mm:PinHeader_1x04_P2.54mm_Vertical_SMD_Pin1Left
- removed Q1: Q_NPN_BCE, ESP32-footprints-Lib:Dpak
- moved J4 28.0 mm to (115.6, 83.2)
- moved R1 27.1 mm to (97.9, 116.2)
- moved R2 27.1 mm to (97.9, 108.2)
- moved J3 25.0 mm to (90.6, 83.2)
- moved J2 23.9 mm to (94.0, 68.5)
Routing:
- net (no net): vias 4 -> 0
Other:
- board outline removed
