File: Solar/solar.kicad_pcb (KiCad board)
At the start: 2 copper layers, 79 x 77 mm, 40 parts, among them IC1 MAX4173H, J1 SOLAR_INPUT, J2 Left, J3 Right, J4 BATTERY_OUTPUT, J5 header3, J6 in, J7 SOLAR_OUTPUT, Q2 IRFIZ44N, U1 HMHA2801, U2 MAX5424

Commit message: merge
Routing:
- net Net-(J3-Pad12): track 45.2 -> 43.7 mm
- net Solar+: track 132.0 -> 131.2 mm
Changed lines of the file:
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@@
   (via (at 101.346 106.934) (size 0.59944) (drill 0.29972) (layers "F.Cu" "B.Cu") (net 2))
   (via (at 114 58) (size 0.59944) (drill 0.29972) (layers "F.Cu" "B.Cu") (net 2))
-  (via (at 72.009 93.853) (size 0.59944) (drill 0.29972) (layers "F.Cu" "B.Cu") (net 2))
+  (via (at 73 95) (size 0.59944) (drill 0.29972) (layers "F.Cu" "B.Cu") (net 2))
   (via (at 95 43) (size 0.59944) (drill 0.29972) (layers "F.Cu" "B.Cu") (net 2))
   (via (at 53 96) (size 0.59944) (drill 0.29972) (layers "F.Cu" "B.Cu") (net 2))
@@
   (segment (start 66.776277 93) (end 71.821477 87.9548) (width 0.14986) (layer "F.Cu") (net 11))
   (segment (start 59.762 93) (end 66.776277 93) (width 0.14986) (layer "F.Cu") (net 11))
-  (segment (start 83.693 79.856376) (end 83.693 83.82) (width 0.14986) (layer "F.Cu") (net 12))
-  (segment (start 83.439 84.074) (end 83.166 84.074) (width 0.14986) (layer "F.Cu") (net 12))
-  (segment (start 84.774 72.898) (end 84.774 78.775376) (width 0.14986) (layer "F.Cu") (net 12))
-  (segment (start 83.166 84.074) (end 80.76 86.48) (width 0.14986) (layer "F.Cu") (net 12))
-  (segment (start 83.693 83.82) (end 83.439 84.074) (width 0.14986) (layer "F.Cu") (net 12))
-  (segment (start 84.774 78.775376) (end 83.693 79.856376) (width 0.14986) (layer "F.Cu") (net 12))
-  (segment (start 80.76 86.48) (end 80.76 86.73) (width 0.14986) (layer "F.Cu") (net 12))
+  (segment (start 84.774 78.775376) (end 84.774 72.898) (width 0.14986) (layer "F.Cu") (net 12))
+  (segment (start 80.76 86.73) (end 80.76 86.48) (width 0.14986) (layer "F.Cu") (net 12))
+  (segment (start 80.76 86.48) (end 83.693 83.547) (width 0.14986) (layer "F.Cu") (net 12))
+  (segment (start 83.693 79.856376) (end 84.774 78.775376) (width 0.14986) (layer "F.Cu") (net 12))
+  (segment (start 83.693 83.547) (end 83.693 79.856376) (width 0.14986) (layer "F.Cu") (net 12))
+  (segment (start 106.89938 51.95932) (end 110 55.05994) (width 0.5) (layer "F.Cu") (net 13))
   (segment (start 104.013 50.038) (end 98.112 50.038) (width 0.5) (layer "F.Cu") (net 13))
-  (segment (start 106.89938 51.95932) (end 110 55.05994) (width 0.5) (layer "F.Cu") (net 13))
   (segment (start 106.00036 54.04954) (end 105.93432 53.9835) (width 0.14986) (layer "F.Cu") (net 13))
+  (segment (start 110 55.05994) (end 110 67.375) (width 0.5) (layer "F.Cu") (net 13))
   (segment (start 95.25 54.14518) (end 93.9499 54.14518) (width 0.5) (layer "F.Cu") (net 13))
+  (segment (start 105.93432 51.95932) (end 106.89938 51.95932) (width 0.5) (layer "F.Cu") (net 13))
   (segment (start 106.138 50.038) (end 104.013 50.038) (width 0.5) (layer "F.Cu") (net 13))
   (segment (start 64.135 57.023) (end 62.255 58.903) (width 0.5) (layer "F.Cu") (net 13))
-  (segment (start 105.93432 51.95932) (end 106.89938 51.95932) (width 0.5) (layer "F.Cu") (net 13))
   (segment (start 98.112 50.038) (end 98.04 50.11) (width 0.5) (layer "F.Cu") (net 13))
   (segment (start 105.93432 54.38355) (end 105.93432 53.9835) (width 0.5) (layer "F.Cu") (net 13))
@@
   (segment (start 105.93432 53.13387) (end 105.93432 51.95932) (width 0.14986) (layer "F.Cu") (net 13))
   (segment (start 117.469861 109.480139) (end 117.469861 85.410111) (width 0.5) (layer "F.Cu") (net 13))
-  (segment (start 111.3155 68.6905) (end 114 71.375) (width 0.5) (layer "F.Cu") (net 13))
   (segment (start 116.32 112.13) (end 116.32 110.63) (width 0.5) (layer "F.Cu") (net 13))
+  (segment (start 110 67.375) (end 114 71.375) (width 0.5) (layer "F.Cu") (net 13))
   (segment (start 116.32 110.63) (end 117.469861 109.480139) (width 0.5) (layer "F.Cu") (net 13))
-  (segment (start 110 55.05994) (end 110 68.6905) (width 0.5) (layer "F.Cu") (net 13))
   (segment (start 73.406 57.023) (end 64.135 57.023) (width 0.5) (layer "F.Cu") (net 13))
-  (segment (start 114 71.375) (end 114 73.145) (width 0.5) (layer "F.Cu") (net 13))
   (segment (start 105.93432 53.9835) (end 105.93432 53.13387) (width 0.14986) (layer "F.Cu") (net 13))
   (segment (start 62.255 62.865) (end 68.555 62.865) (width 0.5) (layer "F.Cu") (net 13))
+  (segment (start 114 71.375) (end 114 73.145) (width 0.5) (layer "F.Cu") (net 13))
   (segment (start 75.438 62.357) (end 73.646 60.565) (width 0.5) (layer "F.Cu") (net 13))
   (segment (start 73.646 60.565) (end 73.646 57.263) (width 0.5) (layer "F.Cu") (net 13))
@@
   (segment (start 85.73808 62.357) (end 75.438 62.357) (width 0.5) (layer "F.Cu") (net 13))
   (segment (start 73.646 57.263) (end 73.406 57.023) (width 0.5) (layer "F.Cu") (net 13))
-  (segment (start 110 68.6905) (end 111.3155 68.6905) (width 0.5) (layer "F.Cu") (net 13))
-  (segment (start 69.375209 93.091) (end 69.485698 92.980511) (width 0.14986) (layer "F.Cu") (net 14))
+  (segment (start 62 102.762) (end 62.254 102.762) (width 0.14986) (layer "F.Cu") (net 14))
   (segment (start 62 102.762) (end 62 105.78986) (width 0.14986) (layer "F.Cu") (net 14))
-  (segment (start 62 102.762) (end 62.254 102.762) (width 0.14986) (layer "F.Cu") (net 14))
   (segment (start 63.71014 107.5) (end 64.46 107.5) (width 0.14986) (layer "F.Cu") (net 14))
-  (segment (start 69.485698 92.980511) (end 87.601489 92.980511) (width 0.14986) (layer "F.Cu") (net 14))
-  (segment (start 88.38 86.73) (end 88.38 92.202) (width 0.14986) (layer "F.Cu") (net 14))
+  (segment (start 62.254 102.762) (end 72.035489 92.980511) (width 0.14986) (layer "F.Cu") (net 14))
+  (segment (start 87.601489 92.980511) (end 88.38 92.202) (width 0.14986) (layer "F.Cu") (net 14))
+  (segment (start 72.035489 92.980511) (end 87.601489 92.980511) (width 0.14986) (layer "F.Cu") (net 14))
   (segment (start 64.25014 107.5) (end 65 107.5) (width 0.14986) (layer "F.Cu") (net 14))
-  (segment (start 62.254 102.762) (end 69.375209 95.640791) (width 0.14986) (layer "F.Cu") (net 14))
-  (segment (start 69.375209 95.640791) (end 69.375209 93.091) (width 0.14986) (layer "F.Cu") (net 14))
-  (segment (start 87.601489 92.980511) (end 88.38 92.202) (width 0.14986) (layer "F.Cu") (net 14))
+  (segment (start 88.38 92.202) (end 88.38 86.73) (width 0.14986) (layer "F.Cu") (net 14))
   (segment (start 62 105.78986) (end 63.71014 107.5) (width 0.14986) (layer "F.Cu") (net 14))
   (segment (start 62 102.762) (end 61.746 102.762) (width 0.14986) (layer "F.Cu") (net 14))
@@
   (segment (start 101.346 55.58224) (end 102.94474 53.9835) (width 0.14986) (layer "F.Cu") (net 18))
   (via (at 103.39432 53.9835) (size 0.59944) (drill 0.29972) (layers "F.Cu" "B.Cu") (net 18))
-  (segment (start 112.209 53.721) (end 115.82 50.11) (width 0.14986) (layer "B.Cu") (net 18))
-  (segment (start 109.9735 53.9835) (end 110.236 53.721) (width 0.14986) (layer "B.Cu") (net 18))
-  (segment (start 103.39432 53.9835) (end 109.9735 53.9835) (width 0.14986) (layer "B.Cu") (net 18))
-  (segment (start 110.236 53.721) (end 112.209 53.721) (width 0.14986) (layer "B.Cu") (net 18))
+  (segment (start 103.39432 53.9835) (end 111.9465 53.9835) (width 0.14986) (layer "B.Cu") (net 18))
+  (segment (start 111.9465 53.9835) (end 115.82 50.11) (width 0.14986) (layer "B.Cu") (net 18))
   (segment (start 107.155 99.568) (end 106.83 99.568) (width 0.14986) (layer "F.Cu") (net 19))
   (segment (start 111.24 110.98014) (end 111.24 112.13) (width 0.14986) (layer "F.Cu") (net 19))

Commit message: update
Routing:
- net Net-(J3-Pad12): track 43.7 -> 42.2 mm
- net Net-(D5-Pad2): track 4.34 -> 3.35 mm
- net +3V3: track 96.3 -> 95.4 mm
- net Solar+: track 131.2 -> 130.4 mm
- net Net-(IC1-Pad8): track 25.3 -> 24.7 mm
- net Net-(TX1-Pad1): track 6.17 -> 5.66 mm
