File: drone/Crazyflie contol board.kicad_sch (KiCad schematic)
At the start: 40 parts

Commit message: update
Parts:
- C1: value (none) -> 22uF; footprint (none) -> ESP32-footprints-Lib:0603_new_new
- C2, C3, C5: value (none) -> 100nF; footprint (none) -> ESP32-footprints-Lib:0603_new_new
- C4: value (none) -> 4.7uF; footprint (none) -> ESP32-footprints-Lib:0603_new_new
- D1, D2, D3, D4: value (none) -> BAT54; footprint (none) -> SOD323
- D5: value (none) -> RED LED; footprint (none) -> SMDLED-0603
- D6: value (none) -> GREEN LED; footprint (none) -> SMDLED-0603
- P1, P2, P3, P4: value (none) -> CONN_2; footprint (none) -> PINHEADER_127_2X1
- Q1, Q2, Q3, Q4: value (none) -> PMV31XN; footprint (none) -> SOT23GDS
- Q7, Q8: value (none) -> SS8050-G; footprint (none) -> digikey-footprints:SOT-23-3
- R1, R2, R3, R4: value (none) -> 10k; footprint (none) -> SM0402
- R10, R8, R9: value (none) -> 10k; footprint (none) -> ESP32-footprints-Lib:0603_new_new
- R13, R14: value (none) -> 2.2k; footprint (none) -> ESP32-footprints-Lib:0603_new_new
- R39, R40, R41: value (none) -> 100R; footprint (none) -> SM0402
- R42: value (none) -> 100R; footprint (none) -> digikey-footprints:0603
- R5: value (none) -> 330R; footprint (none) -> ESP32-footprints-Lib:0603_new_new
- R6: value (none) -> 220R; footprint (none) -> ESP32-footprints-Lib:0603_new_new
- R7: value (none) -> 1k; footprint (none) -> ESP32-footprints-Lib:0603_new_new
- SW2: value (none) -> BOOT; footprint (none) -> ESP32-footprints-Lib:Switch_Tactile_SMD_B3U-1000P_new_new
- U11: value (none) -> ESP32-WROOM; footprint (none) -> ESP32-footprints-Lib:ESP32-WROOM-32_new
- U12: value (none) -> CP2102N-A01-GQFN24; footprint (none) -> ESP32-footprints-Lib:QFN-24-1EP_4x4mm_new_new_new
