File: drone/IMU.kicad_sch (KiCad schematic)
At the start: 5 parts

Commit message: update
Parts:
- C18, C20, C24: value (none) -> 100nF; footprint (none) -> ESP32-footprints-Lib:0603_new_new
- U1: value (none) -> BMX160; footprint (none) -> digikey-footprints:LGA-14L_2.5x3mm__LSM6DS3
- U5: value (none) -> MS5611-01BA03; footprint (none) -> MS5611
Changed lines of the file:
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@@
       (effects (font (size 1.27 1.27)) (justify left))
     )
-    (property "Value" "" (id 1) (at 138.43 85.09 0)
+    (property "Value" "100nF" (id 1) (at 138.43 85.09 0)
       (effects (font (size 1.27 1.27)) (justify left))
     )
-    (property "Footprint" "" (id 2) (at 137.16 82.55 0)
+    (property "Footprint" "ESP32-footprints-Lib:0603_new_new" (id 2) (at 137.16 82.55 0)
       (effects (font (size 1.524 1.524)) hide)
     )
@@
       (effects (font (size 1.016 1.016)) hide)
     )
-    (property "Value" "" (id 1) (at 128.27 94.488 0))
+    (property "Value" "AGND" (id 1) (at 128.27 94.488 0))
     (property "Footprint" "" (id 2) (at 128.27 92.71 0)
       (effects (font (size 1.27 1.27)) hide)
@@
       (effects (font (size 0.762 0.762)) hide)
     )
-    (property "Value" "" (id 1) (at 121.92 73.66 0)
+    (property "Value" "VCCA" (id 1) (at 121.92 73.66 0)
       (effects (font (size 0.762 0.762)))
     )
@@
       (effects (font (size 1.27 1.27)) (justify left))
     )
-    (property "Value" "" (id 1) (at 129.54 85.09 0)
+    (property "Value" "100nF" (id 1) (at 129.54 85.09 0)
       (effects (font (size 1.27 1.27)) (justify left))
     )
-    (property "Footprint" "" (id 2) (at 128.27 82.55 0)
+    (property "Footprint" "ESP32-footprints-Lib:0603_new_new" (id 2) (at 128.27 82.55 0)
       (effects (font (size 1.524 1.524)) hide)
     )
@@
       (effects (font (size 1.524 1.524)))
     )
-    (property "Value" "" (id 1) (at 154.94 127 0)
+    (property "Value" "MS5611-01BA03" (id 1) (at 154.94 127 0)
       (effects (font (size 1.524 1.524)))
     )
-    (property "Footprint" "" (id 2) (at 154.94 124.46 0)
+    (property "Footprint" "MS5611" (id 2) (at 154.94 124.46 0)
       (effects (font (size 1.524 1.524)) hide)
     )
@@
       (effects (font (size 1.016 1.016)) hide)
     )
-    (property "Value" "" (id 1) (at 172.72 140.208 0))
+    (property "Value" "AGND" (id 1) (at 172.72 140.208 0))
     (property "Footprint" "" (id 2) (at 172.72 138.43 0)
       (effects (font (size 1.27 1.27)) hide)
@@
       (effects (font (size 1.27 1.27)) (justify left))
     )
-    (property "Value" "" (id 1) (at 135.89 133.35 0)
+    (property "Value" "100nF" (id 1) (at 135.89 133.35 0)
       (effects (font (size 1.27 1.27)) (justify left))
     )
-    (property "Footprint" "" (id 2) (at 134.62 130.81 0)
+    (property "Footprint" "ESP32-footprints-Lib:0603_new_new" (id 2) (at 134.62 130.81 0)
       (effects (font (size 1.524 1.524)) hide)
     )
@@
       (effects (font (size 1.016 1.016)) hide)
     )
-    (property "Value" "" (id 1) (at 132.842 107.95 0))
+    (property "Value" "AGND" (id 1) (at 132.842 107.95 0))
     (property "Footprint" "" (id 2) (at 134.62 107.95 0)
       (effects (font (size 1.27 1.27)) hide)
@@
       (effects (font (size 0.762 0.762)) hide)
     )
-    (property "Value" "" (id 1) (at 125.73 123.19 0)
+    (property "Value" "VCCA" (id 1) (at 125.73 123.19 0)
       (effects (font (size 0.762 0.762)))
     )
@@
       (effects (font (size 1.524 1.524)))
     )
-    (property "Value" "" (id 1) (at 154.94 40.64 0)
+    (property "Value" "BMX160" (id 1) (at 154.94 40.64 0)
       (effects (font (size 1.524 1.524)))
     )
-    (property "Footprint" "" (id 2) (at 154.94 59.69 0)
+    (property "Footprint" "digikey-footprints:LGA-14L_2.5x3mm__LSM6DS3" (id 2) (at 154.94 59.69 0)
       (effects (font (size 1.27 1.27)) hide)
     )
@@
       (effects (font (size 1.016 1.016)) hide)
     )
-    (property "Value" "" (id 1) (at 118.872 48.26 0))
+    (property "Value" "AGND" (id 1) (at 118.872 48.26 0))
     (property "Footprint" "" (id 2) (at 120.65 48.26 0)
       (effects (font (size 1.27 1.27)) hide)
