File: drone/Power.kicad_sch (KiCad schematic)
At the start: 47 parts

Commit message: update
Parts:
- BT1: value (none) -> BATTERY; footprint (none) -> JST-B2B-ZR
- C29, C35: value (none) -> 15pF; footprint (none) -> ESP32-footprints-Lib:0603_new_new
- C30, C31, C34, C37: value (none) -> 4.7uF; footprint (none) -> ESP32-footprints-Lib:0603_new_new
- C32, C40: value (none) -> 10nF; footprint (none) -> ESP32-footprints-Lib:0603_new_new
- C33, C36, C38, C41: value (none) -> 100nF; footprint (none) -> ESP32-footprints-Lib:0603_new_new
- C39: value (none) -> 10uF; footprint (none) -> ESP32-footprints-Lib:0603_new_new
- D7, D8: value (none) -> BLUE LED; footprint (none) -> SMDLED-0603
- P7: value (none) -> MICRO-B-USB; footprint (none) -> ZX62-B-5PA_11_CFK
- P9: value (none) -> CONN_1; footprint (none) -> PINHEADER_127_1X1
- Q5, Q6: value (none) -> 2N7002; footprint (none) -> SOT23GDS
- R16: value (none) -> 39k; footprint (none) -> ESP32-footprints-Lib:0603_new_new
- R17: value (none) -> 10R; footprint (none) -> ESP32-footprints-Lib:0603_new_new
- R18, R28: value (none) -> 30k; footprint (none) -> ESP32-footprints-Lib:0603_new_new
- R19, R29: value (none) -> 0R; footprint (none) -> ESP32-footprints-Lib:0603_new_new
- R20: value (none) -> 42.2k; footprint (none) -> ESP32-footprints-Lib:0603_new_new
- R21: value (none) -> 300k; footprint (none) -> ESP32-footprints-Lib:0603_new_new
- R22, R38: value (none) -> 1k; footprint (none) -> ESP32-footprints-Lib:0603_new_new
- R23: value (none) -> 150k; footprint (none) -> ESP32-footprints-Lib:0603_new_new
- R24: value (none) -> 1.2k; footprint (none) -> ESP32-footprints-Lib:0603_new_new
- R25, R27, R32, R33, R36, R37: value (none) -> 10k; footprint (none) -> ESP32-footprints-Lib:0603_new_new
- R26: value (none) -> 1.2K; footprint (none) -> ESP32-footprints-Lib:0603_new_new
- R30: value (none) -> 20k; footprint (none) -> ESP32-footprints-Lib:0603_new_new
- R31: value (none) -> 100k; footprint (none) -> ESP32-footprints-Lib:0603_new_new
- SW1: value (none) -> PUSH ON/OFF; footprint (none) -> SPST-NO-4x2.5
- U10: value (none) -> MAX16054; footprint (none) -> SOT23_6
- U6: value (none) -> NUF2221; footprint (none) -> SOT363
- U7, U9: value (none) -> TPS79301; footprint (none) -> SOT23_6
- U8: value (none) -> BQ24075; footprint (none) -> QFN16
Other:
- moved on the sheet: SW1
