File: drone/Crazyflie contol board.kicad_pcb (KiCad board)
At the start: 4 copper layers, 40.1 x 38.1 mm, 98 parts, among them P1 CONN_2, P2 CONN_2, P3 CONN_2, P4 CONN_2, P7 MICRO-B-USB, P9 CONN_1, Q1 PMV31XN, Q2 PMV31XN, Q3 PMV31XN, Q4 PMV31XN, Q5 2N7002, Q6 2N7002, Q7 SS8050-G, Q8 SS8050-G, SW1 PUSH ON/OFF, SW2 BOOT, U1 BMX160, U10 MAX16054, U11 ESP32-WROOM, U12 CP2102N-A01-GQFN24, U5 MS5611-01BA03, U6 NUF2221, U7 TPS79301, U8 BQ24075, U9 TPS79301

Commit message: update
Parts:
- moved C4 0.49 mm to (130.2, 95.8)
- moved C1 0.35 mm to (127.2, 118.8)
- moved C3 0.32 mm to (128.8, 95.8)
Routing:
- net DGND: track 50.1 -> 25.6 mm
- net AGND: track 15.5 -> 6.26 mm
- net VCC: track 105.4 -> 103.3 mm
- net /INT_GA: track 27.5 -> 25.9 mm
- net Net-(R6-Pad1): track 33.4 -> 32.5 mm
- net GND: track 78.8 -> 77.8 mm
- net /MOTOR1: track 17.4 -> 16.4 mm
- net /SYSOFF: track 39.8 -> 39.0 mm
- net /I2C_SCK_VCCA: track 41.7 -> 40.9 mm
- net Net-(U11-Pad34): track 32.5 -> 31.7 mm
- net /RED: track 46.9 -> 47.5 mm
- net /I2C_SCL_VCCA: track 43.9 -> 43.3 mm
Other:
- board text added: "Rev. 2.2"
- board text removed: "Rev.2.1"
- board text removed: "Rev.F"

Commit message: save
Routing:
- net GND: track 77.8 -> 51.7 mm
- net /I2C_SCK_VCCA: track 40.9 -> 38.9 mm
- net /RED: track 47.5 -> 46.4 mm
- net Net-(U11-Pad34): track 31.7 -> 30.6 mm
- net DGND: track 25.6 -> 25.5 mm, vias 11 -> 10
