File: TeslaCoil/Tesla_Coil.kicad_pcb (KiCad board)
At the start: 4 copper layers, 200 x 97.5 mm, 37 parts, among them J1 SOLAR_INPUT, J2 SOLAR_OUTPUT, J3 Left, J4 Right, J5 5V, J6 BATTERY_INPUT, J7 BATTERY_OUTPUT, Q1 Q_NPN_BCE, Q4 IRFIZ44N

Commit message: save
Changed lines of the file:
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@@
   (gr_line (start 222.15 141.595) (end 222.6 139.745) (layer "Edge.Cuts") (width 0.2))
   (gr_line (start 211.2 78.345) (end 111.2 78.345) (layer "Edge.Cuts") (width 0.05))
-  (gr_text "12:5" (at 222.2 128.345) (layer "F.Cu")
+  (gr_text "12:5" (at 222.2 130.5) (layer "F.Cu")
     (effects (font (size 1.5 1.5) (thickness 0.3)))
   )
-  (gr_text "5:3" (at 240.2 92.345) (layer "F.Cu")
+  (gr_text "5:3" (at 239 81.5) (layer "F.Cu")
     (effects (font (size 1.5 1.5) (thickness 0.3)))
   )
@@
     (pts (xy 236.2 78.345) (xy 211.2 78.345))
     (height 15.954178)
-    (gr_text "25,0000 mm" (at 223.7 60.590822) (layer "Dwgs.User")
+    (gr_text "25.0000 mm" (at 223.7 60.590822) (layer "Dwgs.User")
       (effects (font (size 1.5 1.5) (thickness 0.3)))
     )
@@
     (pts (xy 221.1 65.845) (xy 221.1 163.345))
     (height 133.1)
-    (gr_text "97,5000 mm" (at 86.2 114.595 90) (layer "Dwgs.User")
+    (gr_text "97.5000 mm" (at 86.2 114.595 90) (layer "Dwgs.User")
       (effects (font (size 1.5 1.5) (thickness 0.3)))
     )
@@
     (pts (xy 111.2 153.345) (xy 111.2 78.345))
     (height -11)
-    (gr_text "75,0000 mm" (at 99.05 115.845 90) (layer "Dwgs.User")
+    (gr_text "75.0000 mm" (at 99.05 115.845 90) (layer "Dwgs.User")
       (effects (font (size 1 1) (thickness 0.15)))
     )
@@
     (pts (xy 311.2 78.345) (xy 211.2 78.345))
     (height 12.5)
-    (gr_text "100,0000 mm" (at 261.2 64.045) (layer "Dwgs.User")
+    (gr_text "100.0000 mm" (at 261.2 64.045) (layer "Dwgs.User")
       (effects (font (size 1.5 1.5) (thickness 0.3)))
     )
@@
     (pts (xy 211.2 78.345) (xy 111.2 78.345))
     (height 7.35)
-    (gr_text "100,0000 mm" (at 161.2 69.845) (layer "Dwgs.User")
+    (gr_text "100.0000 mm" (at 161.2 69.845) (layer "Dwgs.User")
       (effects (font (size 1 1) (thickness 0.15)))
     )
@@
     (pts (xy 231.2 153.345) (xy 211.2 153.345))
     (height -16)
-    (gr_text "20,0000 mm" (at 220.2 173.705355) (layer "Dwgs.User")
+    (gr_text "20.0000 mm" (at 220.2 173.705355) (layer "Dwgs.User")
       (effects (font (size 1.5 1.5) (thickness 0.3)))
     )
@@
     (pts (xy 311.25 153.295) (xy 311.2 78.245))
     (height 11.595253)
-    (gr_text "75,0500 mm" (at 324.62025 115.761076 -89.96182827) (layer "Dwgs.User")
+    (gr_text "75.0500 mm" (at 324.62025 115.761076 -89.96182827) (layer "Dwgs.User")
       (effects (font (size 1.5 1.5) (thickness 0.3)))
     )

Commit message: save
Parts:
- removed the C6 at (139.0, 89.0)
- removed the C6 at (182.0, 142.0)
- removed the C6 at (139.0, 142.0)
- removed the C6 at (182.0, 89.0)
- removed J5: 5V, digikey-footprints:1210
- removed Q1: Q_NPN_BCE, ESP32-footprints-Lib:Dpak
- removed REF** (x4): Diode_DO-35_P10mm, digikey-footprints:Diode_DO-35_P10mm
- added IC1: MAX4173H, Package_SO:SO-8_3.9x4.9mm_P1.27mm, F.Cu at (189.3, 140.8)
- moved J1 100.2 mm to (151.8, 137.6), turned to 90 degrees
- moved D20 99.3 mm to (195.2, 124.1)
- moved J7 78.6 mm to (236.9, 131.5)
- moved R9 72.5 mm to (220.0, 129.9)
- moved C4 71.9 mm to (182.6, 132.6)
- moved J6 70.9 mm to (236.9, 113.5), turned to 90 degrees
- moved Q4 68.6 mm to (166.2, 139.1)
- moved C6 68.2 mm to (231.7, 123.4), turned to 180 degrees
- moved C1 67.8 mm to (195.1, 142.0), turned to 90 degrees
- moved R5 67.5 mm to (177.0, 152.1)
- moved C7 67.4 mm to (219.2, 134.3)
- moved C2 65.6 mm to (204.0, 141.1)
- moved R10 65.6 mm to (219.2, 132.3)
- moved R6 65.5 mm to (209.2, 163.8)
- moved J4 65.5 mm to (219.4, 158.3)
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- renumbered D2 to D20
Routing:
- net Bat+: track 0.00 -> 50.0 mm
- net Net-(D20-K): track 0.00 -> 43.7 mm
- net +12V: track 0.00 -> 23.4 mm
- net U_Sol: track 34.1 -> 11.3 mm
- net Net-(Q4-G): track 32.3 -> 13.7 mm
- net +3V3: track 7.15 -> 22.5 mm
- net I_Sol: track 21.8 -> 36.5 mm
- net U_Bat: track 15.5 -> 6.83 mm
- net Net-(IC1-RS+): track 8.51 -> 3.50 mm
- net Net-(J4-Pin_10): track 0.00 -> 4.17 mm
- net GND: track 0.00 -> 3.72 mm
- net PWM: track 71.2 -> 74.1 mm
- net Net-(D1-A): track 3.30 -> 1.93 mm
Other:
- board size 200 x 97.5 mm -> 93.6 x 97.5 mm
