File: TeslaCoil/Tesla_Coil.kicad_sch (KiCad schematic)
At the start: 21 parts, among them J1 GPIOs, Q1 Q_NPN_BCE, Q2 Q_NPN_BCE, Q3 Q_NPN_BCE, Q4 Q_PNP_BCE, Q5 Q_PNP_BEC, Q6 Q_PNP_BEC, Q7 Q_PNP_BEC

Commit message: save
Parts:
- removed BT1: 3.3v, symbol Device:Battery_Cell
- removed J1: GPIOs, Connector_PinHeader_2.54mm:PinHeader_1x04_P2.54mm_Vertical_SMD_Pin1Left, symbol Header:header4
- added C1, C2, C3, C7: 0.1uF, digikey-footprints:0603, symbol solar-rescue:C-Device
- added C4: 100uF, ESP32-footprints-Lib:Cpol-6.3x7.7, symbol solar-rescue:CP-Device
- added C5: 1nF, digikey-footprints:0603, symbol Device:C
- added C6: 220uF, ESP32-footprints-Lib:Cpol-6.3x7.7, symbol solar-rescue:CP-Device
- added D1: COMMS, digikey-footprints:0603, symbol solar-rescue:LED-Device
- added D2: D_Schottky, digikey-footprints:DO-214AC, symbol Device:D_Schottky
- added IC1: MAX4173H, symbol connectors:MAX4173H
- added J1: SOLAR_INPUT, digikey-footprints:1210, symbol connectors:SOLAR_INPUT
- added J2: SOLAR_OUTPUT, digikey-footprints:1210, symbol connectors:SOLAR_INPUT
- added J3: Left, ESP32-footprints-Lib:PIN16, symbol solar-rescue:Conn_01x16_Female-Connector
- added J4: Right, ESP32-footprints-Lib:PIN16, symbol solar-rescue:Conn_01x16_Female-Connector
- added J5: 5V, digikey-footprints:1210, symbol Connector:Conn_01x02_Female
- added J6: BATTERY_INPUT, digikey-footprints:1210, symbol solar-rescue:Conn_01x02_Male-Connector
- added J7: BATTERY_OUTPUT, digikey-footprints:1210, symbol connectors:Battery_Output
- added L3: 33uH, ESP32-footprints-Lib:7447779139, symbol solar-rescue:L-Device
- added Q4: IRFIZ44N, digikey-footprints:SOT-223, symbol irfiz44n:IRFIZ44N
- added R1, R4, R9: 10k, digikey-footprints:0603, symbol solar-rescue:R-Device
- added R10, R2, R6: 560R, digikey-footprints:0603, symbol solar-rescue:R-Device
- added R3: 0.005R, digikey-footprints:0603, symbol solar-rescue:R-Device
- added R5: 100R, digikey-footprints:0603, symbol Device:R
- added R7: 220R, digikey-footprints:0603, symbol solar-rescue:R-Device
- added R8: 4K7, Resistors_SMD:R_0805_HandSoldering, symbol solar-rescue:R-Device
- added RX1: GPIO, ESP32-footprints-Lib:PIN2, symbol solar-rescue:Conn_01x02_Male-Connector
- added RX2: Receive, Connectors_JST:JST_PH_S2B-PH-K_02x2.00mm_Angled, symbol solar-rescue:Conn_01x02_Male-Connector
- added TX1: Transmit, Connectors_JST:JST_PH_S2B-PH-K_02x2.00mm_Angled, symbol solar-rescue:Conn_01x02_Male-Connector
- added U1: HMHA2801, Housings_SSOP:SOP-4_4.4x2.8mm_Pitch1.27mm, symbol solar-rescue:PC817-Isolator
- added U?: MAX5424, digikey-footprints:TDFN-8-1EP, symbol Device:MAX5424
- renumbered AE3 to AE1, C4 to C8, C1 to C9, D1 to D3, L6 to L4, L1 to L5, L2 to L6, Q4 to Q5, Q5 to Q6, Q6 to Q7, Q1 to Q8, Q7 to Q9, R1 to R11
Connections:
- net VDD is gone; now on net GND: L1.1
- net +12V: now also C4.1, IC1.6 (RS-), J2.1 (Sol+), Q4.2 (D), R3.2
- net +5V: now also J3.16 (Pin_16), J5.2 (Pin_2)
- net 12v: now also J3.11 (Pin_11)
- net 3.3v: now also J3.9 (Pin_9)
- net 5v: now also J3.10 (Pin_10)
- net GND: now also L1.4, C1.2, C2.2, C3.2, C4.2, C5.1, C6.2, C7.2, D1.1 (K), D2.2 (A), IC1.3 (GND), J1.2 (Sol-), J2.2 (Sol-), J3.15 (Pin_15), J4.2 (Pin_2), J5.1 (Pin_1), J6.2 (Pin_2), J7.2 (Bat-), R10.1, R2.1, R4.2, R8.1, RX1.2 (Pin_2), U1.2
- net PWM: now also J4.15 (Pin_15), R5.2
- net Bat+: now reaches Q1.3 (E)
- net Bat+: now also C6.1, J6.1 (Pin_1), J7.1 (Bat+), L3.2, R9.2
- new net: C5.2, Q4.1 (G), R4.1, R5.1
- new net: D2.1 (K), L3.1, Q4.3 (S)
- new net: IC1.8 (RS+), J1.1 (Sol+), R1.2, R3.1
- new net: D1.2 (A), R6.1
- new net: J4.5 (Pin_5), R6.2
- new net: R7.1, U1.1
- new net: TX1.1 (Pin_1), U1.3
- new net: TX1.2 (Pin_2), U1.4
- new net: J4.12 (Pin_12), R8.2, RX2.1 (Pin_1)
- new net: J4.10 (Pin_10), RX1.1 (Pin_1)
- new net: J4.13 (Pin_13), R7.2
- new net +3V3: C1.1, IC1.1 (VCC), J4.1 (Pin_1), RX2.2 (Pin_2)
- new net I_Sol: C2.1, IC1.4 (OUT), J3.6 (Pin_6)
- new net U_Bat: C7.1, J3.8 (Pin_8), R10.2, R9.1
- new net U_Sol: C3.1, J3.5 (Pin_5), R1.1, R2.2
- no-connect marks 0 -> 3
Other:
- note added: "ESP32"
- note added: "Sensor like https://www.dfrobot.com/product-580.html (work in progress)"
- note added: "Solar Input between 7-12V"
- note added: "Step Down DC to DC Converter"
- note added: "Step Motor"
- moved on the sheet: AE1, C8, C9, D3, L1, L2, L4, L5, L6, LS1, Q1, Q2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

Commit message: save
Other:
- moved on the sheet: J5, L1, L2, Q1, Q2, Q3

Commit message: save
Parts:
- removed D2: D_Schottky, digikey-footprints:DO-214AC, symbol Device:D_Schottky
- removed D3: D, symbol Device:D
- removed J5: 5V, digikey-footprints:1210, symbol Connector:Conn_01x02_Female
- removed L1: 33:50, symbol Device:L_Coupled
- removed L2: 5:12, symbol Device:L_Coupled
- removed L4: L, symbol Device:L
- removed L5: 2L, symbol Device:L
- removed L6: 300L, symbol Device:L
- removed Q1: Q_NPN_BCE, ESP32-footprints-Lib:Dpak, symbol Device:Q_NPN_BCE
- removed Q3: Q_NPN_BCE, symbol Device:Q_NPN_BCE
- added C22, C23, C24, C25, C26, C27: 47uF, symbol Device:C
- added D14, D15, D16, D17, D18, D19: D_Bridge_+-AA, symbol Device:D_Bridge_+-AA
- added D20: D, symbol Device:D
- added D22: LED, symbol Device:LED
- added L21, L23: 33:50, symbol Device:L_Coupled
- added L22, L25: 5:12, symbol Device:L_Coupled
- added L24, L26: 11:40, symbol Device:L_Coupled
- added Q25: IRLU3110Z, symbol Device:Q_NPN_BCE
- added Q26: Q_NPN_BCE, symbol Device:Q_NPN_BCE
- added R19: 2k, symbol Device:R
- added R20, R21, R22: 10k, symbol Device:R
- added T2: 2:300, symbol Device:Transformer_1P_1S
- C8: value C -> 1uF
- IC1: footprint (none) -> Package_SO:SO-8_3.9x4.9mm_P1.27mm
- Q2, Q8: value Q_NPN_BCE -> BD535
- Q5: value Q_PNP_BCE -> BC547
Connections:
- net +12V: now also C26.1, C27.1, D15.1 (+), D17.1 (+), L26.2, R20.1
- net +5V: now also C23.1, C25.1, D16.1 (+), D18.1 (+), L22.2, L24.2, R21.1, R22.1
- net 12V: now also T2.1 (AA)
- net 5v: no longer Q2.1 (B)
- net GND: now also C23.2, C25.2, D16.2 (-), D18.2 (-), D20.2 (A), D22.2 (A), L21.1
- net Vcc: now also R19.1
- net switch: now reaches L3.1, Q4.3 (S)
- net switch: now also D20.1 (K)
- net at Q8.1 (B), R11.2: now also D22.1 (K), T2.3 (SA)
- net at Q8.2 (C): now also T2.2 (AB)
- net at AE1.1 (A): now also T2.4 (SB)
- net at C8.1, Q5.2 (C): now also R19.2
- net at Q2.2 (C): now also L26.1
- net at Q2.3 (E): now also L25.2
- new net: D19.3, L26.3
- new net: D19.4, L26.4
- new net: D14.3, L21.3
- new net: D14.4, L21.4
- new net: D18.3, L25.3
- new net: D18.4, L25.4
- new net: Q26.1 (B), R21.2
- new net: L22.1, Q26.2 (C)
- new net: L21.2, Q26.3 (E)
- new net: Q25.1 (B), R22.2
- new net: Q2.1 (B), R20.2
- new net: L23.2, Q25.3 (E)
- new net: D16.3, L23.3
- new net: D16.4, L23.4
- new net: L24.1, Q25.2 (C)
- new net: D15.3, L22.3
- new net: D15.4, L22.4
- new net: D17.3, L24.3
- new net: D17.4, L24.4
- new net +3.3V: C22.2, C24.1, D14.1 (+), D19.2 (-)
- new net AGND: C22.1, C24.2, D14.2 (-), D19.1 (+), L23.1
- new net DGND: C26.2, C27.2, D15.2 (-), D17.2 (-), L25.1
Other:
- moved on the sheet: C8, J1, Q8, R11
