File: TeslaCoil/file61A703D7.kicad_sch (KiCad schematic)
At the start: 23 parts, among them Q2 Q_NPN_BCE, Q3 Q_NPN_BCE, Q8 Q_NPN_BCE, Q9 Q_NPN_BCE, T1 Transformer_1P_2S

Commit message: save
Parts:
- renumbered AE1 to AE2, AE2 to AE3, C5 to C10, C6 to C11, C2 to C12, C3 to C13, D3 to D4, D2 to D5, D4 to D6, D5 to D7, L9 to L10, L4 to L7, L3 to L8, L5 to L9, Q2 to Q10, Q3 to Q11, Q8 to Q12, Q9 to Q13, R3 to R12, R2 to R13, R4 to R14, R5 to R15
Changed lines of the file:
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@@
   (symbol (lib_id "Device:R") (at 95.25 63.5 90) (unit 1)
     (in_bom yes) (on_board yes)
-    (property "Reference" "R3" (id 0) (at 95.25 58.2422 90))
+    (property "Reference" "R12" (id 0) (at 95.25 58.2422 90))
     (property "Value" "220R" (id 1) (at 95.25 60.5536 90))
     (property "Footprint" "" (id 2) (at 95.25 65.278 90)
@@
   (symbol (lib_id "Device:C") (at 191.77 80.01 0) (unit 1)
     (in_bom yes) (on_board yes)
-    (property "Reference" "C2" (id 0) (at 194.691 78.8416 0)
+    (property "Reference" "C12" (id 0) (at 194.691 78.8416 0)
       (effects (font (size 1.27 1.27)) (justify left))
     )
@@
   (symbol (lib_id "Device:L") (at 191.77 53.34 0) (unit 1)
     (in_bom yes) (on_board yes)
-    (property "Reference" "L4" (id 0) (at 193.1162 52.1716 0)
+    (property "Reference" "L7" (id 0) (at 193.1162 52.1716 0)
       (effects (font (size 1.27 1.27)) (justify left))
     )
@@
   (symbol (lib_id "Device:Q_NPN_BCE") (at 153.67 73.66 0) (unit 1)
     (in_bom yes) (on_board yes)
-    (property "Reference" "Q2" (id 0) (at 158.5214 72.4916 0)
+    (property "Reference" "Q10" (id 0) (at 158.5214 72.4916 0)
       (effects (font (size 1.27 1.27)) (justify left))
     )
@@
   (symbol (lib_id "Device:D") (at 121.92 63.5 180) (unit 1)
     (in_bom yes) (on_board yes)
-    (property "Reference" "D3" (id 0) (at 121.92 68.9864 0))
+    (property "Reference" "D4" (id 0) (at 121.92 68.9864 0))
     (property "Value" "D" (id 1) (at 121.92 66.675 0))
     (property "Footprint" "" (id 2) (at 121.92 63.5 0)
@@
   (symbol (lib_id "Device:R") (at 95.25 96.52 90) (unit 1)
     (in_bom yes) (on_board yes)
-    (property "Reference" "R2" (id 0) (at 95.25 91.2622 90))
+    (property "Reference" "R13" (id 0) (at 95.25 91.2622 90))
     (property "Value" "220R" (id 1) (at 95.25 93.5736 90))
     (property "Footprint" "" (id 2) (at 95.25 98.298 90)
@@
   (symbol (lib_id "Device:C") (at 207.01 80.01 0) (unit 1)
     (in_bom yes) (on_board yes)
-    (property "Reference" "C3" (id 0) (at 209.931 78.8416 0)
+    (property "Reference" "C13" (id 0) (at 209.931 78.8416 0)
       (effects (font (size 1.27 1.27)) (justify left))
     )
@@
   (symbol (lib_id "Device:L") (at 191.77 115.57 0) (unit 1)
     (in_bom yes) (on_board yes)
-    (property "Reference" "L3" (id 0) (at 193.1162 114.4016 0)
+    (property "Reference" "L8" (id 0) (at 193.1162 114.4016 0)
       (effects (font (size 1.27 1.27)) (justify left))
     )
@@
   (symbol (lib_id "Device:Q_NPN_BCE") (at 153.67 106.68 0) (unit 1)
     (in_bom yes) (on_board yes)
-    (property "Reference" "Q3" (id 0) (at 158.5214 105.5116 0)
+    (property "Reference" "Q11" (id 0) (at 158.5214 105.5116 0)
       (effects (font (size 1.27 1.27)) (justify left))
     )
@@
   (symbol (lib_id "Device:D") (at 121.92 96.52 180) (unit 1)
     (in_bom yes) (on_board yes)
-    (property "Reference" "D2" (id 0) (at 121.92 102.0064 0))
+    (property "Reference" "D5" (id 0) (at 121.92 102.0064 0))
     (property "Value" "D" (id 1) (at 121.92 99.695 0))
     (property "Footprint" "" (id 2) (at 121.92 96.52 0)
@@
   (symbol (lib_id "Device:L") (at 222.25 80.01 0) (unit 1)
     (in_bom yes) (on_board yes)
-    (property "Reference" "L5" (id 0) (at 223.5708 78.8416 0)
+    (property "Reference" "L9" (id 0) (at 223.5708 78.8416 0)
       (effects (font (size 1.27 1.27)) (justify left))
     )
@@
   (symbol (lib_id "Device:R") (at 95.25 162.56 90) (unit 1)
     (in_bom yes) (on_board yes)
-    (property "Reference" "R4" (id 0) (at 95.25 157.3022 90))
+    (property "Reference" "R14" (id 0) (at 95.25 157.3022 90))
     (property "Value" "220R" (id 1) (at 95.25 159.6136 90))
     (property "Footprint" "" (id 2) (at 95.25 164.338 90)
@@
   (symbol (lib_id "Device:C") (at 171.45 179.07 0) (unit 1)
     (in_bom yes) (on_board yes)
-    (property "Reference" "C5" (id 0) (at 174.371 177.9016 0)
+    (property "Reference" "C10" (id 0) (at 174.371 177.9016 0)
       (effects (font (size 1.27 1.27)) (justify left))
     )
@@
   (symbol (lib_id "Device:Q_NPN_BCE") (at 153.67 172.72 0) (unit 1)
     (in_bom yes) (on_board yes)
-    (property "Reference" "Q8" (id 0) (at 158.5214 171.5516 0)
+    (property "Reference" "Q12" (id 0) (at 158.5214 171.5516 0)
       (effects (font (size 1.27 1.27)) (justify left))
     )
@@
   (symbol (lib_id "Device:D") (at 121.92 162.56 180) (unit 1)
     (in_bom yes) (on_board yes)
-    (property "Reference" "D4" (id 0) (at 121.92 168.0464 0))
+    (property "Reference" "D6" (id 0) (at 121.92 168.0464 0))
     (property "Value" "D" (id 1) (at 121.92 165.735 0))
     (property "Footprint" "" (id 2) (at 121.92 162.56 0)
@@
   (symbol (lib_id "Device:R") (at 95.25 195.58 90) (unit 1)
     (in_bom yes) (on_board yes)
-    (property "Reference" "R5" (id 0) (at 95.25 190.3222 90))
+    (property "Reference" "R15" (id 0) (at 95.25 190.3222 90))
     (property "Value" "220R" (id 1) (at 95.25 192.6336 90))
     (property "Footprint" "" (id 2) (at 95.25 197.358 90)
@@
   (symbol (lib_id "Device:C") (at 186.69 179.07 0) (unit 1)
     (in_bom yes) (on_board yes)
-    (property "Reference" "C6" (id 0) (at 189.611 177.9016 0)
+    (property "Reference" "C11" (id 0) (at 189.611 177.9016 0)
       (effects (font (size 1.27 1.27)) (justify left))
     )
@@
   (symbol (lib_id "Device:Q_NPN_BCE") (at 153.67 205.74 0) (unit 1)
     (in_bom yes) (on_board yes)
-    (property "Reference" "Q9" (id 0) (at 158.5214 204.5716 0)
+    (property "Reference" "Q13" (id 0) (at 158.5214 204.5716 0)
       (effects (font (size 1.27 1.27)) (justify left))
     )
@@
   (symbol (lib_id "Device:D") (at 121.92 195.58 180) (unit 1)
     (in_bom yes) (on_board yes)
-    (property "Reference" "D5" (id 0) (at 121.92 201.0664 0))
+    (property "Reference" "D7" (id 0) (at 121.92 201.0664 0))
     (property "Value" "D" (id 1) (at 121.92 198.755 0))
     (property "Footprint" "" (id 2) (at 121.92 195.58 0)
@@
   (symbol (lib_id "Device:L") (at 240.03 179.07 90) (unit 1)
     (in_bom yes) (on_board yes)
-    (property "Reference" "L9" (id 0) (at 238.8616 177.7492 0)
+    (property "Reference" "L10" (id 0) (at 238.8616 177.7492 0)
       (effects (font (size 1.27 1.27)) (justify left))
     )
@@
   (symbol (lib_id "Device:Antenna") (at 228.6 168.91 0) (unit 1)
     (in_bom yes) (on_board yes)
-    (property "Reference" "AE1" (id 0) (at 230.632 169.1894 0)
+    (property "Reference" "AE2" (id 0) (at 230.632 169.1894 0)
       (effects (font (size 1.27 1.27)) (justify left))
     )
@@
   (symbol (lib_id "Device:Antenna") (at 228.6 189.23 180) (unit 1)
     (in_bom yes) (on_board yes)
-    (property "Reference" "AE2" (id 0) (at 230.632 186.6138 0)
+    (property "Reference" "AE3" (id 0) (at 230.632 186.6138 0)
       (effects (font (size 1.27 1.27)) (justify right))
     )

Commit message: save
Changed lines of the file:
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@@
     (stroke (width 0) (type default) (color 0 0 0 0))
   )
-  (wire (pts (xy 156.21 111.76) (xy 156.21 120.65))
+  (wire (pts (xy 156.21 111.76) (xy 156.21 119.38))
     (stroke (width 0) (type default) (color 0 0 0 0))
   )
@@
     )
   )
-  (global_label "GND" (shape input) (at 156.21 120.65 270) (fields_autoplaced)
+  (global_label "GND" (shape input) (at 156.21 119.38 270) (fields_autoplaced)
     (effects (font (size 1.27 1.27)) (justify right))
-    (property "Intersheet References" "${INTERSHEET_REFS}" (id 0) (at 0 0 0)
+    (property "Intersheet References" "${INTERSHEET_REFS}" (id 0) (at 0 -1.27 0)
       (effects (font (size 1.27 1.27)) hide)
     )

Commit message: save
Parts:
- added C19: 4.7nF, symbol Device:C
- added C20: 100pF, symbol Device:C
- added C21: 10uF (400V), symbol Device:C_Polarized
- added D21: 15V, symbol Device:D_TVS
- added D3: ZD12V, symbol Device:D_Zener
- added L1: 150, symbol Device:L
- added L2: 17, symbol Device:L
- added L27: 5.5, symbol Device:L
- added Q1: IRFP260, TO220, symbol irfiz44n:IRFIZ44N
- added R17, R18: 1k (2W), symbol Device:R
- added RV1: 10k, symbol Device:R_Potentiometer
- D4, D5, D6, D7: value D -> UF4007
- L7, L8: value 100uL -> 100uH
- Q10, Q11: value Q_NPN_BCE -> IRF540
- Q12, Q13: value Q_NPN_BCE -> IRLU3110Z
- T1: value Transformer_1P_2S -> CCFL
Connections:
- net GND: now also C19.2, C21.2, D21.1 (A1), D3.2 (A), Q1.3 (S), RV1.3
- new net: D3.1 (K), R18.2, RV1.1
- new net: C19.1, C20.2, D21.2 (A2), Q1.1 (G), R17.1
- new net: R17.2, RV1.2
- new net: L2.1, L27.2, Q1.2 (D)
- new net: C20.1, L1.2, L27.1
- new net +12V: C21.1, L2.2, R18.1
Other:
- note added: "0.5mm Wire 1.5cm diameter"
- note added: "0.6mm Wire 2.5cm diameter"
- note added: "1-1.3mm Wire 5.5cm diameter"
- note added: "2kV minimum Impulse-proof"
- note added: "Breakoutpoint (Stainless-steel)"
- moved on the sheet: L10
