File: TeslaCoil/file61A87790.kicad_sch (KiCad schematic)
At the start: 33 parts, among them Q10 Q_PNP_BCE, Q11 Q_PNP_BCE, Q12 Q_PNP_BCE, Q13 Q_PNP_BCE, Q14 Q_PNP_BCE, Q15 Q_PNP_BCE, Q16 Q_PNP_BCE, Q17 Q_PNP_BCE, Q18 Q_PNP_BCE, Q19 Q_PNP_BCE, Q20 Q_PNP_BCE

Commit message: save
Parts:
- renumbered C7 to C14, C9 to C15, C10 to C16, C8 to C17, C11 to C18, D6 to D11, D8 to D12, D11 to D13, D7 to D8, L7 to L11, L8 to L12, L11 to L13, L10 to L14, L14 to L15, L12 to L16, L16 to L18, L13 to L19, L15 to L20, Q17 to Q14, Q11 to Q15, Q10 to Q16, Q18 to Q17, Q14 to Q18, Q15 to Q21, Q12 to Q22, Q13 to Q23, Q16 to Q24, R6 to R16
Connections:
- net +12V renamed ~12V
- net +19V renamed ~19V
Other:
- moved on the sheet: D13, D8, D9, L18

Commit message: save
Parts:
- C14, C15, C16, C17, C18: value C -> 47uF
- D10, D11, D12, D13, D8, D9: value D -> 1N5819
- L11: value L_Core_Iron_Coupled -> EMF
- L13: value L_Core_Ferrite_Coupled -> EMF
- L15, L18, L19, L20: value L -> 100uH
- Q15: value Q_PNP_BCE -> BC637
- Q16, Q21, Q22, Q24: value Q_PNP_BCE -> IRF9540
- Q18, Q23: value Q_PNP_BCE -> IRLZ44ZN
Other:
- note added: "Fly Back"
- note added: "Joule Thief"
- note added: "Step Down"
- note added: "Step Up"
- note added: "Step Up and Step Down"
- note added: "Transformers"
- moved on the sheet: C17, C18, D11, D12, D13, L11, L19, L20, Q15, Q22, Q23, Q24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
