File: minikame/minikame.kicad_pcb (KiCad board)
At the start: 2 copper layers, 48.8 x 40.1 mm, 13 parts, among them J1 Conn_01x08_Female, J1 Header, J1 header3, J6 ESP32

Commit message: updated: miniKame
Connections:
- J1 pad 3: Net-(J1-Pad3) -> (no net)
Routing:
- net Net-(J1-Pad3): track 58.5 -> 52.0 mm
- net (no net): track 552.9 -> 555.3 mm
- net 5V: track 105.4 -> 104.7 mm

Commit message: update
Parts:
- added J2: Camera, Connector_PinSocket_2.54mm:PinSocket_2x09_P2.54mm_Vertical, F.Cu at (124.2, 119.4)
- added R1: 4k7, Resistor_SMD:R_0603_1608Metric, F.Cu at (164.3, 100.6)
- added R2: 4k7, Resistor_SMD:R_0603_1608Metric, F.Cu at (149.7, 116.5)
- J1: value header3 -> PWM
- J10: renamed from J1; value Header -> C
- J11: renamed from J1; value Header -> A
- J12: renamed from J1; value Header -> D
- J13: renamed from J1; value Header -> B
- J4: renamed from J5; value (none) -> ESP32
- J5: renamed from J1; value Conn_01x08_Female -> GND
- J6: renamed from J1; value Conn_01x08_Female -> Vcc
- J7: renamed from J1; value Header -> UART
- J8: renamed from J1; value Header -> I2C
- J9: renamed from J1; value Header -> Motor
- moved J10 3.29 mm to (129.3, 113.8)
- moved J11 3.29 mm to (129.3, 103.6)
- moved J13 3.29 mm to (136.9, 103.6)
- moved J12 3.27 mm to (136.9, 113.8)
- renumbered J6 to J3
Connections:
- net Net-(J1-Pad3) renamed G23
- J1 pad 1: (no net) -> G13
- J1 pad 2: (no net) -> G27
- J1 pad 3: (no net) -> G26
- J1 pad 4: (no net) -> G25
- J1 pad 5: (no net) -> G4
- J1 pad 6: (no net) -> G18
- J1 pad 7: (no net) -> G19
- J10 pad 1: 5V -> 3.3v
- J10 pad 2: (no net) -> G25
- J10 pad 3: (no net) -> Net-(J10-Pad3)
- J11 pad 2: (no net) -> Net-(J11-Pad2)
- J11 pad 3: (no net) -> G27
- J11 pad 4: (no net) -> G13
- J12 pad 1: (no net) -> G4
- J12 pad 2: (no net) -> G19
- J12 pad 3: (no net) -> Net-(J12-Pad3)
- J13 pad 2: (no net) -> Net-(J13-Pad2)
- J3 pad 1: 5V -> 3.3v
- J3 pad 10: (no net) -> G19
- J3 pad 11: (no net) -> SDA
- J3 pad 12: (no net) -> Rx
- J3 pad 13: (no net) -> Tx
- J3 pad 14: (no net) -> SCL
- J3 pad 3: (no net) -> D3
- J3 pad 4: (no net) -> D7
- J3 pad 5: (no net) -> G4
- J3 pad 6: (no net) -> D2
- J3 pad 7: (no net) -> D1
- J3 pad 8: (no net) -> D5
- J3 pad 9: (no net) -> G18
- J4 pad 10: (no net) -> X
- J4 pad 11: (no net) -> H
- J4 pad 12: (no net) -> V
- J4 pad 13: (no net) -> D0
- J4 pad 14: (no net) -> unconnected-(J4-Pad14)
- J4 pad 15: (no net) -> RST
- J4 pad 3: (no net) -> G13
- J4 pad 4: (no net) -> D6
- J4 pad 5: (no net) -> D4
- J4 pad 6: (no net) -> G27
- J4 pad 7: (no net) -> G26
- J4 pad 8: (no net) -> G25
- J4 pad 9: (no net) -> P
- J7 pad 1: (no net) -> Rx
- J7 pad 2: (no net) -> Tx
- J7 pad 4: 5V -> 3.3v
- J8 pad 1: (no net) -> SDA
- J8 pad 2: (no net) -> SCL
- J8 pad 4: 5V -> 3.3v
- J9 pad 1: (no net) -> Net-(J11-Pad2)
- J9 pad 2: (no net) -> Net-(J10-Pad3)
- J9 pad 3: (no net) -> Net-(J13-Pad2)
- J9 pad 4: (no net) -> Net-(J12-Pad3)
Routing:
- net (no net): track 555.3 -> 0.00 mm, vias 4 -> 0
- net SCL: track 0.00 -> 81.1 mm, vias 0 -> 1
- net SDA: track 0.00 -> 72.4 mm, vias 0 -> 1
- net 3.3v: track 0.00 -> 70.5 mm, vias 0 -> 2
- net V: track 0.00 -> 69.4 mm, vias 0 -> 1
- net H: track 0.00 -> 66.0 mm
- net RST: track 0.00 -> 64.0 mm
- net 5V: track 104.7 -> 48.4 mm
- net Net-(J10-Pad3): track 0.00 -> 50.8 mm
- net X: track 0.00 -> 49.9 mm
- net Net-(J12-Pad3): track 0.00 -> 46.5 mm
- net G19: track 0.00 -> 43.8 mm
- net P: track 0.00 -> 41.9 mm
- net Net-(J11-Pad2): track 0.00 -> 40.8 mm
- net Net-(J13-Pad2): track 0.00 -> 40.5 mm
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Other:
- board text added: "v2.3"
- board text removed: "v2.0"

Commit message: save
Routing:
- net H: track 66.0 -> 69.9 mm
Changed lines of the file:
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@@
   (segment (start 122.88 115.65) (end 122.3745 115.65) (width 0.25) (layer "F.Cu") (net 7))
   (via (at 122.3745 115.65) (size 0.8) (drill 0.4) (layers "F.Cu" "B.Cu") (net 7))
-  (segment (start 152.134 87.6264) (end 152.134 96.516) (width 0.25) (layer "B.Cu") (net 7))
-  (segment (start 129.698879 85.093969) (end 149.601569 85.093969) (width 0.25) (layer "B.Cu") (net 7))
-  (segment (start 121.15096 114.42646) (end 121.15096 93.641887) (width 0.25) (layer "B.Cu") (net 7))
-  (segment (start 149.601569 85.093969) (end 152.134 87.6264) (width 0.25) (layer "B.Cu") (net 7))
-  (segment (start 122.3745 115.65) (end 121.15096 114.42646) (width 0.25) (layer "B.Cu") (net 7))
-  (segment (start 121.15096 93.641887) (end 129.698879 85.093969) (width 0.25) (layer "B.Cu") (net 7))
-  (segment (start 149.594 96.516) (end 145.60052 92.52252) (width 0.25) (layer "B.Cu") (net 8))
-  (segment (start 125.575489 115.494511) (end 126.75 114.32) (width 0.25) (layer "B.Cu") (net 8))
-  (segment (start 130.106511 85.543489) (end 130.1 85.55) (width 0.25) (layer "B.Cu") (net 8))
-  (segment (start 145.60052 92.52252) (end 145.60052 86.17292) (width 0.25) (layer "B.Cu") (net 8))
-  (segment (start 130.1 85.55) (end 129.878565 85.55) (width 0.25) (layer "B.Cu") (net 8))
-  (segment (start 121.60048 93.828085) (end 121.60048 113.80048) (width 0.25) (layer "B.Cu") (net 8))
-  (segment (start 144.971089 85.543489) (end 130.106511 85.543489) (width 0.25) (layer "B.Cu") (net 8))
-  (segment (start 123.294511 115.494511) (end 125.575489 115.494511) (width 0.25) (layer "B.Cu") (net 8))
-  (segment (start 121.60048 113.80048) (end 123.294511 115.494511) (width 0.25) (layer "B.Cu") (net 8))
-  (segment (start 145.60052 86.17292) (end 144.971089 85.543489) (width 0.25) (layer "B.Cu") (net 8))
-  (segment (start 129.878565 85.55) (end 121.60048 93.828085) (width 0.25) (layer "B.Cu") (net 8))
+  (segment (start 150.237287 85.093969) (end 129.698879 85.093969) (width 0.25) (layer "B.Cu") (net 7))
+  (segment (start 121.15096 114.42646) (end 122.3745 115.65) (width 0.25) (layer "B.Cu") (net 7))
+  (segment (start 129.698879 85.093969) (end 121.15096 93.641887) (width 0.25) (layer "B.Cu") (net 7))
+  (segment (start 121.15096 93.641887) (end 121.15096 114.42646) (width 0.25) (layer "B.Cu") (net 7))
+  (segment (start 152.134 96.516) (end 152.134 86.990682) (width 0.25) (layer "B.Cu") (net 7))
+  (segment (start 152.134 86.990682) (end 150.237287 85.093969) (width 0.25) (layer "B.Cu") (net 7))
+  (segment (start 129.878565 85.55) (end 130.1 85.55) (width 0.25) (layer "B.Cu") (net 8))
+  (segment (start 150.051089 85.543489) (end 150.68052 86.17292) (width 0.25) (layer "B.Cu") (net 8))
+  (segment (start 150.68052 95.42948) (end 149.594 96.516) (width 0.25) (layer "B.Cu") (net 8))
+  (segment (start 130.106511 85.543489) (end 150.051089 85.543489) (width 0.25) (layer "B.Cu") (net 8))
+  (segment (start 130.1 85.55) (end 130.106511 85.543489) (width 0.25) (layer "B.Cu") (net 8))
+  (segment (start 125.575489 115.494511) (end 123.294511 115.494511) (width 0.25) (layer "B.Cu") (net 8))
+  (segment (start 126.75 114.32) (end 125.575489 115.494511) (width 0.25) (layer "B.Cu") (net 8))
+  (segment (start 121.60048 113.80048) (end 121.60048 93.828085) (width 0.25) (layer "B.Cu") (net 8))
+  (segment (start 150.68052 86.17292) (end 150.68052 95.42948) (width 0.25) (layer "B.Cu") (net 8))
+  (segment (start 123.294511 115.494511) (end 121.60048 113.80048) (width 0.25) (layer "B.Cu") (net 8))
+  (segment (start 121.60048 93.828085) (end 129.878565 85.55) (width 0.25) (layer "B.Cu") (net 8))
   (segment (start 141.998 94) (end 122.7 94) (width 0.25) (layer "B.Cu") (net 9))
   (segment (start 122.7 94) (end 122.55 94.15) (width 0.25) (layer "B.Cu") (net 9))
