File: Drone/Crazyflie contol board.kicad_pcb (KiCad board)
At the start: 4 copper layers, 40 x 40 mm, 72 parts, among them J1 Aux, P1 CONN_2, P2 CONN_2, P3 CONN_2, P4 CONN_2, P7 MICRO-B-USB, P9 CONN_1, Q1 PMV31XN, Q2 PMV31XN, Q3 PMV31XN, Q4 PMV31XN, Q7 SS8050-G, Q8 SS8050-G, SW2 BOOT, U1 BMX160, U11 ESP32-WROOM, U12 CP2102N-A01-GQFN24, U5 MS5611-01BA03, U6 NUF2221, U7 TPS79301, U9 TPS79301

Commit message: finished
Routing:
- net /I2C_SCK: track 53.0 -> 62.5 mm
- net /I2C_SCL: track 57.1 -> 64.6 mm
- net /USBD+: track 18.7 -> 12.8 mm
Other:
- board text added: "Rev. 2.3"
- board text removed: "Rev. 2.2"
Changed lines of the file:
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@@
     (effects (font (size 0.8001 0.8001) (thickness 0.200025)))
   )
-  (gr_text "Rev. 2.2" (at 158.1 103.85 270) (layer "B.Cu")
+  (gr_text "Rev. 2.3" (at 158.1 103.85 270) (layer "B.Cu")
     (effects (font (size 0.8001 0.8001) (thickness 0.200025) italic) (justify mirror))
   )
@@
   (segment (start 133.2992 90.7034) (end 135.001 90.7034) (width 0.2032) (layer "F.Cu") (net 32))
   (segment (start 136.00176 91.70162) (end 136.05002 91.65336) (width 0.2032) (layer "F.Cu") (net 32))
+  (segment (start 154.674389 120.524389) (end 147.274389 120.524389) (width 0.1524) (layer "F.Cu") (net 32))
   (segment (start 135.98398 91.7194) (end 135.98398 94.33814) (width 0.2032) (layer "F.Cu") (net 32))
-  (segment (start 147.53062 122.68062) (end 143.8 118.95) (width 0.1524) (layer "F.Cu") (net 32))
   (segment (start 132.05968 90.27922) (end 131.47802 90.27922) (width 0.2032) (layer "F.Cu") (net 32))
   (segment (start 130.70078 89.50198) (end 130.70078 88.5063) (width 0.2032) (layer "F.Cu") (net 32))
+  (segment (start 147.274389 120.524389) (end 138.18616 111.43616) (width 0.1524) (layer "F.Cu") (net 32))
   (segment (start 132.05968 90.27922) (end 132.87502 90.27922) (width 0.2032) (layer "F.Cu") (net 32))
+  (segment (start 154.674389 120.524389) (end 154.911889 120.524389) (width 0.1524) (layer "F.Cu") (net 32))
   (segment (start 136.05002 91.65336) (end 137.57656 91.65336) (width 0.2032) (layer "F.Cu") (net 32))
   (segment (start 137.72992 91.5) (end 139.075 91.5) (width 0.2032) (layer "F.Cu") (net 32))
@@
   (segment (start 132.87502 90.27922) (end 133.2992 90.7034) (width 0.2032) (layer "F.Cu") (net 32))
   (segment (start 129.99974 87.80526) (end 129.99974 87.16518) (width 0.2032) (layer "F.Cu") (net 32))
+  (segment (start 154.911889 120.524389) (end 155.99 121.6025) (width 0.1524) (layer "F.Cu") (net 32))
+  (segment (start 138.18616 111.43616) (end 138.18616 109.855) (width 0.1524) (layer "F.Cu") (net 32))
   (segment (start 135.98398 94.33814) (end 139.1285 97.48266) (width 0.2032) (layer "F.Cu") (net 32))
   (segment (start 135.001 90.7034) (end 136.00176 91.70416) (width 0.2032) (layer "F.Cu") (net 32))
-  (segment (start 154.91188 122.68062) (end 147.53062 122.68062) (width 0.1524) (layer "F.Cu") (net 32))
-  (segment (start 155.99 121.6025) (end 154.91188 122.68062) (width 0.1524) (layer "F.Cu") (net 32))
   (segment (start 131.47802 90.27922) (end 130.70078 89.50198) (width 0.2032) (layer "F.Cu") (net 32))
   (via (at 139.15644 97.55124) (size 0.635) (drill 0.381) (layers "F.Cu" "B.Cu") (net 32))
@@
   (segment (start 141.08 113.2) (end 139.6268 113.2) (width 0.2032) (layer "B.Cu") (net 32))
   (segment (start 137.6 112.989124) (end 137.6 110.44116) (width 0.2032) (layer "B.Cu") (net 32))
+  (segment (start 144.704817 122.68062) (end 157.45188 122.68062) (width 0.1524) (layer "F.Cu") (net 33))
   (segment (start 133.55 90.022182) (end 133.527302 90.022182) (width 0.2032) (layer "F.Cu") (net 33))
   (segment (start 132.04952 88.45296) (end 131.50088 87.90432) (width 0.2032) (layer "F.Cu") (net 33))
   (segment (start 134.02564 89.02954) (end 135.9961 91) (width 0.2032) (layer "F.Cu") (net 33))
   (segment (start 133.52954 89.02954) (end 134.02564 89.02954) (width 0.2032) (layer "F.Cu") (net 33))
-  (segment (start 158.53 121.6025) (end 157.451889 120.524389) (width 0.1524) (layer "F.Cu") (net 33))
+  (segment (start 139.065 117.040803) (end 144.704817 122.68062) (width 0.1524) (layer "F.Cu") (net 33))
   (segment (start 133.52954 89.02954) (end 133.52954 90.001722) (width 0.2032) (layer "F.Cu") (net 33))
+  (segment (start 157.45188 122.68062) (end 158.53 121.6025) (width 0.1524) (layer "F.Cu") (net 33))
   (segment (start 132.04952 89.02954) (end 133.52954 89.02954) (width 0.2032) (layer "F.Cu") (net 33))
   (segment (start 132.04952 89.02954) (end 132.04952 88.45296) (width 0.2032) (layer "F.Cu") (net 33))
   (segment (start 131.50088 87.90432) (end 131.50088 87.16518) (width 0.2032) (layer "F.Cu") (net 33))
-  (segment (start 157.451889 120.524389) (end 147.274389 120.524389) (width 0.1524) (layer "F.Cu") (net 33))
-  (segment (start 147.274389 120.524389) (end 144.95 118.2) (width 0.1524) (layer "F.Cu") (net 33))
+  (segment (start 139.065 116.84) (end 139.065 117.040803) (width 0.1524) (layer "F.Cu") (net 33))
   (segment (start 133.52954 90.001722) (end 133.55 90.022182) (width 0.2032) (layer "F.Cu") (net 33))
   (segment (start 135.9961 91) (end 139.075 91) (width 0.2032) (layer "F.Cu") (net 33))
@@
   (segment (start 125.33648 117.01) (end 125.92304 116.42344) (width 0.2032) (layer "B.Cu") (net 48))
   (segment (start 123.08 117.01) (end 125.33648 117.01) (width 0.2032) (layer "B.Cu") (net 48))
-  (segment (start 132.01904 96.42348) (end 129.949159 98.493361) (width 0.2032) (layer "F.Cu") (net 49))
-  (segment (start 129.949159 98.493361) (end 124.374895 98.493361) (width 0.2032) (layer "F.Cu") (net 49))
-  (segment (start 123.35764 97.476106) (end 123.35764 94.403612) (width 0.2032) (layer "F.Cu") (net 49))
-  (segment (start 124.374895 98.493361) (end 123.35764 97.476106) (width 0.2032) (layer "F.Cu") (net 49))
-  (via (at 132.01904 96.42348) (size 0.635) (drill 0.381) (layers "F.Cu" "B.Cu") (net 49))
-  (via (at 123.34748 94.2848) (size 0.635) (drill 0.381) (layers "F.Cu" "B.Cu") (net 49))
-  (segment (start 132.01904 94.12224) (end 131.95046 94.05366) (width 0.2032) (layer "B.Cu") (net 49))
-  (segment (start 123.360181 94.272099) (end 123.34748 94.2848) (width 0.2032) (layer "B.Cu") (net 49))
-  (segment (start 131.95046 93.25356) (end 131.95046 94.05366) (width 0.2032) (layer "B.Cu") (net 49))
-  (segment (start 125.0228 94.686788) (end 124.608111 94.272099) (width 0.2032) (layer "B.Cu") (net 49))
-  (segment (start 132.01904 96.42348) (end 132.01904 94.12224) (width 0.2032) (layer "B.Cu") (net 49))
-  (segment (start 125.0228 95.28708) (end 125.0228 94.686788) (width 0.2032) (layer "B.Cu") (net 49))
-  (segment (start 124.608111 94.272099) (end 123.360181 94.272099) (width 0.2032) (layer "B.Cu") (net 49))
+  (via (at 132.25 94.8) (size 0.635) (drill 0.381) (layers "F.Cu" "B.Cu") (net 49))
+  (via (at 124.65 93.7) (size 0.635) (drill 0.381) (layers "F.Cu" "B.Cu") (net 49))
+  (segment (start 132.25 94.291776) (end 132.25 94.8) (width 0.2032) (layer "In1.Cu") (net 49))
+  (segment (start 125.462796 92.63126) (end 130.589484 92.63126) (width 0.2032) (layer "In1.Cu") (net 49))
+  (segment (start 124.65 93.7) (end 124.65 93.444056) (width 0.2032) (layer "In1.Cu") (net 49))
+  (segment (start 130.589484 92.63126) (end 132.25 94.291776) (width 0.2032) (layer "In1.Cu") (net 49))
+  (segment (start 124.65 93.444056) (end 125.462796 92.63126) (width 0.2032) (layer "In1.Cu") (net 49))
+  (segment (start 124.608111 94.272099) (end 125.0228 94.686788) (width 0.2032) (layer "B.Cu") (net 49))
+  (segment (start 132.25 94.8) (end 132.25 94.3532) (width 0.2032) (layer "B.Cu") (net 49))
+  (segment (start 125.0228 94.686788) (end 125.0228 95.28708) (width 0.2032) (layer "B.Cu") (net 49))
+  (segment (start 131.95046 94.05366) (end 131.95046 93.25356) (width 0.2032) (layer "B.Cu") (net 49))
+  (segment (start 124.65 93.7) (end 124.608111 93.741889) (width 0.2032) (layer "B.Cu") (net 49))
+  (segment (start 124.608111 93.741889) (end 124.608111 94.272099) (width 0.2032) (layer "B.Cu") (net 49))
+  (segment (start 132.25 94.3532) (end 131.95046 94.05366) (width 0.2032) (layer "B.Cu") (net 49))
   (segment (start 127.454661 94.470219) (end 127.49784 94.42704) (width 0.2032) (layer "F.Cu") (net 50))
   (segment (start 125.36424 94.15272) (end 125.681739 94.470219) (width 0.2032) (layer "F.Cu") (net 50))
