File: Drone/Crazyflie contol board.kicad_pcb (KiCad board)
At the start: 4 copper layers, 40.1 x 38.1 mm, 98 parts, among them P1 CONN_2, P2 CONN_2, P3 CONN_2, P4 CONN_2, P7 MICRO-B-USB, P9 CONN_1, Q1 PMV31XN, Q2 PMV31XN, Q3 PMV31XN, Q4 PMV31XN, Q5 2N7002, Q6 2N7002, Q7 SS8050-G, Q8 SS8050-G, SW1 PUSH ON/OFF, SW2 BOOT, U1 BMX160, U10 MAX16054, U11 ESP32-WROOM, U12 CP2102N-A01-GQFN24, U5 MS5611-01BA03, U6 NUF2221, U7 TPS79301, U8 BQ24075, U9 TPS79301

Commit message: save
Parts:
- removed ? (x6): Fiducial_0.75mm_Dia_1.5mm_Outer, Fiducials:Fiducial_0.75mm_Dia_1.5mm_Outer
- removed C39: 10uF, SM0603_Capa
- removed C41: 100nF, SM0603_Capa
- removed D8: BLUE LED, SMDLED-0603
- removed Q5, Q6: 2N7002, SOT23GDS
- removed R21: 300k, SM0603
- removed R23: 150k, SM0603
- removed R24: 1.2k, SM0603
- removed R25, R27, R32, R33, R36, R37: 10k, SM0603
- removed R26: 1.2K, SM0603
- removed R30: 20k, SM0603
- removed R31: 100k, SM0603
- removed R38: 1k, SM0603
- removed U10: MAX16054, SOT23_6
- removed U8: BQ24075, QFN16
- added J1: Aux, Connector_IDC:IDC-Header_2x05_P2.54mm_Vertical, F.Cu at (148.4, 121.6)
- moved SW1 47.5 mm to (115.3, 115.5)
Connections:
- net /I2C_SCK_VCCA renamed /I2C_SCK
- net /I2C_SCL_VCCA renamed /I2C_SCL
- C33 pad 1: VCOM -> VBUS
- C34 pad 1: VCOM -> VBUS
- C36 pad 1: /POWER/VUSB -> VBUS
- C38 pad 1: VCOM -> VBUS
- P7 pad 1: /POWER/VUSB -> VBUS
- P7 pad 4: (no net) -> unconnected-(P7-Pad4)
- R17 pad 2: VCOM -> VBUS
- SW1 pad 2: Net-(SW1-Pad2) -> unconnected-(SW1-Pad2)
- U1 pad 9: (no net) -> unconnected-(U1-Pad9)
- U11 pad 11: (no net) -> /TDO
- U11 pad 13: (no net) -> unconnected-(U11-Pad13)
- U11 pad 14: (no net) -> unconnected-(U11-Pad14)
- U11 pad 17: (no net) -> unconnected-(U11-Pad17)
- U11 pad 18: (no net) -> unconnected-(U11-Pad18)
- U11 pad 19: (no net) -> unconnected-(U11-Pad19)
- U11 pad 20: (no net) -> unconnected-(U11-Pad20)
- U11 pad 21: (no net) -> unconnected-(U11-Pad21)
- U11 pad 22: (no net) -> unconnected-(U11-Pad22)
- U11 pad 23: (no net) -> unconnected-(U11-Pad23)
- U11 pad 29: (no net) -> unconnected-(U11-Pad29)
- U11 pad 30: /PGOOD -> /PGO
- U11 pad 32: (no net) -> unconnected-(U11-Pad32)
- U11 pad 4: (no net) -> unconnected-(U11-Pad4)
- U11 pad 5: (no net) -> unconnected-(U11-Pad5)
- U11 pad 6: (no net) -> unconnected-(U11-Pad6)
- U11 pad 7: (no net) -> unconnected-(U11-Pad7)
- U11 pad 8: /SYSOFF -> /SYS
- U12 pad 1: (no net) -> unconnected-(U12-Pad1)
- U12 pad 10: (no net) -> unconnected-(U12-Pad10)
- U12 pad 11: (no net) -> unconnected-(U12-Pad11)
- U12 pad 12: (no net) -> unconnected-(U12-Pad12)
- U12 pad 13: (no net) -> unconnected-(U12-Pad13)
- U12 pad 14: (no net) -> unconnected-(U12-Pad14)
- U12 pad 15: (no net) -> unconnected-(U12-Pad15)
- U12 pad 16: (no net) -> unconnected-(U12-Pad16)
- U12 pad 17: (no net) -> unconnected-(U12-Pad17)
- U12 pad 18: (no net) -> unconnected-(U12-Pad18)
- U12 pad 22: (no net) -> unconnected-(U12-Pad22)
- U12 pad 24: (no net) -> unconnected-(U12-Pad24)
- U12 pad 8: (no net) -> VBUS
- U5 pad 6: (no net) -> unconnected-(U5-Pad6)
- U9 pad 1: VCOM -> VBUS
- U9 pad 3: VCOM -> VBUS
Routing:
- net /PGOOD: track 51.4 -> 0.00 mm, vias 3 -> 0
- net /EN1: track 43.0 -> 0.00 mm, vias 2 -> 0
- net VBUS: track 0.00 -> 41.8 mm, vias 0 -> 6
- net /SYSOFF: track 39.0 -> 0.00 mm, vias 2 -> 0
- net /EN2: track 38.0 -> 0.00 mm, vias 3 -> 0
- net /POWER/VUSB: track 37.9 -> 0.00 mm, vias 3 -> 0
- net GND: track 51.7 -> 18.6 mm
- net VCOM: track 23.5 -> 0.00 mm, vias 6 -> 0
- net +BATT: track 48.0 -> 28.3 mm
- net /CHG: track 16.6 -> 0.00 mm, vias 1 -> 0
- net Net-(Q6-PadD): track 16.5 -> 0.00 mm, vias 1 -> 0
- net VCC: track 103.3 -> 92.7 mm
- net Net-(SW1-Pad2): track 7.39 -> 0.00 mm
- net Net-(R27-Pad2): track 5.54 -> 0.00 mm
- net Net-(R33-Pad1): track 4.74 -> 0.00 mm, vias 1 -> 0
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- added copper zone on In2.Cu, net VBUS
- removed copper zone on In2.Cu, net VCOM
Other:
- board size 40.1 x 38.1 mm -> 40 x 40 mm

Commit message: update
Parts:
- removed SW1: PUSH ON/OFF, SPST-NO-4x2.5
- moved C33 3.87 mm to (147.8, 97.3)
Connections:
- J1 pad 1: /EN2 -> /EN1
- J1 pad 2: /TDO -> /EN2
- J1 pad 3: /EN1 -> /TDO
Routing:
- net /TDO: track 0.00 -> 38.6 mm
- net /SYS: track 0.00 -> 37.1 mm
- net /EN1: track 0.00 -> 36.2 mm
- net /EN2: track 0.00 -> 36.2 mm
- net /CHG: track 0.00 -> 33.4 mm
- net /PGO: track 0.00 -> 16.6 mm
- net /I2C_SCK: track 38.9 -> 53.0 mm
- net /I2C_SCL: track 43.0 -> 57.1 mm
- net DGND: track 24.5 -> 29.9 mm, vias 10 -> 11
- net /MOTOR2: track 22.8 -> 19.2 mm
- net VBUS: track 41.8 -> 44.9 mm
- net GND: track 18.6 -> 16.5 mm, vias 8 -> 7
- net AGND: track 6.26 -> 7.29 mm
- net Net-(Q4-PadG): track 30.1 -> 29.4 mm
- net VCC: track 92.7 -> 92.2 mm, vias 14 -> 12
Other:
- board text removed: "ON/OFF"

Commit message: save
Parts:
- removed BT1: BATTERY, JST-B2B-ZR
- removed C29, C35: 15pF, SM0603_Capa
- removed C3: 100nF, ESP32-footprints-Lib:0603_new_new
- removed C30, C31, C4: 4.7uF, SM0603_Capa
- removed C32, C40: 10nF, SM0603_Capa
- removed C33: 100nF, SM0603_Capa
- removed D6: GREEN LED, SMDLED-0603
- removed P9: CONN_1, PINHEADER_127_1X1
- removed Q7, Q8: SS8050-G, digikey-footprints:SOT-23-3
- removed R10, R8: 10k, ESP32-footprints-Lib:0603_new_new
- removed R16: 39k, SM0603
- removed R18, R28: 30k, SM0603
- removed R19, R29: 0R, SM0603
- removed R20: 42.2k, SM0603
- removed R6: 220R, SM0603
- removed R7: 1k, ESP32-footprints-Lib:0603_new_new
- removed SW2: BOOT, ESP32-footprints-Lib:Switch_Tactile_SMD_B3U-1000P_new_new
- removed U12: CP2102N-A01-GQFN24, ESP32-footprints-Lib:QFN-24-1EP_4x4mm_new_new_new
- removed U7: TPS79301, SOT23_6
- moved R17 12.7 mm to (155.4, 104.6), turned to 90 degrees
Connections:
- C18 pad 2: AGND -> GND
- C20 pad 2: AGND -> GND
- C24 pad 2: AGND -> GND
- D1 pad 2: +BATT -> VBUS
- D2 pad 2: +BATT -> VBUS
- D3 pad 2: +BATT -> VBUS
- D4 pad 2: +BATT -> VBUS
- D7 pad 2: DGND -> GND
- J1 pad 1: /EN1 -> /P1
- J1 pad 2: /EN2 -> /P2
- J1 pad 3: /TDO -> /P3
- J1 pad 4: /PGO -> /TX
- J1 pad 5: /SYS -> /P4
- J1 pad 6: /CHG -> /RX
- J1 pad 7: /I2C_SCK -> /I2C_SDA
- P7 pad 5: DGND -> GND
- R13 pad 2: /I2C_SCK -> /I2C_SDA
- R17 pad 1: Net-(C31-Pad1) -> Net-(U9-EN)
- U1 pad 1: AGND -> GND
- U1 pad 14: /I2C_SCK -> /I2C_SDA
- U1 pad 2: AGND -> GND
- U1 pad 3: AGND -> GND
- U1 pad 6: AGND -> GND
- U1 pad 7: AGND -> GND
- U11 pad 13: unconnected-(U11-Pad13) -> /USBD-
- U11 pad 14: unconnected-(U11-Pad14) -> /USBD+
- U11 pad 16: /MOTOR1 -> unconnected-(U11-IO13-Pad16)
- U11 pad 24: Net-(R6-Pad1) -> unconnected-(U11-IO2-Pad24)
- U11 pad 28: /CHG -> (no net)
- U11 pad 29: unconnected-(U11-Pad29) -> /MOTOR1
- U11 pad 30: /PGO -> (no net)
- U11 pad 33: /I2C_SCK -> (no net)
- U11 pad 34: Net-(U11-Pad34) -> /RX
- U11 pad 35: Net-(U11-Pad35) -> /TX
- U11 pad 36: /I2C_SCL -> (no net)
- U11 pad 6: unconnected-(U11-Pad6) -> /I2C_SDA
- U11 pad 7: unconnected-(U11-Pad7) -> /I2C_SCL
- U5 pad 3: AGND -> GND
- U5 pad 4: AGND -> GND
- U5 pad 5: AGND -> GND
- U5 pad 7: /I2C_SCK -> /I2C_SDA
- U6 pad 2: DGND -> GND
- U9 pad 3: VBUS -> Net-(U9-EN)
- U9 pad 4: Net-(C40-Pad1) -> unconnected-(U9-NR-Pad4)
- U9 pad 5: Net-(C35-Pad2) -> unconnected-(U9-FB-Pad5)
Routing:
- net /I2C_SDA: track 0.00 -> 77.1 mm, vias 0 -> 3
- net /I2C_SCK: track 53.0 -> 0.00 mm, vias 2 -> 0
- net /TDO: track 38.6 -> 0.00 mm
- net /SYS: track 37.1 -> 0.00 mm
- net VCC: track 92.2 -> 55.2 mm
- net /EN1: track 36.2 -> 0.00 mm
- net /EN2: track 36.2 -> 0.00 mm
- net /CHG: track 33.4 -> 0.00 mm
- net Net-(U11-Pad35): track 33.2 -> 0.00 mm
- net Net-(R6-Pad1): track 32.2 -> 0.00 mm, vias 1 -> 0
- net Net-(Q7-Pad2): track 31.9 -> 0.00 mm, vias 1 -> 0
- net Net-(U11-Pad34): track 30.6 -> 0.00 mm, vias 2 -> 0
- net +BATT: track 28.1 -> 0.00 mm
- net /I2C_SCL: track 57.1 -> 80.1 mm, vias 3 -> 4
- net Net-(Q8-C): track 18.4 -> 0.00 mm, vias 1 -> 0
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- added copper zone on B.Cu, net (none)
- removed copper zone on B.Cu, net AGND
- removed copper zone on F.Cu, net AGND
- removed copper zone on In1.Cu, net AGND
Other:
- rule pad_to_mask_clearance: 0.07112 -> 0.07
- board text added: "Rev. 2.4"
- board text removed: "BOOT"
- board text removed: "Rev. 2.2"

Commit message: save
Parts:
- removed C1: 22uF, ESP32-footprints-Lib:0603_new_new
- removed C2: 100nF, ESP32-footprints-Lib:0603_new_new
- removed C38: 100nF, SM0603_Capa
- removed P1, P2, P3, P4: CONN_2, PINHEADER_127_2X1
- added J2: Motors, Connector_IDC:IDC-Header_2x05_P2.54mm_Vertical, B.Cu at (137.7, 96.1)
- C18, C20: footprint SM0603_Capa -> Capacitor_SMD:C_0603_1608Metric
- C24: footprint SM0603_Capa -> Capacitor_SMD:C_0603_1608Metric; moved to B.Cu
- C34: value 4.7uF -> 2.2uF; footprint SM0603_Capa -> Capacitor_SMD:C_0603_1608Metric
- C36: footprint SM0603_Capa -> Capacitor_SMD:C_0603_1608Metric; moved to F.Cu
- C37: value 4.7uF -> 2.2uF; footprint SM0603_Capa -> Capacitor_SMD:C_0603_1608Metric; moved to F.Cu
- C5: footprint ESP32-footprints-Lib:0603_new_new -> Capacitor_SMD:C_0603_1608Metric
- D1, D2, D3, D4: footprint sod323 -> Diode_SMD:D_SOD-323; moved to F.Cu
- J1, U5: moved to B.Cu
- P7, U11, U6, U9: moved to F.Cu
- R1, R2, R3, R4: footprint SM0603 -> Resistor_SMD:R_0402_1005Metric
- R13, R14, R22, R5: footprint SM0603 -> Resistor_SMD:R_0603_1608Metric
- R17: value 10R -> 100k; footprint SM0603 -> Resistor_SMD:R_0603_1608Metric; moved to F.Cu
- R39, R40, R41: footprint SM0402 -> Resistor_SMD:R_0402_1005Metric
- R42, R9: footprint ESP32-footprints-Lib:0603_new_new -> Resistor_SMD:R_0402_1005Metric
- moved R9 43.1 mm to (164.9, 112.9)
- moved C5 42.2 mm to (164.9, 116.1), turned to 90 degrees
- moved D5 38.9 mm to (163.5, 85.7), turned to -45 degrees
- moved R5 37.2 mm to (163.4, 89.7), turned to 90 degrees
- moved C36 28.2 mm to (157.0, 93.2), turned to 180 degrees
- moved D7 27.8 mm to (127.8, 114.8), turned to -90 degrees
- moved P7 26.8 mm to (156.3, 86.2), turned to 180 degrees
- moved R4 26.1 mm to (126.8, 105.5), turned to 0 degrees
- moved R17 24.7 mm to (131.0, 108.4), turned to 0 degrees
- moved U5 24.2 mm to (155.0, 90.9), turned to 180 degrees
- moved D4 23.4 mm to (128.9, 98.6)
- moved U6 23.2 mm to (154.5, 92.3)
- moved Q4 22.6 mm to (129.4, 102.8), turned to 90 degrees
- moved R22 22.6 mm to (132.4, 115.2), turned to 0 degrees
- moved R14 22.4 mm to (151.4, 96.8), turned to 180 degrees
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Connections:
- net Net-(D1-A) renamed M1
- net Net-(D2-A) renamed M2
- net Net-(D3-A) renamed M3
- net Net-(D4-A) renamed M4
- C18 pad 1: VCCA -> VCC
- C20 pad 1: VCCA -> VCC
- C24 pad 1: VCCA -> VCC
- C36 pad 2: DGND -> GND
- C37 pad 2: DGND -> GND
- C5 pad 1: DGND -> GND
- R13 pad 1: VCCA -> VCC
- R14 pad 1: VCCA -> VCC
- R17 pad 1: Net-(U9-EN) -> VBUS
- R17 pad 2: VBUS -> Net-(U9-EN)
- U1 pad 12: VCCA -> VCC
- U1 pad 5: VCCA -> VCC
- U1 pad 8: VCCA -> VCC
- U11 pad 1: DGND -> GND
- U11 pad 10: /EN1 -> /P1
- U11 pad 11: /TDO -> unconnected-(U11-IO26-Pad11)
- U11 pad 12: /EN2 -> unconnected-(U11-IO27-Pad12)
- U11 pad 15: DGND -> GND
- U11 pad 25: Net-(Q8-C) -> /P2
- U11 pad 26: /MOTOR3 -> /MOTOR1
- U11 pad 27: /MOTOR4 -> /MOTOR2
- U11 pad 28: (no net) -> unconnected-(U11-IO17-Pad28)
- U11 pad 29: /MOTOR1 -> /MOTOR3
- U11 pad 30: (no net) -> unconnected-(U11-IO18-Pad30)
- U11 pad 33: (no net) -> /P4
- U11 pad 36: (no net) -> /P3
- U11 pad 37: /MOTOR2 -> /MOTOR4
- U11 pad 38: DGND -> GND
- U11 pad 39: DGND -> GND
- U11 pad 8: /SYS -> unconnected-(U11-IO32-Pad8)
- U5 pad 1: VCCA -> VCC
- U5 pad 2: VCCA -> VCC
Routing:
- net VCC: track 55.2 -> 89.1 mm, vias 12 -> 7
- net /P1: track 0.00 -> 33.7 mm
- net VCCA: track 32.2 -> 0.00 mm, vias 5 -> 0
- net /MOTOR4: track 4.38 -> 31.4 mm, vias 1 -> 2
- net /P2: track 0.00 -> 23.2 mm, vias 0 -> 1
- net Net-(Q4-PadG): track 29.4 -> 8.63 mm
- net DGND: track 17.6 -> 0.00 mm, vias 6 -> 0
- net /P4: track 0.00 -> 16.8 mm
- net /I2C_SCL: track 80.1 -> 95.3 mm
- net /MOTOR2: track 19.2 -> 4.27 mm, vias 2 -> 0
- net /I2C_SDA: track 77.1 -> 90.4 mm
- net /INT_GA: track 25.8 -> 37.2 mm, vias 3 -> 2
- net /P3: track 0.00 -> 8.75 mm
- net /MOTOR1: track 11.3 -> 2.68 mm, vias 1 -> 0
- net Net-(Q1-PadG): track 10.3 -> 3.76 mm
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- added copper zone on B.Cu, net GND
- added copper zone on B.Cu, net VBUS
- added copper zone on F.Cu, net VCC
- removed copper zone on B.Cu, net (none)
- removed copper zone on B.Cu, net DGND
- removed copper zone on F.Cu, net DGND
- removed copper zone on In1.Cu, net DGND
- removed copper zone on In1.Cu, net GND
- removed copper zone on In2.Cu, net VBUS
- removed copper zone on In2.Cu, net VCC
- removed copper zone on In2.Cu, net VCCA
Other:
- copper layers 4 -> 2
- rule pad_to_mask_clearance: 0.07 -> 0.05
- rule solder_mask_min_width: 0.25 -> 0.15
- board text removed: "1"
- board text removed: "2"
- board text removed: "3"
- board text removed: "4"

Commit message: save
Parts:
- removed P7: MICRO-B-USB, ZX62-B-5PA_11_CFK
- removed U5: MS5611-01BA03, MS5611
- added C3: 100nF, Capacitor_SMD:C_0603_1608Metric, F.Cu at (139.2, 86.1)
- added J3: USB_C_Receptacle_USB2.0, Connector_USB:USB_C_Receptacle_HRO_TYPE-C-31-M-12, F.Cu at (156.8, 85.4)
- added R6: 5k1, Resistor_SMD:R_0603_1608Metric, F.Cu at (160.4, 92.4)
- added R7: 5k1, Resistor_SMD:R_0603_1608Metric, F.Cu at (151.8, 92.3)
- added U2: BMP388, Package_LGA:ST_HLGA-10_2x2mm_P0.5mm_LayoutBorder3x2y, F.Cu at (141.1, 88.9)
- C24: moved to F.Cu
- moved C24 14.0 mm to (138.3, 89.0), turned to 90 degrees
- moved J1 2.95 mm to (137.7, 120.0)
- moved C20 1.62 mm to (134.5, 86.1), turned to 0 degrees
- moved R41 1.60 mm to (140.4, 107.9)
- moved C37 1.51 mm to (135.5, 113.6)
- moved D7 1.30 mm to (129.1, 114.8)
- moved C36 0.75 mm to (157.4, 92.6), turned to -90 degrees
- moved U6 0.68 mm to (155.1, 92.5)
- moved R4 0.63 mm to (127.4, 105.7)
- moved C34 0.22 mm to (131.9, 106.2)
- moved R22 0.20 mm to (132.4, 115.0)
- moved D2 0.18 mm to (136.9, 98.7)
- moved Q4 0.11 mm to (129.3, 102.7)
- moved Q1 0.05 mm to (141.1, 98.4)
Connections:
- U1 pad 4: /INT_GA -> /INT1
- U1 pad 9: unconnected-(U1-INT2-Pad9) -> INT2
- U11 pad 12: unconnected-(U11-IO27-Pad12) -> INT3
- U11 pad 8: unconnected-(U11-IO32-Pad8) -> /INT1
- U11 pad 9: /INT_GA -> INT2
Routing:
- net GND: track 20.6 -> 64.9 mm, vias 8 -> 24
- net INT2: track 0.00 -> 41.0 mm, vias 0 -> 2
- net /INT1: track 0.00 -> 37.7 mm, vias 0 -> 2
- net INT3: track 0.00 -> 37.4 mm, vias 0 -> 2
- net /INT_GA: track 37.2 -> 0.00 mm, vias 2 -> 0
- net VCC: track 89.1 -> 107.4 mm, vias 7 -> 8
- net VBUS: track 64.1 -> 82.2 mm
- net /I2C_SDA: track 90.4 -> 78.4 mm, vias 3 -> 4
- net /P4: track 16.8 -> 9.41 mm
- net /MOTOR4: track 31.4 -> 24.8 mm
- net Net-(J3-CC2): track 0.00 -> 4.36 mm
- net /I2C_SCL: track 95.3 -> 90.9 mm, vias 4 -> 3
- net Net-(J3-CC1): track 0.00 -> 4.14 mm
- net /RX: track 10.8 -> 6.88 mm
- net /TX: track 8.23 -> 4.69 mm
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Other:
- rule solder_mask_min_width: 0.15 -> 0.1

Commit message: save
Parts:
- removed R6, R7: 5k1, Resistor_SMD:R_0603_1608Metric
- removed U1: BMX160, digikey-footprints:LGA-14L_2.5x3mm__LSM6DS3
- added C1: 22uF, Capacitor_SMD:C_0603_1608Metric, F.Cu at (165.0, 117.9)
- added C2: 100nF, Capacitor_SMD:C_0603_1608Metric, F.Cu at (165.0, 121.0)
- added C4: 1uF, Capacitor_SMD:C_0603_1608Metric, F.Cu at (128.1, 88.4)
- added C6: 470pF, Capacitor_SMD:C_0603_1608Metric, F.Cu at (130.8, 112.0)
- added R8: 10k, Resistor_SMD:R_0603_1608Metric, F.Cu at (130.0, 84.2)
- added U3: BNO055, Package_LGA:LGA-28_5.2x3.8mm_P0.5mm, F.Cu at (131.4, 88.4)
- C18: value 100nF -> 120nF
- moved R9 18.4 mm to (164.8, 94.5)
- moved C20 2.02 mm to (135.2, 84.2)
- moved C5 1.31 mm to (165.0, 114.8)
- moved C18 1.18 mm to (135.4, 88.0), turned to -90 degrees
- moved U9 0.24 mm to (134.0, 110.0)
- moved U11 0.15 mm to (153.6, 114.4)
- moved R42 0.15 mm to (127.8, 108.8)
Connections:
- J3 pad A5: Net-(J3-CC1) -> unconnected-(J3-CC1-PadA5)
- J3 pad B5: Net-(J3-CC2) -> unconnected-(J3-CC2-PadB5)
- U9 pad 4: unconnected-(U9-NR-Pad4) -> Net-(U9-NR)
Routing:
- net INT2: track 41.0 -> 0.00 mm, vias 2 -> 0
- net Net-(U11-EN): track 4.38 -> 23.4 mm
- net /P4: track 9.41 -> 19.0 mm
- net /I2C_SCL: track 90.9 -> 82.4 mm, vias 3 -> 5
- net /MOTOR4: track 24.8 -> 31.7 mm
- net /TX: track 4.69 -> 11.1 mm
- net /INT1: track 37.7 -> 43.9 mm
- net /RX: track 6.88 -> 12.8 mm
- net /I2C_SDA: track 78.4 -> 84.3 mm
- net GND: track 64.9 -> 70.6 mm, vias 24 -> 29
- net Net-(J3-CC2): track 4.36 -> 0.00 mm
- net Net-(J3-CC1): track 4.14 -> 0.00 mm
- net /P2: track 21.0 -> 25.1 mm
- net VBUS: track 82.2 -> 78.5 mm
- net /P3: track 7.00 -> 10.7 mm
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
Commit message: save
Parts:
- removed C1: 22uF, Capacitor_SMD:C_0603_1608Metric
- removed C2, C36, C5: 100nF, Capacitor_SMD:C_0603_1608Metric
- removed C34, C37: 2.2uF, Capacitor_SMD:C_0603_1608Metric
- removed C6: 470pF, Capacitor_SMD:C_0603_1608Metric
- removed D5: RED LED, SMDLED-0603
- removed J3: USB_C_Receptacle_USB2.0, Connector_USB:USB_C_Receptacle_HRO_TYPE-C-31-M-12
- removed R17: 100k, Resistor_SMD:R_0603_1608Metric
- removed R9: 10k, Resistor_SMD:R_0402_1005Metric
- removed U11: ESP32-WROOM, ESP32-footprints-Lib:ESP32-WROOM-32_new
- removed U6: NUF2221, SOT363
- removed U9: TPS79301, SOT23_6
- R5: value 330R -> Battery; footprint Resistor_SMD:R_0603_1608Metric -> Connector_PinHeader_2.54mm:PinHeader_1x02_P2.54mm_Vertical
- moved R5 35.5 mm to (137.4, 113.9)
- moved J1 10.5 mm to (132.5, 110.8), turned to 180 degrees
- moved D7 8.69 mm to (130.9, 106.3), turned to 90 degrees
- moved R22 6.39 mm to (133.1, 108.7)
- moved R14 6.35 mm to (145.0, 96.7), turned to -90 degrees
- moved R13 0.81 mm to (146.9, 96.7)
Connections:
- J1 pad 1: /P1 -> /I2C_SCL
- J1 pad 2: /P2 -> /MOTOR4
- J1 pad 3: /P3 -> /I2C_SDA
- J1 pad 4: /TX -> /MOTOR1
- J1 pad 5: /P4 -> INT3
- J1 pad 6: /RX -> /INT1
- J1 pad 7: /I2C_SDA -> /MOTOR2
- J1 pad 8: VBUS -> VCC
- J1 pad 9: /I2C_SCL -> /MOTOR3
- R5 pad 1: /RED -> GND
- R5 pad 2: Net-(D5-K) -> VBUS
Routing:
- net /I2C_SCL: track 82.4 -> 38.6 mm, vias 5 -> 2
- net VCC: track 106.0 -> 64.3 mm, vias 10 -> 7
- net /I2C_SDA: track 84.3 -> 45.9 mm, vias 4 -> 2
- net /P1: track 37.8 -> 0.00 mm
- net /RED: track 31.7 -> 0.00 mm, vias 2 -> 0
- net /MOTOR4: track 31.7 -> 2.93 mm, vias 2 -> 0
- net /P2: track 25.1 -> 0.00 mm, vias 1 -> 0
- net Net-(U11-EN): track 23.4 -> 0.00 mm
- net /MOTOR1: track 2.99 -> 22.4 mm, vias 0 -> 1
- net /P4: track 19.0 -> 0.00 mm
- net /USBD+: track 16.1 -> 0.00 mm
- net /USBD-: track 15.9 -> 0.00 mm
- net VBUS: track 78.5 -> 62.7 mm, vias 4 -> 2
- net /RX: track 12.8 -> 0.00 mm
- net GND: track 70.6 -> 57.8 mm, vias 29 -> 19
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Other:
- board size 40 x 40 mm -> 23 x 40 mm

Commit message: save
Parts:
- removed C3: 100nF, Capacitor_SMD:C_0603_1608Metric
- removed R8: 10k, Resistor_SMD:R_0603_1608Metric
- C18: value 120nF -> 10uF
- C4: value 1uF -> 100nF
Connections:
- U3 pad 4: Net-(U3-~{BOOT_LOAD_PIN}) -> VCC
- U3 pad 6: VCC -> GND
Routing:
- net /I2C_SCL: track 38.6 -> 32.8 mm, vias 2 -> 3
- net /I2C_SDA: track 45.9 -> 40.1 mm, vias 2 -> 0
- net VCC: track 64.3 -> 58.6 mm
- net GND: track 57.8 -> 54.8 mm, vias 19 -> 22
- net Net-(U3-~{BOOT_LOAD_PIN}): track 1.95 -> 0.00 mm
- net INT3: track 32.4 -> 33.1 mm
