File: Drone/Crazyflie contol board.kicad_pcb (KiCad board)
At the start: 2 copper layers, 23 x 40 mm, 29 parts, among them J1 Aux, J2 Motors, Q1 PMV31XN, Q2 PMV31XN, Q3 PMV31XN, Q4 PMV31XN, U2 BMP388, U3 BNO055

Commit message: save
Parts:
- removed D1, D2, D3, D4: BAT54, Diode_SMD:D_SOD-323
- removed Q1, Q2, Q3, Q4: PMV31XN, SOT23GDS
- removed R1, R2, R3, R4: 10k, Resistor_SMD:R_0402_1005Metric
- removed R39, R40, R41, R42: 100R, Resistor_SMD:R_0402_1005Metric
- added J3: Conn_01x05_Pin, Connector_PinHeader_2.54mm:PinHeader_1x05_P2.54mm_Vertical, F.Cu at (137.8, 98.6)
Connections:
- net VBUS renamed +BATT
- J1 pad 2: /MOTOR4 -> M4
- J1 pad 4: /MOTOR1 -> M1
- J1 pad 7: /MOTOR2 -> M2
- J1 pad 9: /MOTOR3 -> M3
Routing:
- net M1: track 4.91 -> 32.3 mm, vias 0 -> 1
- net M3: track 6.37 -> 30.2 mm
- net +BATT: track 62.7 -> 39.4 mm, vias 2 -> 1
- net /MOTOR1: track 22.4 -> 0.00 mm, vias 1 -> 0
- net M2: track 6.22 -> 26.5 mm
- net /MOTOR3: track 15.1 -> 0.00 mm
- net /MOTOR2: track 14.4 -> 0.00 mm
- net Net-(Q3-PadG): track 9.62 -> 0.00 mm
- net M4: track 7.00 -> 16.1 mm
- net GND: track 54.8 -> 46.0 mm
- net Net-(Q4-PadG): track 7.87 -> 0.00 mm
- net Net-(Q2-PadG): track 6.04 -> 0.00 mm
- net Net-(Q1-PadG): track 3.76 -> 0.00 mm
- net /MOTOR4: track 2.93 -> 0.00 mm

Commit message: save
Parts:
- removed J2: Motors, Connector_IDC:IDC-Header_2x05_P2.54mm_Vertical
- removed J3: Conn_01x05_Pin, Connector_PinHeader_2.54mm:PinHeader_1x05_P2.54mm_Vertical
- added C1: 10uF, Capacitor_SMD:C_0603_1608Metric, F.Cu at (134.2, 100.5)
- added C2: 10uF, Capacitor_SMD:C_0603_1608Metric, F.Cu at (140.1, 97.1)
- added C3: 100nF, Capacitor_SMD:C_0603_1608Metric, F.Cu at (140.4, 100.5)
- added C5: 10uF, Capacitor_SMD:C_0603_1608Metric, F.Cu at (139.4, 94.8)
- added J4: Conn_01x08_Pin, Connector_PinHeader_2.54mm:PinHeader_1x08_P2.54mm_Vertical, F.Cu at (111.6, 77.4)
- added J5: Conn_01x04_Pin, Connector_PinHeader_2.54mm:PinHeader_1x04_P2.54mm_Vertical, F.Cu at (164.9, 82.2)
- added L1: 2.2uH, Inductor_SMD:L_0805_2012Metric_Pad1.05x1.20mm_HandSolder, F.Cu at (132.6, 97.7)
- added P1: USB_C_Plug_USB2.0, Connector_USB:USB_C_Receptacle_HRO_TYPE-C-31-M-12, F.Cu at (175.8, 91.4)
- added R1: 100R, Resistor_SMD:R_0603_1608Metric, F.Cu at (137.3, 100.4)
- added R2: 10k, Resistor_SMD:R_0603_1608Metric, F.Cu at (151.4, 130.7)
- added R3: 5.1k, Resistor_SMD:R_0603_1608Metric, F.Cu at (169.3, 88.9)
- added R4: 5.1k, Resistor_SMD:R_0603_1608Metric, F.Cu at (166.8, 96.9)
- added SW1: SW_Push, Button_Switch_SMD:SW_Push_1P1T_XKB_TS-1187A, F.Cu at (109.0, 117.0)
- added SW2: SW_Push, Button_Switch_SMD:SW_Push_1P1T_XKB_TS-1187A, F.Cu at (101.0, 110.0)
- added SW3: SW_Push, Button_Switch_SMD:SW_Push_1P1T_XKB_TS-1187A, F.Cu at (109.0, 103.0)
- added SW4: SW_Push, Button_Switch_SMD:SW_Push_1P1T_XKB_TS-1187A, F.Cu at (165.0, 117.0)
- added SW5: SW_Push, Button_Switch_SMD:SW_Push_1P1T_XKB_TS-1187A, F.Cu at (173.0, 110.0)
- added SW6: SW_Push, Button_Switch_SMD:SW_Push_1P1T_XKB_TS-1187A, F.Cu at (165.0, 103.0)
- added SW7: SW_Push, Button_Switch_SMD:SW_Push_1P1T_XKB_TS-1187A, F.Cu at (157.0, 110.0)
- added SW8: SW_Push, Button_Switch_SMD:SW_Push_1P1T_XKB_TS-1187A, F.Cu at (116.0, 110.0)
- added U1: ESP32-S3-WROOM-1, RF_Module:ESP32-S3-WROOM-1, F.Cu at (138.5, 127.2)
- added U4: TPS63000, Package_SON:Texas_DRC0010J_ThermalVias, F.Cu at (137.0, 97.7)
- added U5: NUF2221-Crazyflie-contol-board-rescue, Package_TO_SOT_SMD:SOT-363_SC-70-6, F.Cu at (166.9, 94.1)
- J1: value Aux -> Conn_01x05_Pin; footprint Connector_IDC:IDC-Header_2x05_P2.54mm_Vertical -> Connector_PinHeader_2.54mm:PinHeader_1x05_P2.54mm_Vertical; moved to F.Cu
- moved J1 23.6 mm to (117.3, 128.9), turned to -90 degrees
- moved BAT 20.5 mm to (127.2, 96.1), turned to 180 degrees
- renumbered R5 to BAT
Connections:
- J1 pad 1: /I2C_SCL -> INT0
- J1 pad 2: M4 -> GND
- J1 pad 3: /I2C_SDA -> VCC
- J1 pad 4: M1 -> /RX
- J1 pad 5: INT3 -> /TX
- U2 pad 7: INT3 -> INT2
Routing:
- net /SCK: track 0.00 -> 116.4 mm
- net VCC: track 58.6 -> 167.6 mm, vias 7 -> 9
- net /MOSI: track 0.00 -> 97.1 mm
- net /MISO: track 0.00 -> 52.5 mm, vias 0 -> 1
- net /CS2: track 0.00 -> 48.7 mm
- net /DC: track 0.00 -> 44.8 mm
- net GND: track 46.0 -> 90.2 mm, vias 22 -> 23
- net /CS1: track 0.00 -> 43.7 mm, vias 0 -> 2
- net /USBD-: track 0.00 -> 40.4 mm
- net INT2: track 0.00 -> 40.3 mm, vias 0 -> 2
- net +BATT: track 39.4 -> 79.1 mm, vias 1 -> 4
- net /USBD+: track 0.00 -> 38.8 mm
- net Net-(U1-IO2): track 0.00 -> 33.2 mm
- net INT3: track 33.1 -> 0.00 mm
- net M1: track 32.3 -> 0.00 mm, vias 1 -> 0
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- removed copper zone on B.Cu, net +BATT
Other:
- board size 23 x 40 mm -> 83 x 59 mm
- board text added: "Rev. 1.0"
- board text removed: "Rev. 2.4"

Commit message: save
Parts:
- R13, R14: value 2.2k -> 2k2
- moved P1 1.80 mm to (175.8, 93.2)
- moved R3 1.61 mm to (169.1, 90.5)
Connections:
- P1 pad B6: (no net) -> /USBD+
- P1 pad B7: (no net) -> /USBD-
Routing:
- net /USBD+: track 38.8 -> 43.4 mm
- net /SCK: track 116.4 -> 111.9 mm
- net /USBD-: track 40.4 -> 44.3 mm
- net GND: track 90.2 -> 92.5 mm, vias 23 -> 89
- net Net-(P1-CC): track 6.61 -> 5.42 mm
