File: Drone/Crazyflie contol board.kicad_pcb (KiCad board)
At the start: 2 copper layers, 83 x 59 mm, 35 parts, among them J1 Conn_01x05_Pin, J4 Conn_01x08_Pin, J5 Conn_01x04_Pin, P1 USB_C_Plug_USB2.0, SW1 SW_Push, SW2 SW_Push, SW3 SW_Push, SW4 SW_Push, SW5 SW_Push, SW6 SW_Push, SW7 SW_Push, SW8 SW_Push, U1 ESP32-S3-WROOM-1, U2 BMP388, U3 BNO055, U4 TPS63000, U5 NUF2221-Crazyflie-contol-boar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

Commit message: save
Routing:
- net VCC: track 167.8 -> 170.0 mm
- net GND: track 92.5 -> 93.6 mm
