File: Drone/Crazyflie contol board.kicad_sch (KiCad schematic)
At the start: 40 parts, among them P1 CONN_2, P2 CONN_2, P3 CONN_2, P4 CONN_2, Q1 PMV31XN, Q2 PMV31XN, Q3 PMV31XN, Q4 PMV31XN, Q7 SS8050-G, Q8 SS8050-G, SW2 BOOT, U11 ESP32-WROOM, U12 CP2102N-A01-GQFN24

Commit message: save
Parts:
- added J1: Aux, Connector_IDC:IDC-Header_2x05_P2.54mm_Vertical, symbol Connector_Generic:Conn_02x05_Odd_Even
Connections:
- net CHG: now also J1.6 (Pin_6)
- net EN1: now also J1.3 (Pin_3)
- net EN2: now also J1.1 (Pin_1)
- net GND: now also J1.10 (Pin_10)
- net TDO: now also J1.2 (Pin_2)
- net VBUS: now reaches U12.8 (VBUS)
- net VBUS: now also J1.8 (Pin_8)
- net I2C_SCK_VCCA renamed I2C_SCK
- net I2C_SCK: now also J1.7 (Pin_7)
- net I2C_SCL_VCCA renamed I2C_SCL
- net I2C_SCL: now also J1.9 (Pin_9)
- net PGOOD renamed PGO
- net PGO: now also J1.4 (Pin_4)
- net SYSOFF renamed SYS
- net SYS: now also J1.5 (Pin_5)
Other:
- sheet POWER ports: added none; removed CHG, EN1, EN2, PGOOD, SYSOFF, USB_CON, VBAT

Commit message: update
Connections:
- net EN1: now also J1.1 (Pin_1); no longer J1.3 (Pin_3)
- net EN2: now also J1.2 (Pin_2); no longer J1.1 (Pin_1)
- net TDO: now also J1.3 (Pin_3); no longer J1.2 (Pin_2)
Changed lines of the file:
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@@
   (title_block
     (title "Crazyflie control board")
-    (date "2020-05-12")
-    (rev "2.1")
+    (date "2022-08-07")
+    (rev "2.2")
     (company "Bitcraze AB (CC BY-NC-SA)")
   )
@@
     (effects (font (size 1.524 1.524)) (justify right bottom))
   )
-  (label "EN2" (at 25.4 121.92 180)
+  (label "EN1" (at 25.4 121.92 180)
     (effects (font (size 1.524 1.524)) (justify right bottom))
   )
@@
     (effects (font (size 1.524 1.524)) (justify left bottom))
   )
-  (label "EN1" (at 25.4 124.46 180)
+  (label "TDO" (at 25.4 124.46 180)
     (effects (font (size 1.524 1.524)) (justify right bottom))
   )
@@
     (effects (font (size 1.524 1.524)) (justify left bottom))
   )
-  (label "TDO" (at 38.1 121.92 0)
+  (label "EN2" (at 38.1 121.92 0)
     (effects (font (size 1.27 1.27)) (justify left bottom))
   )
@@
       (reference "#PWR065") (unit 1) (value "+BATT") (footprint "")
     )
-    (path "/00000000-0000-0000-0000-00004de77332/00000000-0000-0000-0000-00004defa9bf"
-      (reference "#PWR068") (unit 1) (value "GND") (footprint "")
-    )
     (path "/00000000-0000-0000-0000-00004de77332/00000000-0000-0000-0000-00004de7ddcc"
       (reference "#PWR073") (unit 1) (value "VCCA") (footprint "")
@@
       (reference "R42") (unit 1) (value "100R") (footprint "digikey-footprints:0603")
     )
-    (path "/00000000-0000-0000-0000-00004de77332/00000000-0000-0000-0000-00004defa9a9"
-      (reference "SW1") (unit 1) (value "PUSH ON/OFF") (footprint "SPST-NO-4x2.5")
-    )
     (path "/00000000-0000-0000-0000-00005c766a94"
