File: Drone/Crazyflie contol board.kicad_sch (KiCad schematic)
At the start: 41 parts, among them J1 Aux, P1 CONN_2, P2 CONN_2, P3 CONN_2, P4 CONN_2, Q1 PMV31XN, Q2 PMV31XN, Q3 PMV31XN, Q4 PMV31XN, Q7 SS8050-G, Q8 SS8050-G, SW2 BOOT, U11 ESP32-WROOM, U12 CP2102N-A01-GQFN24

Commit message: save
Parts:
- removed C3: 100nF, ESP32-footprints-Lib:0603_new_new, symbol Crazyflie-contol-board-rescue:C-Crazyflie-contol-board-rescue
- removed C4: 4.7uF, ESP32-footprints-Lib:0603_new_new, symbol Crazyflie-contol-board-rescue:C-Crazyflie-contol-board-rescue
- removed D6: GREEN LED, SMDLED-0603, symbol Crazyflie-contol-board-rescue:LED-Crazyflie-contol-board-rescue
- removed Q7, Q8: SS8050-G, digikey-footprints:SOT-23-3, symbol Crazyflie-contol-board-rescue:BC817-Transistor_BJT
- removed R10, R8: 10k, ESP32-footprints-Lib:0603_new_new, symbol Crazyflie-contol-board-rescue:R-Crazyflie-contol-board-rescue
- removed R6: 220R, ESP32-footprints-Lib:0603_new_new, symbol Crazyflie-contol-board-rescue:R-Crazyflie-contol-board-rescue
- removed R7: 1k, ESP32-footprints-Lib:0603_new_new, symbol Crazyflie-contol-board-rescue:R-Crazyflie-contol-board-rescue
- removed SW2: BOOT, ESP32-footprints-Lib:Switch_Tactile_SMD_B3U-1000P_new_new, symbol Crazyflie-contol-board-rescue:SW_PUSH-Crazyflie-contol-board-rescue
- removed U12: CP2102N-A01-GQFN24, ESP32-footprints-Lib:QFN-24-1EP_4x4mm_new_new_new, symbol Crazyflie-contol-board-rescue:CP2102N-A01-GQFN24-Interface_USB
- C1, C2, C5, R13, R14, R5, R9: footprint ESP32-footprints-Lib:0603_new_new -> ESP32-footprints-Lib:0603
- U11: footprint ESP32-footprints-Lib:ESP32-WROOM-32_new -> ESP32-footprints-Lib:ESP32-WROOM-32
Connections:
- net I2C_SCL: now also U11.7 (IO35); no longer U11.36 (IO22)
- net MOTOR1: now also U11.29 (IO5); no longer U11.16 (IO13)
- net USBD+: now also U11.14 (IO12)
- net USBD-: now also U11.13 (IO14)
- net RX: now reaches U11.34 (RXD0)
- net RX: now also J1.6 (Pin_6)
- net TX: now reaches U11.35 (TXD0)
- net TX: now also J1.4 (Pin_4)
- net I2C_SDA: now reaches U11.6 (IO34)
- net I2C_SDA: now also J1.7 (Pin_7), R13.2
- net CHG: no longer names the net of U11.28 (IO17)
- net CHG: no longer J1.6 (Pin_6)
- net EN1 renamed P1
- net EN2 renamed P2
- removed net I2C_SCK: J1.7 (Pin_7), R13.2, U11.33 (IO21)
- net PGO: no longer names the net of U11.30 (IO18)
- net PGO: no longer J1.4 (Pin_4)
- net SYS renamed P4
- net TDO renamed P3
Other:
- moved on the sheet: C2, C5, D4, D5, J1, P4, Q4, R4, R42, R5, R9

Commit message: save
Parts:
- removed P1, P2, P3, P4: CONN_2, PINHEADER_127_2X1, symbol Crazyflie-contol-board-rescue:CONN_2-Crazyflie-contol-board-rescue
- added J2: Motors, Connector_IDC:IDC-Header_2x05_P2.54mm_Vertical, symbol Connector_Generic:Conn_02x05_Odd_Even
- C1, C2, C5: footprint ESP32-footprints-Lib:0603 -> Capacitor_SMD:C_0603_1608Metric
- D1, D2, D3, D4: footprint SOD323 -> Diode_SMD:D_SOD-323
- R1, R2, R3, R39, R4, R40, R41: footprint SM0402 -> Resistor_SMD:R_0402_1005Metric
- R13, R14, R5: footprint ESP32-footprints-Lib:0603 -> Resistor_SMD:R_0603_1608Metric
- R42: footprint digikey-footprints:0603 -> Resistor_SMD:R_0402_1005Metric
- R9: footprint ESP32-footprints-Lib:0603 -> Resistor_SMD:R_0402_1005Metric
Connections:
- net DGND is gone; now on net GND: C1.2, C2.2, C5.1, U11.1 (GND), U11.15 (GND), U11.38 (GND), U11.39 (GND-PAD)
- net VBUS is gone; now on net +BATT: J1.8 (Pin_8)
- net VCCA is gone; now on net VCC: R13.1, R14.1
- net +BATT: now also J2.10 (Pin_10), J2.2 (Pin_2), J2.4 (Pin_4), J2.6 (Pin_6), J2.8 (Pin_8)
- net GND: now also J2.9 (Pin_9)
- net MOTOR1: now also U11.26 (IO4); no longer U11.29 (IO5)
- net MOTOR2: now also U11.27 (IO16); no longer U11.37 (IO23)
- net MOTOR3: now also U11.29 (IO5); no longer U11.26 (IO4)
- net MOTOR4: now also U11.37 (IO23); no longer U11.27 (IO16)
- net P2: now also U11.25 (IO0); no longer U11.12 (IO27)
- net P3: now also U11.36 (IO22); no longer U11.11 (IO26)
- net P4: now also U11.33 (IO21); no longer U11.8 (IO32)
- net M1: now reaches D1.1 (A), Q1.D
- net M1: now also J2.1 (Pin_1)
- net M2: now reaches D2.1 (A), Q2.D
- net M2: now also J2.3 (Pin_3)
- net M3: now reaches D3.1 (A), Q3.D
- net M3: now also J2.5 (Pin_5)
- net M4: now reaches D4.1 (A), Q4.D
- net M4: now also J2.7 (Pin_7)

Commit message: save
Connections:
- net INT3: now reaches U11.12 (IO27)
- net INT1: now reaches U11.8 (IO32)
- net INT_GA renamed INT2
Other:
- sheet IMU ports: added INT1; removed INT_GA
- moved on the sheet: C5

Commit message: save
Parts:
- removed C1: 22uF, Capacitor_SMD:C_0603_1608Metric, symbol Crazyflie-contol-board-rescue:C-Crazyflie-contol-board-rescue
- removed C2, C5: 100nF, Capacitor_SMD:C_0603_1608Metric, symbol Crazyflie-contol-board-rescue:C-Crazyflie-contol-board-rescue
- removed D5: RED LED, SMDLED-0603, symbol Crazyflie-contol-board-rescue:LED-Crazyflie-contol-board-rescue
- removed R5: 330R, Resistor_SMD:R_0603_1608Metric, symbol Crazyflie-contol-board-rescue:R-Crazyflie-contol-board-rescue
- removed R9: 10k, Resistor_SMD:R_0402_1005Metric, symbol Crazyflie-contol-board-rescue:R-Crazyflie-contol-board-rescue
- removed U11: ESP32-WROOM, ESP32-footprints-Lib:ESP32-WROOM-32, symbol Crazyflie-contol-board-rescue:ESP32-WROOM-ESP32-footprints-Shem-Lib
- added R5: Battery, Connector_PinHeader_2.54mm:PinHeader_1x02_P2.54mm_Vertical, symbol Device:R
Connections:
- net +BATT: now also R5.2; no longer J1.8 (Pin_8)
- net GND: now also R5.1
- net I2C_SCL: now also J1.1 (Pin_1); no longer J1.9 (Pin_9)
- net I2C_SDA: now also J1.3 (Pin_3); no longer J1.7 (Pin_7)
- net INT1: now also J1.6 (Pin_6)
- net INT3: now also J1.5 (Pin_5)
- net MOTOR1: now also J1.4 (Pin_4)
- net MOTOR2: now also J1.7 (Pin_7)
- net MOTOR3: now also J1.9 (Pin_9)
- net MOTOR4: now also J1.2 (Pin_2)
- net P1: no longer J1.1 (Pin_1)
- net P2: no longer J1.2 (Pin_2)
- net P3: no longer J1.3 (Pin_3)
- net P4: no longer J1.5 (Pin_5)
- net RX: no longer J1.6 (Pin_6)
- net TX: no longer J1.4 (Pin_4)
- net VCC renamed VCCA
- net VCCA: now also J1.8 (Pin_8)

Commit message: save
Parts:
- removed D1, D2, D3, D4: BAT54, Diode_SMD:D_SOD-323, symbol Crazyflie-contol-board-rescue:DIODESCH-Crazyflie-contol-board-rescue
- removed Q1, Q2, Q3, Q4: PMV31XN, SOT23GDS, symbol Crazyflie-contol-board-rescue:MOSFET_N-Crazyflie-contol-board-rescue
- removed R1, R2, R3, R4: 10k, Resistor_SMD:R_0402_1005Metric, symbol Crazyflie-contol-board-rescue:R-Crazyflie-contol-board-rescue
- removed R39, R40, R41, R42: 100R, Resistor_SMD:R_0402_1005Metric, symbol Crazyflie-contol-board-rescue:R-Crazyflie-contol-board-rescue
- added J3: Conn_01x05_Pin, Connector_PinHeader_2.54mm:PinHeader_1x05_P2.54mm_Vertical, symbol Connector:Conn_01x05_Pin
Connections:
- net GND: now also J3.1 (Pin_1), J3.2 (Pin_2), J3.3 (Pin_3), J3.4 (Pin_4), J3.5 (Pin_5)
- net M1: now also J1.4 (Pin_4)
- net M2: now also J1.7 (Pin_7)
- net M3: now also J1.9 (Pin_9)
- net M4: now also J1.2 (Pin_2)
- net MOTOR1: no longer J1.4 (Pin_4)
- net MOTOR2: no longer J1.7 (Pin_7)
- net MOTOR3: no longer J1.9 (Pin_9)
- net MOTOR4: no longer J1.2 (Pin_2)
Other:
- note removed: "Coreless motor"

Commit message: save
Parts:
- removed J1: Aux, Connector_IDC:IDC-Header_2x05_P2.54mm_Vertical, symbol Connector_Generic:Conn_02x05_Odd_Even
- removed J2: Motors, Connector_IDC:IDC-Header_2x05_P2.54mm_Vertical, symbol Connector_Generic:Conn_02x05_Odd_Even
- removed J3: Conn_01x05_Pin, Connector_PinHeader_2.54mm:PinHeader_1x05_P2.54mm_Vertical, symbol Connector:Conn_01x05_Pin
- added C1, C2, C5: 10uF, Capacitor_SMD:C_0603_1608Metric, symbol Device:C
- added C3: 100nF, Capacitor_SMD:C_0603_1608Metric, symbol Device:C
- added J1: Conn_01x05_Pin, symbol Connector:Conn_01x05_Pin
- added J4: Conn_01x08_Pin, symbol Connector:Conn_01x08_Pin
- added J5: Conn_01x04_Pin, symbol Connector:Conn_01x04_Pin
- added L1: 2.2uH, symbol Device:L
- added P1: USB_C_Plug_USB2.0, symbol Connector:USB_C_Plug_USB2.0
- added R1: 100R, Resistor_SMD:R_0603_1608Metric, symbol Device:R
- added R2: 10k, Resistor_SMD:R_0603_1608Metric, symbol Device:R
- added R3, R4: 5.1k, Resistor_SMD:R_0603_1608Metric, symbol Device:R
- added SW1, SW2, SW3, SW4, SW5, SW6, SW7, SW8: SW_Push, symbol Switch:SW_Push
- added U1: ESP32-S3-WROOM-1, RF_Module:ESP32-S3-WROOM-1, symbol RF_Module:ESP32-S3-WROOM-1
- added U4: TPS63000, Package_SON:Texas_DRC0010J_ThermalVias, symbol Regulator_Switching:TPS63000
- added U5: NUF2221-Crazyflie-contol-board-rescue, symbol Crazyflie-contol-board-rescue:NUF2221-Crazyflie-contol-board-rescue
- R13, R14: value 2.2k -> 2k2
Connections:
- net +BATT: now also C1.1, P1.A4 (VBUS), P1.A9 (VBUS), P1.B4 (VBUS), P1.B9 (VBUS), R1.1, U4.5 (VIN), U5.5 (VBUS)
- net GND: now also C1.2, C2.2, C3.2, C5.2, J1.2 (Pin_2), J4.2 (Pin_2), P1.A1 (GND), P1.A12 (GND), P1.B1 (GND), P1.B12 (GND), P1.S1 (SHIELD), R3.2, R4.1, SW1.1, SW2.1, SW3.1, SW4.1, SW5.1, SW6.1, SW7.1, SW8.1, U1.1 (GND), U1.40 (GND), U1.41 (GND), U4.11 (PGND), U4.3 (PGND), U4.9 (GND), U5.2 (GND)
- net I2C_SCL: now also U1.17 (IO9)
- net I2C_SDA: now also U1.12 (IO8)
- net INT1: now also U1.9 (IO16)
- net INT2: now also U1.10 (IO17)
- net RX: now also J1.4 (Pin_4), U1.36 (RXD0)
- net TX: now also J1.5 (Pin_5), U1.37 (TXD0)
- net USBD+: now also P1.A6 (D+), U1.14 (USB_D+), U5.1 (D1I), U5.6 (D1C)
- net USBD-: now also P1.A7 (D-), U1.13 (USB_D-), U5.3 (D2I), U5.4 (D2C)
- net VCCA: now also C2.1, C5.1, J1.3 (Pin_3), J4.1 (Pin_1), J4.8 (Pin_8), R2.1, U1.2 (3V3), U4.1 (VOUT), U4.10 (FB)
- new net: C3.1, R1.2, U4.6 (EN), U4.7 (PS/SYNC), U4.8 (VINA)
- new net: SW5.2, U1.5 (IO5)
- new net: SW6.2, U1.6 (IO6)
- new net: P1.A5 (CC), R4.2
- new net: P1.B5 (VCONN), R3.1
- new net: SW7.2, U1.7 (IO7)
- new net: SW8.2, U1.22 (IO14)
- new net: R2.2, U1.3 (EN)
- new net: L1.2, U4.2 (L2)
- new net: L1.1, U4.4 (L1)
- new net: SW4.2, U1.4 (IO4)
- new net: SW2.2, U1.38 (IO2)
- new net: SW1.2, U1.39 (IO1)
- new net CS1: J5.4 (Pin_4), U1.11 (IO18)
- new net CS2: J4.3 (Pin_3), U1.18 (IO10)
- new net DC: J4.5 (Pin_5), U1.31 (IO38)
- new net INT0: J1.1 (Pin_1), U1.27 (IO0)
- new net MISO: J5.2 (Pin_2), U1.21 (IO13)
- new net MOSI: J4.6 (Pin_6), J5.3 (Pin_3), U1.19 (IO11)
- new net SCK: J4.7 (Pin_7), J5.1 (Pin_1), U1.20 (IO12)
- new net SW3: SW3.2, U1.35 (IO42)
Other:
- company: Bitcraze AB (CC BY-NC-SA) -> (none)
- title: Crazyflie control board -> (none)
- moved on the sheet: R5

Commit message: save
Parts:
- added R6, R7: 22R, Resistor_SMD:R_0603_1608Metric, symbol Device:R
Connections:
- net USBD+: now also R6.2; no longer U5.1 (D1I)
- net USBD-: now also R7.2; no longer U5.3 (D2I)
- new net: R7.1, U5.3 (D2I)
- new net: R6.1, U5.1 (D1I)
Changed lines of the file:
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@@
 	(wire
 		(pts
-			(xy 163.83 129.54) (xy 170.18 129.54)
-		)
-		(stroke
-			(width 0)
-			(type default)
-		)
-	)
-	(wire
-		(pts
 			(xy 242.57 74.93) (xy 247.65 74.93)
 		)
@@
 	(wire
 		(pts
-			(xy 163.83 132.08) (xy 170.18 132.08)
-		)
-		(stroke
-			(width 0)
-			(type default)
-		)
-	)
-	(wire
-		(pts
 			(xy 77.47 64.77) (xy 77.47 54.61)
 		)
@@
 	)
 	(label "USBD-"
-		(at 170.18 132.08 0)
+		(at 171.45 132.08 0)
 		(effects
 			(font
@@
 	)
 	(label "USBD+"
-		(at 170.18 129.54 0)
+		(at 171.45 129.54 0)
 		(effects
 			(font
@@
 	)
 	(symbol
+		(lib_id "Device:R")
+		(at 167.64 132.08 90)
+		(unit 1)
+		(exclude_from_sim no)
+		(in_bom yes)
+		(on_board yes)
+		(dnp no)
+		(property "Reference" "R7"
+			(at 167.894 134.62 90)
+			(effects
+				(font
+					(size 1.27 1.27)
+				)
+			)
+		)
+		(property "Value" "22R"
+			(at 167.894 132.08 90)
+			(effects
+				(font
+					(size 1.27 1.27)
+				)
+			)
+		)
+		(property "Footprint" "Resistor_SMD:R_0603_1608Metric"
+			(at 167.64 133.858 90)
+			(effects
+				(font
+					(size 1.27 1.27)
+				)
+				(hide yes)
+			)
+		)
+		(property "Datasheet" "~"
+			(at 167.64 132.08 0)
+			(effects
+				(font
+					(size 1.27 1.27)
+				)
+				(hide yes)
+			)
+		)
+		(property "Description" "Resistor"
+			(at 167.64 132.08 0)
+			(effects
+				(font
+					(size 1.27 1.27)
+				)
+				(hide yes)
+			)
+		)
+		(pin "2"
+		)
+		(pin "1"
+		)
+		(instances
+			(project ""
+				(path "/3e9fa01f-48e9-4c58-997e-0bab5b5694a8"
+					(reference "R7")
+					(unit 1)
+				)
+			)
+		)
+	)
+	(symbol
 		(lib_id "RF_Module:ESP32-S3-WROOM-1")
 		(at 140.97 55.88 0)
@@
 					(unit 1)
 				)
+			)
+		)
+	)
+	(symbol
+		(lib_id "Device:R")
+		(at 167.64 129.54 90)
+		(unit 1)
+		(exclude_from_sim no)
+		(in_bom yes)
+		(on_board yes)
+		(dnp no)
+		(property "Reference" "R6"
+			(at 167.64 127 90)
+			(effects
+				(font
+					(size 1.27 1.27)
+				)
+			)
+		)
+		(property "Value" "22R"
+			(at 168.148 129.54 90)
+			(effects
+				(font
+					(size 1.27 1.27)
+				)
+			)
+		)
+		(property "Footprint" "Resistor_SMD:R_0603_1608Metric"
+			(at 167.64 131.318 90)
+			(effects
+				(font
+					(size 1.27 1.27)
+				)
+				(hide yes)
+			)
+		)
+		(property "Datasheet" "~"
+			(at 167.64 129.54 0)
+			(effects
+				(font
+					(size 1.27 1.27)
+				)
+				(hide yes)
+			)
+		)
+		(property "Description" "Resistor"
+			(at 167.64 129.54 0)
+			(effects
+				(font
+					(size 1.27 1.27)
+				)
+				(hide yes)
+			)
+		)
+		(pin "2"
+		)
+		(pin "1"
+		)
+		(instances
+			(project ""
+				(path "/3e9fa01f-48e9-4c58-997e-0bab5b5694a8"
+					(reference "R6")
+					(unit 1)
+				)
