File: Drone/Power.kicad_sch (KiCad schematic)
At the start: 47 parts, among them P7 MICRO-B-USB, P9 CONN_1, Q5 2N7002, Q6 2N7002, SW1 PUSH ON/OFF, U10 MAX16054, U6 NUF2221, U7 TPS79301, U8 BQ24075, U9 TPS79301

Commit message: save
Parts:
- removed C39: 10uF, ESP32-footprints-Lib:0603_new_new, symbol Crazyflie-contol-board-rescue:C-Crazyflie-contol-board-rescue
- removed C41: 100nF, ESP32-footprints-Lib:0603_new_new, symbol Crazyflie-contol-board-rescue:C-Crazyflie-contol-board-rescue
- removed D8: BLUE LED, SMDLED-0603, symbol Crazyflie-contol-board-rescue:LED-Crazyflie-contol-board-rescue
- removed Q5, Q6: 2N7002, SOT23GDS, symbol Crazyflie-contol-board-rescue:MOSFET_N-Crazyflie-contol-board-rescue
- removed R21: 300k, ESP32-footprints-Lib:0603_new_new, symbol Crazyflie-contol-board-rescue:R-Crazyflie-contol-board-rescue
- removed R23: 150k, ESP32-footprints-Lib:0603_new_new, symbol Crazyflie-contol-board-rescue:R-Crazyflie-contol-board-rescue
- removed R24: 1.2k, ESP32-footprints-Lib:0603_new_new, symbol Crazyflie-contol-board-rescue:R-Crazyflie-contol-board-rescue
- removed R25, R27, R32, R33, R36, R37: 10k, ESP32-footprints-Lib:0603_new_new, symbol Crazyflie-contol-board-rescue:R-Crazyflie-contol-board-rescue
- removed R26: 1.2K, ESP32-footprints-Lib:0603_new_new, symbol Crazyflie-contol-board-rescue:R-Crazyflie-contol-board-rescue
- removed R30: 20k, ESP32-footprints-Lib:0603_new_new, symbol Crazyflie-contol-board-rescue:R-Crazyflie-contol-board-rescue
- removed R31: 100k, ESP32-footprints-Lib:0603_new_new, symbol Crazyflie-contol-board-rescue:R-Crazyflie-contol-board-rescue
- removed R38: 1k, ESP32-footprints-Lib:0603_new_new, symbol Crazyflie-contol-board-rescue:R-Crazyflie-contol-board-rescue
- removed U10: MAX16054, SOT23_6, symbol Crazyflie-contol-board-rescue:MAX16054-Crazyflie-contol-board-rescue
- removed U8: BQ24075, QFN16, symbol Crazyflie-contol-board-rescue:BQ24075-Crazyflie-contol-board-rescue
- BT1: footprint JST-B2B-ZR -> Connector_IDC:IDC-Header_2x05_P2.54mm_Vertical
Connections:
- net VUSB is gone; now on net VCOM: C36.1, P7.1 (VCC)
- no-connect marks 2 -> 1
Other:
- note added: "Analog LDO configured to 2.8V"
- note removed: "Analod LDO configured to 2.8V"
- note removed: "Max input current set to 1.3A Fastcharge current set to 740mA Safty timer is set to 80min No battery temp monitoring Standby current <7uA"
- note removed: "Standby current 3uA@3.7V"
- moved on the sheet: C37, D7, R22, SW1

Commit message: update
Parts:
- removed SW1: PUSH ON/OFF, SPST-NO-4x2.5, symbol Crazyflie-contol-board-rescue:SW_PUSH-Crazyflie-contol-board-rescue
Changed lines of the file:
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@@
-    (stroke (width 0) (type default) (color 0 0 0 0))
-  )
-  (wire (pts (xy 72.39 144.78) (xy 83.82 144.78))
     (stroke (width 0) (type default) (color 0 0 0 0))
   )
@@
   )
   (wire (pts (xy 121.92 58.42) (xy 121.92 48.26))
-    (stroke (width 0) (type default) (color 0 0 0 0))
-  )
-  (wire (pts (xy 99.06 144.78) (xy 104.14 144.78))
     (stroke (width 0) (type default) (color 0 0 0 0))
   )
@@
     (pin "2")
   )
-  (symbol (lib_id "Crazyflie-contol-board-rescue:SW_PUSH-Crazyflie-contol-board-rescue") (at 91.44 144.78 0) (unit 1)
-    (in_bom yes) (on_board yes)
-    (property "Reference" "SW1" (id 0) (at 95.25 141.986 0))
-    (property "Value" "PUSH ON/OFF" (id 1) (at 91.44 144.78 0)
-      (effects (font (size 1.524 1.524)) hide)
-    )
-    (property "Footprint" "SPST-NO-4x2.5" (id 2) (at 91.44 144.78 0)
-      (effects (font (size 1.524 1.524)) hide)
-    )
-    (property "Datasheet" "" (id 3) (at 91.44 144.78 0)
-      (effects (font (size 1.27 1.27)) hide)
-    )
-    (property "Field4" "Omron" (id 4) (at 91.44 144.78 0)
-      (effects (font (size 1.524 1.524)) hide)
-    )
-    (property "Field5" "B3U-3000P" (id 5) (at 91.44 144.78 0)
-      (effects (font (size 1.524 1.524)) hide)
-    )
-    (pin "1")
-    (pin "2")
-  )
-  (symbol (lib_id "Crazyflie-contol-board-rescue:GND-Crazyflie-contol-board-rescue") (at 72.39 144.78 270) (unit 1)
-    (in_bom yes) (on_board yes)
-    (property "Reference" "#PWR068" (id 0) (at 72.39 144.78 0)
-      (effects (font (size 0.762 0.762)) hide)
-    )
-    (property "Value" "GND" (id 1) (at 70.612 144.78 0)
-      (effects (font (size 0.762 0.762)) hide)
-    )
-    (property "Footprint" "" (id 2) (at 72.39 144.78 0)
-      (effects (font (size 1.27 1.27)) hide)
-    )
-    (property "Datasheet" "" (id 3) (at 72.39 144.78 0)
-      (effects (font (size 1.27 1.27)) hide)
-    )
-    (pin "1")
-  )
   (symbol (lib_id "Crazyflie-contol-board-rescue:R-Crazyflie-contol-board-rescue") (at 245.11 92.71 180) (unit 1)

Commit message: save
Parts:
- removed C29, C35: 15pF, ESP32-footprints-Lib:0603_new_new, symbol Crazyflie-contol-board-rescue:C-Crazyflie-contol-board-rescue
- removed C30, C31: 4.7uF, ESP32-footprints-Lib:0603_new_new, symbol Crazyflie-contol-board-rescue:C-Crazyflie-contol-board-rescue
- removed C32, C40: 10nF, ESP32-footprints-Lib:0603_new_new, symbol Crazyflie-contol-board-rescue:C-Crazyflie-contol-board-rescue
- removed C33: 100nF, ESP32-footprints-Lib:0603_new_new, symbol Crazyflie-contol-board-rescue:C-Crazyflie-contol-board-rescue
- removed R16: 39k, ESP32-footprints-Lib:0603_new_new, symbol Crazyflie-contol-board-rescue:R-Crazyflie-contol-board-rescue
- removed R18, R28: 30k, ESP32-footprints-Lib:0603_new_new, symbol Crazyflie-contol-board-rescue:R-Crazyflie-contol-board-rescue
- removed R19, R29: 0R, ESP32-footprints-Lib:0603_new_new, symbol Crazyflie-contol-board-rescue:R-Crazyflie-contol-board-rescue
- removed R20: 42.2k, ESP32-footprints-Lib:0603_new_new, symbol Crazyflie-contol-board-rescue:R-Crazyflie-contol-board-rescue
- removed U7: TPS79301, SOT23_6, symbol Crazyflie-contol-board-rescue:TPS79301-Crazyflie-contol-board-rescue
- BT1: footprint Connector_IDC:IDC-Header_2x05_P2.54mm_Vertical -> Connector_PinHeader_2.54mm:PinHeader_1x02_P2.54mm_Vertical
- C34, C36, C37, C38, R17, R22: footprint ESP32-footprints-Lib:0603_new_new -> ESP32-footprints-Lib:0603
Connections:
- net +BATT: now also C34.1, C36.1, C38.1, P7.1 (VCC), R17.1, U9.1 (IN)
- net DGND: no longer C36.2, C37.2, D7.2 (K), P7.5 (GND), U6.2 (GND)
- net GND: now also C36.2, C37.2, D7.2 (K), P7.5 (GND), U6.2 (GND)
- removed net VCOM: C34.1, C36.1, C38.1, P7.1 (VCC), R17.2, U9.1 (IN), U9.3 (EN)
- new net: R17.2, U9.3 (EN)
Other:
- note removed: "AGND star connection @ LDO GND pin"
- note removed: "Analog LDO configured to 2.8V"
- note removed: "DGND star connection @ LDO GND pin"
- note removed: "When USB is connected digital LDO will give 3.3V otherwise 2.8V"
- moved on the sheet: C34, C36, C38, R17

Commit message: save
Parts:
- removed BT1: BATTERY, Connector_PinHeader_2.54mm:PinHeader_1x02_P2.54mm_Vertical, symbol Crazyflie-contol-board-rescue:BATTERY-Crazyflie-contol-board-rescue
- removed C38: 100nF, ESP32-footprints-Lib:0603, symbol Crazyflie-contol-board-rescue:C-Crazyflie-contol-board-rescue
- C34, C37: value 4.7uF -> 2.2uF; footprint ESP32-footprints-Lib:0603 -> Capacitor_SMD:C_0603_1608Metric
- C36: footprint ESP32-footprints-Lib:0603 -> Capacitor_SMD:C_0603_1608Metric
- R17: value 10R -> 100k; footprint ESP32-footprints-Lib:0603 -> Resistor_SMD:R_0603_1608Metric
- R22: footprint ESP32-footprints-Lib:0603 -> Resistor_SMD:R_0603_1608Metric
Changed lines of the file:
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@@
   (junction (at 68.58 81.28) (diameter 0) (color 0 0 0 0)
   )
-  (junction (at 165.1 116.84) (diameter 0) (color 0 0 0 0)
-  )
   (junction (at 233.68 83.82) (diameter 0) (color 0 0 0 0)
   )
   (junction (at 121.92 48.26) (diameter 0) (color 0 0 0 0)
-  )
-  (junction (at 165.1 96.52) (diameter 0) (color 0 0 0 0)
-  )
-  (junction (at 203.2 146.05) (diameter 0) (color 0 0 0 0)
   )
   (junction (at 245.11 83.82) (diameter 0) (color 0 0 0 0)
@@
     (stroke (width 0) (type default))
   )
-  (wire (pts (xy 68.58 116.84) (xy 165.1 116.84))
+  (wire (pts (xy 68.58 116.84) (xy 173.99 116.84))
     (stroke (width 0) (type default))
   )
@@
     (stroke (width 0) (type default))
   )
-  (wire (pts (xy 265.43 153.67) (xy 265.43 158.75))
-    (stroke (width 0) (type default))
-  )
   (wire (pts (xy 41.91 39.37) (xy 41.91 83.82))
     (stroke (width 0) (type default))
@@
     (stroke (width 0) (type default))
   )
-  (wire (pts (xy 203.2 146.05) (xy 205.74 146.05))
-    (stroke (width 0) (type default))
-  )
   (wire (pts (xy 44.45 86.36) (xy 44.45 36.83))
     (stroke (width 0) (type default))
@@
     (stroke (width 0) (type default))
   )
-  (wire (pts (xy 165.1 96.52) (xy 165.1 101.6))
-    (stroke (width 0) (type default))
-  )
   (wire (pts (xy 265.43 134.62) (xy 265.43 138.43))
     (stroke (width 0) (type default))
@@
     (stroke (width 0) (type default))
   )
-  (wire (pts (xy 165.1 111.76) (xy 165.1 116.84))
-    (stroke (width 0) (type default))
-  )
   (wire (pts (xy 198.12 146.05) (xy 203.2 146.05))
     (stroke (width 0) (type default))
@@
     (stroke (width 0) (type default))
   )
-  (wire (pts (xy 223.52 146.05) (xy 220.98 146.05))
-    (stroke (width 0) (type default))
-  )
   (wire (pts (xy 39.37 91.44) (xy 39.37 116.84))
     (stroke (width 0) (type default))
@@
   )
   (wire (pts (xy 41.91 83.82) (xy 36.83 83.82))
-    (stroke (width 0) (type default))
-  )
-  (wire (pts (xy 173.99 116.84) (xy 165.1 116.84))
     (stroke (width 0) (type default))
   )
@@
     )
   )
-  (symbol (lib_id "Crazyflie-contol-board-rescue:C-Crazyflie-contol-board-rescue") (at 165.1 106.68 0) (unit 1)
-    (in_bom yes) (on_board yes) (dnp no)
-    (property "Reference" "C38" (at 166.37 104.14 0)
-      (effects (font (size 1.27 1.27)) (justify left))
-    )
-    (property "Value" "100nF" (at 166.37 109.22 0)
-      (effects (font (size 1.27 1.27)) (justify left))
-    )
-    (property "Footprint" "ESP32-footprints-Lib:0603" (at 165.1 106.68 0)
-      (effects (font (size 1.524 1.524)) hide)
-    )
-    (property "Datasheet" "" (at 165.1 106.68 0)
-      (effects (font (size 1.27 1.27)) hide)
-    )
-    (pin "1")
-    (pin "2")
-    (instances
-      (project "Crazyflie contol board"
-        (path "/3e9fa01f-48e9-4c58-997e-0bab5b5694a8/00000000-0000-0000-0000-00004de77332"
-          (reference "C38") (unit 1)
-        )
-      )
-    )
-  )
   (symbol (lib_id "Crazyflie-contol-board-rescue:C-Crazyflie-contol-board-rescue") (at 233.68 100.33 0) (unit 1)
     (in_bom yes) (on_board yes) (dnp no)
@@
       (effects (font (size 1.27 1.27)) (justify left))
     )
-    (property "Value" "4.7uF" (at 234.95 102.87 0)
+    (property "Value" "2.2uF" (at 234.95 102.87 0)
       (effects (font (size 1.27 1.27)) (justify left))
     )
-    (property "Footprint" "ESP32-footprints-Lib:0603" (at 233.68 100.33 0)
+    (property "Footprint" "Capacitor_SMD:C_0603_1608Metric" (at 233.68 100.33 0)
       (effects (font (size 1.524 1.524)) hide)
     )
@@
       (effects (font (size 1.27 1.27)))
     )
-    (property "Value" "10R" (at 191.77 146.05 90)
+    (property "Value" "100k" (at 191.77 146.05 90)
       (effects (font (size 1.27 1.27)))
     )
-    (property "Footprint" "ESP32-footprints-Lib:0603" (at 191.77 146.05 0)
+    (property "Footprint" "Resistor_SMD:R_0603_1608Metric" (at 191.77 146.05 0)
       (effects (font (size 1.524 1.524)) hide)
     )
@@
       (effects (font (size 1.27 1.27)) (justify left))
     )
-    (property "Footprint" "ESP32-footprints-Lib:0603" (at 68.58 97.79 0)
+    (property "Footprint" "Capacitor_SMD:C_0603_1608Metric" (at 68.58 97.79 0)
       (effects (font (size 1.524 1.524)) hide)
     )
@@
       (effects (font (size 1.27 1.27)) (justify left))
     )
-    (property "Value" "4.7uF" (at 123.19 60.96 0)
+    (property "Value" "2.2uF" (at 123.19 60.96 0)
       (effects (font (size 1.27 1.27)) (justify left))
     )
-    (property "Footprint" "ESP32-footprints-Lib:0603" (at 121.92 58.42 0)
+    (property "Footprint" "Capacitor_SMD:C_0603_1608Metric" (at 121.92 58.42 0)
       (effects (font (size 1.524 1.524)) hide)
     )
@@
       (effects (font (size 1.27 1.27)))
     )
-    (property "Footprint" "ESP32-footprints-Lib:0603" (at 245.11 92.71 0)
+    (property "Footprint" "Resistor_SMD:R_0603_1608Metric" (at 245.11 92.71 0)
       (effects (font (size 1.524 1.524)) hide)
     )
@@
         (path "/3e9fa01f-48e9-4c58-997e-0bab5b5694a8/00000000-0000-0000-0000-00004de77332"
           (reference "D7") (unit 1)
-        )
-      )
-    )
-  )
-  (symbol (lib_id "Crazyflie-contol-board-rescue:BATTERY-Crazyflie-contol-board-rescue") (at 213.36 146.05 0) (unit 1)
-    (in_bom yes) (on_board yes) (dnp no)
-    (property "Reference" "BT1" (at 213.36 140.97 0)
-      (effects (font (size 1.27 1.27)))
-    )
-    (property "Value" "BATTERY" (at 213.36 146.05 0)
-      (effects (font (size 1.524 1.524)) hide)
-    )
-    (property "Footprint" "Connector_PinHeader_2.54mm:PinHeader_1x02_P2.54mm_Vertical" (at 213.36 146.05 0)
-      (effects (font (size 1.524 1.524)) hide)
-    )
-    (property "Datasheet" "" (at 213.36 146.05 0)
-      (effects (font (size 1.27 1.27)) hide)
-    )
-    (property "Field4" "JST" (at 213.36 146.05 0)
-      (effects (font (size 1.524 1.524)) hide)
-    )
-    (property "Field5" "B2B-ZR" (at 213.36 146.05 0)
-      (effects (font (size 1.524 1.524)) hide)
-    )
-    (pin "1")
-    (pin "2")
-    (instances
-      (project "Crazyflie contol board"
-        (path "/3e9fa01f-48e9-4c58-997e-0bab5b5694a8/00000000-0000-0000-0000-00004de77332"
-          (reference "BT1") (unit 1)
         )
       )
@@
         )
       )
-    )
-  )
-  (symbol (lib_id "Crazyflie-contol-board-rescue:DGND-Crazyflie-contol-board-rescue") (at 265.43 158.75 0) (unit 1)
-    (in_bom yes) (on_board yes) (dnp no)
-    (property "Reference" "#PWR059" (at 265.43 158.75 0)
-      (effects (font (size 1.016 1.016)) hide)
-    )
-    (property "Value" "DGND" (at 265.43 160.528 0)
-      (effects (font (size 1.016 1.016)))
-    )
-    (property "Footprint" "" (at 265.43 158.75 0)
-      (effects (font (size 1.27 1.27)) hide)
-    )
-    (property "Datasheet" "" (at 265.43 158.75 0)
-      (effects (font (size 1.27 1.27)) hide)
-    )
-    (pin "1")
-    (instances
-      (project "Crazyflie contol board"
-        (path "/3e9fa01f-48e9-4c58-997e-0bab5b5694a8/00000000-0000-0000-0000-00004de77332"
-          (reference "#PWR059") (unit 1)
-        )
-      )
-    )
-  )
-  (symbol (lib_id "Crazyflie-contol-board-rescue:PWR_FLAG-power") (at 265.43 153.67 0) (unit 1)
-    (in_bom yes) (on_board yes) (dnp no)
-    (property "Reference" "#FLG058" (at 265.43 146.812 0)
-      (effects (font (size 0.762 0.762)) hide)
-    )
-    (property "Value" "PWR_FLAG" (at 265.43 147.828 0)
-      (effects (font (size 0.762 0.762)))
-    )
-    (property "Footprint" "" (at 265.43 153.67 0)
-      (effects (font (size 1.27 1.27)) hide)
-    )
-    (property "Datasheet" "" (at 265.43 153.67 0)
-      (effects (font (size 1.27 1.27)) hide)
-    )
-    (pin "1")
-    (instances
-      (project "Crazyflie contol board"
-        (path "/3e9fa01f-48e9-4c58-997e-0bab5b5694a8/00000000-0000-0000-0000-00004de77332"
-          (reference "#FLG058") (unit 1)
-        )
-      )

Commit message: save
Parts:
- removed P7: MICRO-B-USB, ZX62-B-5PA_11_CFK, symbol Crazyflie-contol-board-rescue:MICRO-B-USB-Crazyflie-contol-board-rescue
- added J3: USB_C_Receptacle_USB2.0, Connector_USB:USB_C_Receptacle_HRO_TYPE-C-31-M-12, symbol Connector:USB_C_Receptacle_USB2.0
- added R6, R7: 5k1, Resistor_SMD:R_0603_1608Metric, symbol Device:R
Connections:
- net +BATT: now also J3.A4 (VBUS), J3.A9 (VBUS), J3.B4 (VBUS), J3.B9 (VBUS)
- net D+: now also J3.A6 (D+), J3.B6 (D+)
- net D-: now also J3.A7 (D-), J3.B7 (D-)
- net GND: now also J3.A1 (GND), J3.A12 (GND), J3.B1 (GND), J3.B12 (GND), J3.S1 (SHIELD), R6.2, R7.2
- new net: J3.A5 (CC1), R6.1
- new net: J3.B5 (CC2), R7.1
- no-connect marks 1 -> 0
Other:
- moved on the sheet: C34, C36, C37, P9, R17, U6

Commit message: save
Parts:
- removed R6, R7: 5k1, Resistor_SMD:R_0603_1608Metric, symbol Device:R
- added C6: 470pF, Capacitor_SMD:C_0603_1608Metric, symbol Device:C
Connections:
- net GND: now also C6.2
- net at U9.4 (NR): now also C6.1
Changed lines of the file:
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@@
-	)
-	(junction
-		(at 64.77 118.11)
-		(diameter 0)
-		(color 0 0 0 0)
 	)
 	(junction
@@
 		(color 0 0 0 0)
 	)
-	(junction
-		(at 64.77 77.47)
-		(diameter 0)
-		(color 0 0 0 0)
-	)
 	(polyline
 		(pts
@@
 	(wire
 		(pts
+			(xy 210.82 116.84) (xy 223.52 116.84)
+		)
+		(stroke
+			(width 0)
+			(type default)
+		)
+	)
+	(wire
+		(pts
 			(xy 172.72 99.06) (xy 172.72 118.11)
 		)
@@
 	(wire
 		(pts
-			(xy 64.77 118.11) (xy 86.36 118.11)
-		)
-		(stroke
-			(width 0)
-			(type default)
-		)
-	)
-	(wire
-		(pts
 			(xy 59.69 40.64) (xy 59.69 85.09)
 		)
@@
 	(wire
 		(pts
-			(xy 64.77 77.47) (xy 64.77 118.11)
-		)
-		(stroke
-			(width 0)
-			(type default)
-		)
-	)
-	(wire
-		(pts
 			(xy 62.23 87.63) (xy 62.23 38.1)
 		)
@@
 	(wire
 		(pts
+			(xy 210.82 109.22) (xy 210.82 116.84)
+		)
+		(stroke
+			(width 0)
+			(type default)
+		)
+	)
+	(wire
+		(pts
 			(xy 265.43 134.62) (xy 265.43 138.43)
 		)
@@
 	(wire
 		(pts
-			(xy 64.77 74.93) (xy 64.77 77.47)
-		)
-		(stroke
-			(width 0)
-			(type default)
-		)
-	)
-	(wire
-		(pts
-			(xy 54.61 74.93) (xy 57.15 74.93)
-		)
-		(stroke
-			(width 0)
-			(type default)
-		)
-	)
-	(wire
-		(pts
 			(xy 227.33 123.19) (xy 223.52 123.19)
 		)
@@
 	(wire
 		(pts
+			(xy 208.28 101.6) (xy 210.82 101.6)
+		)
+		(stroke
+			(width 0)
+			(type default)
+		)
+	)
+	(wire
+		(pts
 			(xy 165.1 118.11) (xy 165.1 120.65)
 		)
@@
 	(wire
 		(pts
-			(xy 39.37 118.11) (xy 64.77 118.11)
-		)
-		(stroke
-			(width 0)
-			(type default)
-		)
-	)
-	(wire
-		(pts
-			(xy 54.61 77.47) (xy 57.15 77.47)
+			(xy 39.37 118.11) (xy 86.36 118.11)
 		)
 		(stroke
@@
 				(path "/3e9fa01f-48e9-4c58-997e-0bab5b5694a8/00000000-0000-0000-0000-00004de77332"
 					(reference "#PWR0114")
-					(unit 1)
-				)
-			)
-		)
-	)
-	(symbol
-		(lib_id "Device:R")
-		(at 60.96 74.93 90)
-		(unit 1)
-		(exclude_from_sim no)
-		(in_bom yes)
-		(on_board yes)
-		(dnp no)
-		(property "Reference" "R6"
-			(at 60.96 72.39 90)
-			(effects
-				(font
-					(size 1.27 1.27)
-				)
-			)
-		)
-		(property "Value" "5k1"
-			(at 60.96 74.93 90)
-			(effects
-				(font
-					(size 1.27 1.27)
-				)
-			)
-		)
-		(property "Footprint" "Resistor_SMD:R_0603_1608Metric"
-			(at 60.96 76.708 90)
-			(effects
-				(font
-					(size 1.27 1.27)
-				)
-				(hide yes)
-			)
-		)
-		(property "Datasheet" "~"
-			(at 60.96 74.93 0)
-			(effects
-				(font
-					(size 1.27 1.27)
-				)
-				(hide yes)
-			)
-		)
-		(property "Description" ""
-			(at 60.96 74.93 0)
-			(effects
-				(font
-					(size 1.27 1.27)
-				)
-				(hide yes)
-			)
-		)
-		(pin "1"
-		)
-		(pin "2"
-		)
-		(instances
-			(project "Crazyflie contol board"
-				(path "/3e9fa01f-48e9-4c58-997e-0bab5b5694a8/00000000-0000-0000-0000-00004de77332"
-					(reference "R6")
-					(unit 1)
-				)
-			)
-		)
-	)
-	(symbol
-		(lib_id "Device:R")
-		(at 60.96 77.47 90)
-		(unit 1)
-		(exclude_from_sim no)
-		(in_bom yes)
-		(on_board yes)
-		(dnp no)
-		(property "Reference" "R7"
-			(at 60.96 80.01 90)
-			(effects
-				(font
-					(size 1.27 1.27)
-				)
-			)
-		)
-		(property "Value" "5k1"
-			(at 60.96 77.47 90)
-			(effects
-				(font
-					(size 1.27 1.27)
-				)
-			)
-		)
-		(property "Footprint" "Resistor_SMD:R_0603_1608Metric"
-			(at 60.96 79.248 90)
-			(effects
-				(font
-					(size 1.27 1.27)
-				)
-				(hide yes)
-			)
-		)
-		(property "Datasheet" "~"
-			(at 60.96 77.47 0)
-			(effects
-				(font
-					(size 1.27 1.27)
-				)
-				(hide yes)
-			)
-		)
-		(property "Description" ""
-			(at 60.96 77.47 0)
-			(effects
-				(font
-					(size 1.27 1.27)
-				)
-				(hide yes)
-			)
-		)
-		(pin "1"
-		)
-		(pin "2"
-		)
-		(instances
-			(project "Crazyflie contol board"
-				(path "/3e9fa01f-48e9-4c58-997e-0bab5b5694a8/00000000-0000-0000-0000-00004de77332"
-					(reference "R7")
 					(unit 1)
 				)
@@
 					(unit 1)
 				)
+			)
+		)
+	)
+	(symbol
+		(lib_id "Device:C")
+		(at 210.82 105.41 0)
+		(unit 1)
+		(exclude_from_sim no)
+		(in_bom yes)
+		(on_board yes)
+		(dnp no)
+		(fields_autoplaced yes)
+		(property "Reference" "C6"
+			(at 214.63 104.1399 0)
+			(effects
+				(font
+					(size 1.27 1.27)
+				)
+				(justify left)
+			)
+		)
+		(property "Value" "470pF"
+			(at 214.63 106.6799 0)
+			(effects
+				(font
+					(size 1.27 1.27)
+				)
+				(justify left)
+			)
+		)
+		(property "Footprint" "Capacitor_SMD:C_0603_1608Metric"
+			(at 211.7852 109.22 0)
+			(effects
+				(font
+					(size 1.27 1.27)
+				)
+				(hide yes)
+			)
+		)
+		(property "Datasheet" "~"
+			(at 210.82 105.41 0)
+			(effects
+				(font
+					(size 1.27 1.27)
+				)
+				(hide yes)
+			)
+		)
+		(property "Description" "Unpolarized capacitor"
+			(at 210.82 105.41 0)
+			(effects
+				(font
+					(size 1.27 1.27)
+				)
+				(hide yes)
+			)
+		)
+		(pin "2"
+		)
+		(pin "1"
+		)
+		(instances
+			(project ""
+				(path "/3e9fa01f-48e9-4c58-997e-0bab5b5694a8/00000000-0000-0000-0000-00004de77332"
+					(reference "C6")
+					(unit 1)
+				)

Commit message: save
Parts:
- removed C34, C37: 2.2uF, Capacitor_SMD:C_0603_1608Metric, symbol Crazyflie-contol-board-rescue:C-Crazyflie-contol-board-rescue
- removed C36: 100nF, Capacitor_SMD:C_0603_1608Metric, symbol Crazyflie-contol-board-rescue:C-Crazyflie-contol-board-rescue
- removed C6: 470pF, Capacitor_SMD:C_0603_1608Metric, symbol Device:C
- removed J3: USB_C_Receptacle_USB2.0, Connector_USB:USB_C_Receptacle_HRO_TYPE-C-31-M-12, symbol Connector:USB_C_Receptacle_USB2.0
- removed R17: 100k, Resistor_SMD:R_0603_1608Metric, symbol Crazyflie-contol-board-rescue:R-Crazyflie-contol-board-rescue
- removed U6: NUF2221, SOT363, symbol Crazyflie-contol-board-rescue:NUF2221-Crazyflie-contol-board-rescue
- removed U9: TPS79301, SOT23_6, symbol Crazyflie-contol-board-rescue:TPS79301-Crazyflie-contol-board-rescue
Other:
- moved on the sheet: D7, P9, R22
