File: Drone/IMU.kicad_sch (KiCad schematic)
At the start: 5 parts, among them U1 BMX160, U5 MS5611-01BA03

Commit message: save
Parts:
- C18, C20, C24: footprint ESP32-footprints-Lib:0603_new_new -> ESP32-footprints-Lib:0603
Connections:
- net AGND renamed GND

Commit message: save
Parts:
- C18, C20, C24: footprint ESP32-footprints-Lib:0603 -> Capacitor_SMD:C_0603_1608Metric
Changed lines of the file:
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@@
   (junction (at 134.62 135.89) (diameter 0) (color 0 0 0 0)
+  )
+  (junction (at 124.46 73.66) (diameter 0) (color 0 0 0 0)
   )
   (junction (at 137.16 73.66) (diameter 0) (color 0 0 0 0)
@@
     (stroke (width 0) (type default))
   )
+  (wire (pts (xy 124.46 123.19) (xy 124.46 73.66))
+    (stroke (width 0) (type default))
+  )
   (wire (pts (xy 139.7 107.95) (xy 137.16 107.95))
     (stroke (width 0) (type default))
   )
-  (wire (pts (xy 128.27 123.19) (xy 134.62 123.19))
+  (wire (pts (xy 124.46 123.19) (xy 134.62 123.19))
     (stroke (width 0) (type default))
   )
@@
       (effects (font (size 1.27 1.27)) (justify left))
     )
-    (property "Footprint" "ESP32-footprints-Lib:0603" (at 137.16 82.55 0)
+    (property "Footprint" "Capacitor_SMD:C_0603_1608Metric" (at 137.16 82.55 0)
       (effects (font (size 1.524 1.524)) hide)
     )
@@
       (effects (font (size 1.27 1.27)) (justify left))
     )
-    (property "Footprint" "ESP32-footprints-Lib:0603" (at 128.27 82.55 0)
+    (property "Footprint" "Capacitor_SMD:C_0603_1608Metric" (at 128.27 82.55 0)
       (effects (font (size 1.524 1.524)) hide)
     )
@@
       (effects (font (size 1.27 1.27)) (justify left))
     )
-    (property "Footprint" "ESP32-footprints-Lib:0603" (at 134.62 130.81 0)
+    (property "Footprint" "Capacitor_SMD:C_0603_1608Metric" (at 134.62 130.81 0)
       (effects (font (size 1.524 1.524)) hide)
     )
@@
         )
       )
-    )
-  )
-  (symbol (lib_id "Crazyflie-contol-board-rescue:VCCA-Crazyflie-contol-board-rescue") (at 128.27 123.19 90) (unit 1)
-    (in_bom yes) (on_board yes) (dnp no)
-    (property "Reference" "#PWR031" (at 125.73 123.19 0)
-      (effects (font (size 0.762 0.762)) hide)
-    )
-    (property "Value" "VCC" (at 125.73 123.19 0)
-      (effects (font (size 0.762 0.762)))
-    )
-    (property "Footprint" "" (at 128.27 123.19 0)
-      (effects (font (size 1.27 1.27)) hide)
-    )
-    (property "Datasheet" "" (at 128.27 123.19 0)
-      (effects (font (size 1.27 1.27)) hide)
-    )
-    (pin "1")
-    (instances
-      (project "Crazyflie contol board"
-        (path "/3e9fa01f-48e9-4c58-997e-0bab5b5694a8/00000000-0000-0000-0000-00004de1273c"
-          (reference "#PWR031") (unit 1)
-        )
-      )

Commit message: save
Parts:
- removed U5: MS5611-01BA03, MS5611, symbol Crazyflie-contol-board-rescue:MS5611-01BA01-Crazyflie-contol-board-rescue
- added C3: 100nF, Capacitor_SMD:C_0603_1608Metric, symbol Crazyflie-contol-board-rescue:C-Crazyflie-contol-board-rescue
- added U2: BMP388, Package_LGA:ST_HLGA-10_2x2mm_P0.5mm_LayoutBorder3x2y, symbol Sensor_Pressure:BMP280
Connections:
- net GND: now also C3.2, U2.3 (GND), U2.5 (SDO), U2.8 (GND), U2.9 (GND)
- net I2C_SCL_VCCA: now also U2.2 (SCK)
- net I2C_SDA_VCCA: now also U2.4 (SDI)
- net VCCA: now also C3.1, U2.1 (VDDIO), U2.10 (VDD), U2.6 (CSB)
- net INT2: now reaches U1.9 (INT2)
- net INT_GA renamed INT1
- new net INT3: U2.7 (INT)
- no-connect marks 1 -> 0
Other:
- moved on the sheet: C24

Commit message: save
Parts:
- removed U1: BMX160, digikey-footprints:LGA-14L_2.5x3mm__LSM6DS3, symbol Crazyflie-contol-board-rescue:BMX160-SensorMotion
- added C4: 1uF, Capacitor_SMD:C_0603_1608Metric, symbol Device:C
- added R8: 10k, Resistor_SMD:R_0603_1608Metric, symbol Device:R
- added U3: BNO055, Package_LGA:LGA-28_5.2x3.8mm_P0.5mm, symbol Sensor_Motion:BNO055
- C18: value 100nF -> 120nF
Connections:
- net GND: now also C4.2, U3.17 (COM3), U3.18 (COM2), U3.2 (GND), U3.25 (GNDIO), U3.5 (PS1)
- net I2C_SCL_VCCA: now also U3.19 (COM1)
- net I2C_SDA_VCCA: now also U3.20 (COM0)
- net INT1: now also U3.14 (INT)
- net VCCA: now also R8.1, U3.28 (VDDIO), U3.3 (VDD), U3.6 (PS0)
- new net: C4.1, U3.9 (CAP)
- new net: R8.2, U3.4 (~{BOOT_LOAD_PIN})

Commit message: save
Changed lines of the file:
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@@
-	(wire
-		(pts
-			(xy 172.72 45.72) (xy 186.69 45.72)
-		)
-		(stroke
-			(width 0)
-			(type default)
-		)
-	)
 	(wire
 		(pts
@@
 		)
 	)
-	(global_label "INT2"
-		(shape input)
-		(at 179.07 45.72 90)
-		(fields_autoplaced yes)
-		(effects
-			(font
-				(size 1.27 1.27)
-			)
-			(justify left)
-		)
-		(property "Intersheetrefs" "${INTERSHEET_REFS}"
-			(at 179.07 39.356 90)
-			(effects
-				(font
-					(size 1.27 1.27)
-				)
-				(justify left)
-				(hide yes)
-			)
-		)
-	)
 	(hierarchical_label "I2C_SCL_VCCA"
 		(shape input)
@@
 		)
 	)
-	(hierarchical_label "INT2"
-		(shape output)
-		(at 186.69 45.72 0)
-		(effects
-			(font
-				(size 1.524 1.524)
-			)
-			(justify left)
-		)
-	)

Commit message: save
Parts:
- removed C3: 100nF, Capacitor_SMD:C_0603_1608Metric, symbol Crazyflie-contol-board-rescue:C-Crazyflie-contol-board-rescue
- removed R8: 10k, Resistor_SMD:R_0603_1608Metric, symbol Device:R
- C18: value 120nF -> 10uF
- C4: value 1uF -> 100nF
Connections:
- net GND: now also U3.6 (PS0)
- net VCCA: now also U3.4 (~{BOOT_LOAD_PIN}); no longer U3.6 (PS0)

Commit message: save
Connections:
- net INT3 renamed INT2
Changed lines of the file:
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@@
 		)
 	)
-	(global_label "INT3"
+	(global_label "INT2"
 		(shape input)
 		(at 147.32 107.95 90)
@@
 		)
 		(property "Intersheetrefs" "${INTERSHEET_REFS}"
-			(at 147.32 101.586 90)
+			(at 147.32 101.5066 90)
 			(effects
 				(font
