File: ESC/BLDC_4.kicad_pcb (KiCad board)
At the start: 4 copper layers, 39 x 59 mm, 70 parts, among them J1 Conn_02x09_Odd_Even, P1 IN+, P2 IN-, P3 MOTOR3, P4 MOTOR2, P5 MOTOR1, Q1 IRFS7530, Q2 IRFS7530, Q3 IRFS7530, Q4 IRFS7530, Q5 IRFS7530, Q6 IRFS7530, U1 DRV8302

Commit message: save
Parts:
- J1: value Conn_02x09_Odd_Even -> Motor; footprint Connector_Harwin:Harwin_M20-7810945_2x09_P2.54mm_Vertical -> Connector_PinHeader_2.54mm:PinHeader_2x09_P2.54mm_Vertical
- moved D3 13.0 mm to (113.6, 125.5), turned to -90 degrees
- moved J1 9.31 mm to (113.6, 132.9), turned to -90 degrees
Connections:
- J1 pad 1: +5V -> /Mosfet driver/BR_SO1
- J1 pad 2: GND -> /Mosfet driver/BR_SO2
- J1 pad 3: VCC -> +5V
- J1 pad 5: /Mosfet driver/DC_CAL -> VCC
- J1 pad 6: /Mosfet driver/EN_GATE -> GND
- J1 pad 7: /Mosfet driver/BR_SO2 -> EN
- J1 pad 9: /Mosfet driver/BR_SO1 -> DC
- U1 pad 12: /Mosfet driver/DC_CAL -> DC
- U1 pad 16: /Mosfet driver/EN_GATE -> EN
Routing:
- net VCC: track 23.1 -> 29.5 mm
- net /Mosfet driver/SENS1: track 3.06 -> 8.41 mm
Other:
- board size 39 x 59 mm -> 38.5 x 59 mm
- board text added: "5V"
- board text added: "H1 L1"
- board text added: "H2 L2"
- board text added: "H3 L3"
- board text removed: "H1"
- board text removed: "H2"
- board text removed: "H3"

Commit message: update
Connections:
- J1 pad 1: /Mosfet driver/BR_SO1 -> /Mosfet driver/BR_SO2
- J1 pad 10: /Mosfet driver/L1 -> /Mosfet driver/H3
- J1 pad 12: /Mosfet driver/H2 -> /Mosfet driver/L2
- J1 pad 14: /Mosfet driver/L2 -> /Mosfet driver/H2
- J1 pad 16: /Mosfet driver/H3 -> /Mosfet driver/L1
- J1 pad 18: /Mosfet driver/L3 -> /Mosfet driver/H1
- J1 pad 2: /Mosfet driver/BR_SO2 -> /Mosfet driver/BR_SO1
- J1 pad 8: /Mosfet driver/H1 -> /Mosfet driver/L3
Routing:
- net +5V: track 17.6 -> 97.4 mm
- net /Mosfet driver/L1: track 0.00 -> 22.1 mm, vias 0 -> 2
- net /Mosfet driver/H1: track 0.00 -> 21.4 mm
- net /Mosfet driver/L2: track 0.00 -> 20.3 mm, vias 0 -> 2
- net /Mosfet driver/L3: track 0.00 -> 19.9 mm, vias 0 -> 2
- net /Mosfet driver/FAULT: track 0.00 -> 19.7 mm, vias 0 -> 1
- net EN: track 0.00 -> 18.9 mm, vias 0 -> 1
- net /Mosfet driver/BR_SO1: track 0.00 -> 18.4 mm
- net DC: track 0.00 -> 18.3 mm, vias 0 -> 1
- net /Mosfet driver/H2: track 0.00 -> 18.1 mm
- net /Mosfet driver/H3: track 0.00 -> 16.4 mm
- net /Mosfet driver/BR_SO2: track 0.00 -> 15.6 mm
- net /Mosfet driver/SENS2: track 3.15 -> 15.8 mm
- net /Mosfet driver/SENS3: track 3.09 -> 14.6 mm
- net GND: track 189.9 -> 188.1 mm
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