File: ESC/BLDC_4.kicad_pcb (KiCad board)
At the start: 4 copper layers, 38.5 x 59 mm, 70 parts, among them J1 Motor, P1 IN+, P2 IN-, P3 MOTOR3, P4 MOTOR2, P5 MOTOR1, Q1 IRFS7530, Q2 IRFS7530, Q3 IRFS7530, Q4 IRFS7530, Q5 IRFS7530, Q6 IRFS7530, U1 DRV8302

Commit message: save
Parts:
- removed J1: Motor, Connector_PinHeader_2.54mm:PinHeader_2x09_P2.54mm_Vertical
- added C26: C, CRF1:SMD-0603_c, F.Cu at (80.5, 136.3)
- added C27: C, CRF1:SMD-0603_c, F.Cu at (87.5, 134.9)
- added P6: USB_C_Plug_USB2.0, Connector_USB:USB_C_Receptacle_HRO_TYPE-C-31-M-12, B.Cu at (82.6, 146.4)
- added U2: ESP32-S3-WROOM-2, RF_Module:ESP32-S3-WROOM-2, F.Cu at (105.3, 149.0)
- added U3: TPS62177DQC, Package_SON:WSON-10-1EP_2x3mm_P0.5mm_EP0.84x2.4mm_ThermalVias, F.Cu at (84.0, 137.6)
Connections:
- net /Mosfet driver/SENS1 renamed S1
- net /Mosfet driver/SENS2 renamed S2
- net /Mosfet driver/SENS3 renamed S3
- U1 pad 17: /Mosfet driver/H1 -> H1
- U1 pad 18: /Mosfet driver/L1 -> L1
- U1 pad 19: /Mosfet driver/H2 -> H2
- U1 pad 20: /Mosfet driver/L2 -> L2
- U1 pad 21: /Mosfet driver/H3 -> H3
- U1 pad 22: /Mosfet driver/L3 -> L3
- U1 pad 25: /Mosfet driver/BR_SO1 -> B1
- U1 pad 26: /Mosfet driver/BR_SO2 -> B2
- U1 pad 6: /Mosfet driver/FAULT -> F
Routing:
- net +5V: track 97.4 -> 43.5 mm
- net V_SUPPLY: track 266.4 -> 317.6 mm
- net L1: track 0.00 -> 33.7 mm, vias 0 -> 2
- net H1: track 0.00 -> 33.4 mm
- net L3: track 0.00 -> 33.2 mm, vias 0 -> 2
- net Net-(P6-D+): track 0.00 -> 32.9 mm, vias 0 -> 1
- net B2: track 0.00 -> 32.4 mm
- net F: track 0.00 -> 32.4 mm, vias 0 -> 1
- net L2: track 0.00 -> 31.3 mm, vias 0 -> 2
- net Net-(P6-D-): track 0.00 -> 30.3 mm, vias 0 -> 1
- net B1: track 0.00 -> 29.4 mm
- net H2: track 0.00 -> 29.2 mm
- net H3: track 0.00 -> 28.4 mm
- net S1: track 8.41 -> 30.8 mm
- net /Mosfet driver/L1: track 22.1 -> 0.00 mm, vias 2 -> 0
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Other:
- board size 38.5 x 59 mm -> 38.5 x 75 mm
