File: ESC/Power.kicad_sch (KiCad schematic)
At the start: 45 parts, among them U1 DRV8302

Commit message: update
Other:
- title: BLDC Driver 4.11 -> BLDC Driver 4.12
Changed lines of the file:
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@@
   (paper "A4")
   (title_block
-    (title "BLDC Driver 4.11")
-    (date "21 aug 2015")
-    (rev "4.12")
+    (title "BLDC Driver 4.12")
+    (date "2022-08-07")
+    (rev "A")
     (company "Benjamin Vedder")
   )
