File: ESC/BLDC_4.kicad_sch (KiCad schematic)
At the start: 10 parts, among them J1 Conn_02x09_Odd_Even, P1 IN+, P2 IN-, P3 MOTOR3, P4 MOTOR2, P5 MOTOR1

Commit message: save
Parts:
- J1: value Conn_02x09_Odd_Even -> Motor; footprint Connector_Harwin:Harwin_M20-7810945_2x09_P2.54mm_Vertical -> Connector_PinHeader_2.54mm:PinHeader_2x09_P2.54mm_Vertical
Connections:
- net Mosfet driver/DC_CAL is gone; now on net VCC: J1.5 (Pin_5)
- net Mosfet driver/EN_GATE is gone; now on net GND: J1.6 (Pin_6)
- net +5V: now also J1.3 (Pin_3); no longer J1.1 (Pin_1)
- net GND: no longer J1.2 (Pin_2)
- net Mosfet driver/BR_SO1: now also J1.1 (Pin_1); no longer J1.9 (Pin_9)
- net Mosfet driver/BR_SO2: now also J1.2 (Pin_2); no longer J1.7 (Pin_7)
- net VCC: no longer J1.3 (Pin_3)
- new net DC: J1.9 (Pin_9)
- new net EN: J1.7 (Pin_7)

Commit message: update
Connections:
- net Mosfet driver/BR_SO1: now also J1.2 (Pin_2); no longer J1.1 (Pin_1)
- net Mosfet driver/BR_SO2: now also J1.1 (Pin_1); no longer J1.2 (Pin_2)
- net Mosfet driver/H1: now also J1.18 (Pin_18); no longer J1.8 (Pin_8)
- net Mosfet driver/H2: now also J1.14 (Pin_14); no longer J1.12 (Pin_12)
- net Mosfet driver/H3: now also J1.10 (Pin_10); no longer J1.16 (Pin_16)
- net Mosfet driver/L1: now also J1.16 (Pin_16); no longer J1.10 (Pin_10)
- net Mosfet driver/L2: now also J1.12 (Pin_12); no longer J1.14 (Pin_14)
- net Mosfet driver/L3: now also J1.8 (Pin_8); no longer J1.18 (Pin_18)
Other:
- title: BLDC Driver 4.11 -> BLDC Driver 4.12
Changed lines of the file:
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@@
   (paper "A4")
   (title_block
-    (title "BLDC Driver 4.11")
-    (date "21 aug 2015")
-    (rev "4.12")
+    (title "BLDC Driver 4.12")
+    (date "2022-08-07")
+    (rev "A")
     (company "Benjamin Vedder")
     (comment 4 "Top level")
@@
       (effects (font (size 1.524 1.524)) (justify left))
     )
-    (pin "H1" input (at 157.48 67.31 180)
+    (pin "L3" input (at 157.48 67.31 180)
       (effects (font (size 1.524 1.524)) (justify left))
     )
-    (pin "L1" input (at 157.48 69.85 180)
+    (pin "H3" input (at 157.48 69.85 180)
       (effects (font (size 1.524 1.524)) (justify left))
     )
-    (pin "H2" input (at 157.48 72.39 180)
+    (pin "L2" input (at 157.48 72.39 180)
       (effects (font (size 1.524 1.524)) (justify left))
     )
-    (pin "L2" input (at 157.48 74.93 180)
+    (pin "H2" input (at 157.48 74.93 180)
       (effects (font (size 1.524 1.524)) (justify left))
     )
-    (pin "H3" input (at 157.48 77.47 180)
+    (pin "L1" input (at 157.48 77.47 180)
       (effects (font (size 1.524 1.524)) (justify left))
     )
-    (pin "L3" input (at 157.48 80.01 180)
+    (pin "H1" input (at 157.48 80.01 180)
       (effects (font (size 1.524 1.524)) (justify left))
     )
-    (pin "BR_SO1" output (at 157.48 107.95 180)
+    (pin "BR_SO2" output (at 157.48 107.95 180)
       (effects (font (size 1.524 1.524)) (justify left))
     )
-    (pin "BR_SO2" output (at 157.48 110.49 180)
+    (pin "BR_SO1" output (at 157.48 110.49 180)
       (effects (font (size 1.524 1.524)) (justify left))
     )

Commit message: save
Parts:
- added C26: 2.2uF, CRF1:SMD-0603_c, symbol Device:C
- added C27: 22uF, CRF1:SMD-0603_c, symbol Device:C
- added L2: 10uH, symbol Device:L
- added P6: USB_C_Plug_USB2.0, Connector_USB:USB_C_Receptacle_HRO_TYPE-C-31-M-12, symbol Connector:USB_C_Plug_USB2.0
- added U2: ESP32-S3-WROOM-2, RF_Module:ESP32-S3-WROOM-2, symbol RF_Module:ESP32-S3-WROOM-2
- added U3: TPS62177DQC, Package_SON:WSON-10-1EP_2x3mm_P0.5mm_EP0.84x2.4mm_ThermalVias, symbol Regulator_Switching:TPS62177DQC
Connections:
- net +5V: now also C27.1, L2.2, U3.10 (VOS), U3.8 (~{SLEEP})
- net EN: now also U2.7 (IO7)
- net GND: now also C26.2, C27.2, P6.A1 (GND), P6.A12 (GND), P6.A5 (CC), P6.B1 (GND), P6.B12 (GND), P6.B5 (VCONN), P6.S1 (SHIELD), U3.1 (PGND), U3.11 (PAD), U3.5 (FB), U3.6 (AGND)
- net V_SUPPLY: now also C26.1, P6.A4 (VBUS), P6.A9 (VBUS), P6.B4 (VBUS), P6.B9 (VBUS), U3.2 (VIN), U3.3 (EN)
- net Mosfet driver/BR_SO1 renamed B1
- net Mosfet driver/BR_SO2 renamed B2
- net Mosfet driver/FAULT renamed F
- net F: now also U2.12 (IO8)
- net Mosfet driver/H1 renamed H1
- net H1: now also U2.34 (MTDI/IO41)
- net Mosfet driver/H2 renamed H2
- net H2: now also U2.32 (MTCK/IO39)
- net Mosfet driver/H3 renamed H3
- net Mosfet driver/L1 renamed L1
- net L1: now also U2.33 (MTDO/IO40)
- net Mosfet driver/L2 renamed L2
- net L2: now also U2.31 (IO38)
- net Mosfet driver/L3 renamed L3
- net Mosfet driver/SENS1 renamed S1
- net Mosfet driver/SENS2 renamed S2
- net Mosfet driver/SENS3 renamed S3
- new net: L2.1, U3.9 (SW)
- new net: P6.A6 (D+), U2.14 (USB_D+/IO20)
- new net: P6.A7 (D-), U2.13 (USB_D-/IO19)
- new net: U2.1 (GND), U2.40 (GND), U2.41 (GND)
Other:
- moved on the sheet: D1, R1
