File: miniKame/minikame.kicad_pcb (KiCad board)
At the start: 2 copper layers, 48.8 x 40.1 mm, 16 parts, among them J1 PWM, J10 C, J11 A, J12 D, J13 B, J2 Camera, J3 ESP32, J4 ESP32, J5 GND, J6 Vcc, J7 UART, J8 I2C, J9 Motor

Commit message: save
Parts:
- removed Battery: 1210, digikey-footprints:1210
- removed J1: PWM, ESP32-footprints-Lib:PIN8
- removed J2: Camera, Connector_PinSocket_2.54mm:PinSocket_2x09_P2.54mm_Vertical
- removed J5: GND, ESP32-footprints-Lib:PIN8
- removed J6: Vcc, ESP32-footprints-Lib:PIN8
- removed J7: UART, ESP32-footprints-Lib:PIN4
- removed J8: I2C, ESP32-footprints-Lib:PIN4
- removed R1, R2: 4k7, Resistor_SMD:R_0603_1608Metric
- added BT1: Battery_Cell, digikey-footprints:1210, F.Cu at (136.9, 79.7)
- added C1: C, digikey-footprints:0603, F.Cu at (134.4, 88.9)
- added C2: C, digikey-footprints:0603, F.Cu at (142.5, 89.8)
- added P1: USB_C_Plug_USB2.0, Connector_USB:USB_C_Receptacle_HRO_TYPE-C-31-M-12, F.Cu at (124.7, 86.7)
- added U1: ESP32-S3-WROOM-2, RF_Module:ESP32-S3-WROOM-2, F.Cu at (161.0, 109.2)
- added U2: TPS62177DQC, Package_SON:WSON-10-1EP_2x3mm_P0.5mm_EP0.84x2.4mm_ThermalVias, F.Cu at (138.2, 90.3)
Routing:
- net G13: track 9.03 -> 53.2 mm
- net H: track 69.9 -> 31.9 mm
- net V: track 69.7 -> 32.7 mm, vias 1 -> 0
- net G23: track 48.0 -> 13.9 mm
- net 3.3v: track 70.5 -> 100.1 mm
- net G19: track 43.8 -> 14.5 mm
- net G18: track 30.8 -> 1.52 mm
- net X: track 49.9 -> 25.8 mm
- net G27: track 15.9 -> 38.2 mm
- net SDA: track 72.4 -> 51.5 mm, vias 1 -> 0
- net P: track 41.9 -> 22.9 mm
- net SCL: track 81.1 -> 64.4 mm, vias 1 -> 0
- net Tx: track 32.9 -> 16.5 mm, vias 1 -> 0
- net D5: track 35.0 -> 19.3 mm
- net D6: track 21.8 -> 6.03 mm
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