File: miniKame/minikame.kicad_sch (KiCad schematic)
At the start: 16 parts, among them J1 PWM, J10 C, J11 A, J12 D, J13 B, J2 Camera, J3 ESP32, J4 ESP32, J5 GND, J6 Vcc, J7 UART, J8 I2C, J9 Motor

Commit message: save
Parts:
- removed J1: PWM, symbol Connector:Conn_01x08_Male
- removed J2: Camera, Connector_PinSocket_2.54mm:PinSocket_2x09_P2.54mm_Vertical, symbol Header:HDMI
- removed J5: GND, symbol Connector:Conn_01x08_Male
- removed J6: Vcc, symbol Connector:Conn_01x08_Male
- removed J7: UART, symbol Connector:Conn_01x04_Male
- removed J8: I2C, symbol Connector:Conn_01x04_Male
- removed R1, R2: 4k7, Resistor_SMD:R_0603_1608Metric, symbol Device:R
- added C1: 2.2uF, digikey-footprints:0603, symbol Device:C
- added C2: 22uF, digikey-footprints:0603, symbol Device:C
- added L1: 10uH, symbol Device:L
- added P1: USB_C_Plug_USB2.0, Connector_USB:USB_C_Receptacle_HRO_TYPE-C-31-M-12, symbol Connector:USB_C_Plug_USB2.0
- added U1: ESP32-S3-WROOM-2, RF_Module:ESP32-S3-WROOM-2, symbol RF_Module:ESP32-S3-WROOM-2
- added U2: TPS62177DQC, Package_SON:WSON-10-1EP_2x3mm_P0.5mm_EP0.84x2.4mm_ThermalVias, symbol Regulator_Switching:TPS62177DQC
- J10: footprint (none) -> digikey-footprints:0603
Connections:
- net 3.3v: now also C2.1, L1.2, U1.2 (3V3), U2.10 (VOS), U2.8 (~{SLEEP})
- net 5V: now also C1.1, P1.A4 (VBUS), P1.A9 (VBUS), P1.B4 (VBUS), P1.B9 (VBUS), U2.2 (VIN), U2.3 (EN)
- net G13: now also U1.7 (IO7)
- net G23: now also U1.12 (IO8)
- net G27: now also U1.6 (IO6)
- net GND: now also C1.2, C2.2, P1.A1 (GND), P1.A12 (GND), P1.A5 (CC), P1.B1 (GND), P1.B12 (GND), P1.B5 (VCONN), P1.S1 (SHIELD), U1.1 (GND), U1.40 (GND), U1.41 (GND), U2.1 (PGND), U2.11 (PAD), U2.5 (FB), U2.6 (AGND)
- new net: P1.A6 (D+), U1.14 (USB_D+/IO20)
- new net: P1.A7 (D-), U1.13 (USB_D-/IO19)
- new net: L1.1, U2.9 (SW)
