File: motordriver/klepcontroller.kicad_pcb (KiCad board)
At the start: 2 copper layers, 61 x 47 mm, 23 parts, among them J4 Motor, J5 Motor, J6 Power, P1 USB_C_Plug_USB2.0, U1 TMC2660, U2 ESP32-S3-WROOM-2, U3 TPS62177DQC

Commit message: save
Parts:
- removed C12: 10uF, digikey-footprints:0603
- removed C16, C3: 100nF, digikey-footprints:0603
- removed C17, C8: 10nF, digikey-footprints:0603
- removed the C4 at (151.6, 103.0)
- removed R5, R6: 100m, digikey-footprints:0603
- added C26: 100n, Capacitor_SMD:C_0402_1005Metric, F.Cu at (135.5, 91.5)
- added C4: 22uF, Capacitor_SMD:C_0402_1005Metric, F.Cu at (131.3, 87.8)
- added C4: 22u, Capacitor_SMD:C_0603_1608Metric, F.Cu at (154.5, 116.5)
- added C5: 100n, Capacitor_SMD:C_0402_1005Metric, F.Cu at (127.1, 89.5)
- added C9: 22n, Capacitor_SMD:C_0402_1005Metric, F.Cu at (130.8, 96.7)
- added D1: SS14, Diode_SMD:D_SMA, F.Cu at (155.6, 106.4)
- added J3: SPI, Connector_PinHeader_2.54mm:PinHeader_1x05_P2.54mm_Vertical, F.Cu at (167.3, 94.9)
- added L1: 10uH, tetra:IND-SMD_L3.9-W3.9-1, F.Cu at (149.7, 115.1)
- added R14: 1K, Resistor_SMD:R_0402_1005Metric, F.Cu at (135.0, 83.7)
- added R15: 10K, Resistor_SMD:R_0402_1005Metric, F.Cu at (129.7, 86.6)
- added R16: 1K, Resistor_SMD:R_0402_1005Metric, F.Cu at (135.5, 90.4)
- added R9: 5k1, Resistor_SMD:R_0402_1005Metric, F.Cu at (157.9, 98.2)
- added TP1: +3V3, TestPoint:TestPoint_Pad_2.0x2.0mm, F.Cu at (144.0, 116.8)
- added TP2: GND, TestPoint:TestPoint_Pad_2.0x2.0mm, F.Cu at (134.2, 102.0)
- added TP3: +24V, TestPoint:TestPoint_Pad_2.0x2.0mm, F.Cu at (161.5, 116.9)
- added TP5: Vref, TestPoint:TestPoint_Pad_2.0x2.0mm, F.Cu at (137.9, 102.0)
- added U4: SOT-363_SC-70-6, Package_TO_SOT_SMD:SOT-363_SC-70-6, F.Cu at (156.6, 99.5)
- C1: value 470nF -> 2.2uF; footprint digikey-footprints:0603 -> Capacitor_SMD:C_0402_1005Metric
- C19, C20: value 10uF -> 47uF; footprint Capacitors_SMD:CP_Elec_6.3x5.8 -> Capacitor_SMD:CP_Elec_6.3x5.8
- C2: value C -> 2.2uF; footprint digikey-footprints:0603 -> Capacitor_SMD:C_1206_3216Metric
- C6: footprint digikey-footprints:0603 -> Capacitor_SMD:C_0402_1005Metric
- C7: value 10uF -> 100nF; footprint digikey-footprints:0603 -> Capacitor_SMD:C_0402_1005Metric
- R7: value 10R -> 10k; footprint digikey-footprints:0603 -> Resistor_SMD:R_0402_1005Metric
- R8: value 10R -> 5k1; footprint digikey-footprints:0603 -> Resistor_SMD:R_0402_1005Metric
- U1: value TMC2660 -> TMC2209-LA; footprint Housings_QFP:PQFP-44_10x10mm_Pitch0.8mm -> Package_DFN_QFN:VQFN-28-1EP_5x5mm_P0.5mm_EP3.7x3.7mm_ThermalVias
- moved R8 36.8 mm to (157.1, 104.0)
- moved C20 21.3 mm to (122.7, 99.2)
- moved R7 14.5 mm to (127.9, 87.1), turned to -90 degrees
- moved C6 11.3 mm to (131.8, 98.1)
- moved C19 9.99 mm to (122.8, 89.3), turned to 90 degrees
- moved U3 7.23 mm to (154.8, 112.9), turned to 180 degrees
- moved C7 6.93 mm to (127.1, 95.8), turned to 90 degrees
- moved C2 6.61 mm to (158.4, 114.4), turned to -90 degrees
- moved U1 6.45 mm to (130.8, 92.6), turned to 90 degrees
- moved C1 4.80 mm to (135.2, 94.6), turned to 0 degrees
Connections:
- C1 pad 1: GND -> 5V
- C1 pad 2: 5V -> GND
- C2 pad 1: GND -> +24V
- C2 pad 2: +24V -> GND
- C6 pad 1: +24V -> Net-(U1-VCP)
- C6 pad 2: Net-(U1-VHS) -> +24V
- P1 pad A4: +24V -> +5V
- P1 pad A5: GND -> Net-(P1-CC)
- P1 pad A9: +24V -> +5V
- P1 pad B4: +24V -> +5V
- P1 pad B5: GND -> Net-(P1-VCONN)
- P1 pad B6: (no net) -> Net-(P1-D+)
- P1 pad B7: (no net) -> Net-(P1-D-)
- P1 pad B9: +24V -> +5V
- R7 pad 1: Net-(U1-BRA) -> +3V3
- R7 pad 2: Net-(U1-SRA) -> ENABLE
- R8 pad 1: Net-(U1-BRB) -> GND
- R8 pad 2: Net-(U1-SRB) -> Net-(P1-CC)
- U1 pad 1: (no net) -> B2
- U1 pad 10: A2 -> GND
- U1 pad 11: A2 -> unconnected-(U1-DIAG-Pad11)
- U1 pad 12: Net-(U1-SRA) -> unconnected-(U1-INDEX-Pad12)
- U1 pad 13: 5V -> unconnected-(U1-CLK-Pad13)
- U1 pad 14: SDO -> /pusher/M_UART
- U1 pad 15: SDI -> +3V3
- U1 pad 16: SCK -> STEP
- U1 pad 17: GND -> /pusher/Vref
- U1 pad 18: CS -> GND
- U1 pad 19: ENABLE -> DIRECTION
- U1 pad 2: A1 -> ENABLE
- U1 pad 20: (no net) -> ENABLE
- U1 pad 21: unconnected-(U1-CLK-Pad21) -> A2
- U1 pad 22: Net-(U1-SRB) -> +24V
- U1 pad 23: B2 -> GND
- U1 pad 24: B2 -> A1
- U1 pad 25: Net-(U1-BRB) -> GND
- U1 pad 27: B1 -> GND
- U1 pad 28: B2 -> +24V
- U1 pad 29: B2 -> GND
- U1 pad 3: A1 -> GND
- U1 pad 4: +24V -> Net-(U1-CPO)
- U1 pad 5: A2 -> Net-(U1-CPI)
- U1 pad 6: A2 -> Net-(U1-VCP)
- U1 pad 7: A1 -> unconnected-(U1-SPREAD-Pad7)
- U1 pad 8: A1 -> 5V
- U1 pad 9: Net-(U1-BRA) -> GND
- U2 pad 1: Net-(U2-GND-Pad1) -> GND
- U2 pad 10: unconnected-(U2-IO17-Pad10) -> /pusher/M_UART
- U2 pad 11: unconnected-(U2-IO18-Pad11) -> SDO
- U2 pad 12: unconnected-(U2-IO8-Pad12) -> STEP
- U2 pad 2: unconnected-(U2-3V3-Pad2) -> +3V3
- U2 pad 27: unconnected-(U2-IO0-Pad27) -> GPIO0
- U2 pad 3: unconnected-(U2-EN-Pad3) -> Net-(U2-EN)
- U2 pad 31: unconnected-(U2-IO38-Pad31) -> DIRECTION
- U2 pad 32: SCK -> unconnected-(U2-MTCK/IO39-Pad32)
- U2 pad 33: SDO -> ENABLE
- U2 pad 34: SDI -> unconnected-(U2-MTDI/IO41-Pad34)
- U2 pad 35: CS -> unconnected-(U2-MTMS/IO42-Pad35)
- U2 pad 36: unconnected-(U2-RXD0/IO44-Pad36) -> Rx
- U2 pad 37: unconnected-(U2-TXD0/IO43-Pad37) -> Tx
- U2 pad 40: Net-(U2-GND-Pad1) -> GND
- U2 pad 41: Net-(U2-GND-Pad1) -> GND
- U2 pad 9: unconnected-(U2-IO16-Pad9) -> /pusher/M_PWM
- U3 pad 10: 5V -> +3V3
- U3 pad 8: 5V -> +3V3
Routing:
- net +3V3: track 12.2 -> 101.0 mm, vias 0 -> 4
- net ENABLE: track 27.9 -> 79.2 mm, vias 1 -> 2
- net CS: track 48.6 -> 0.00 mm, vias 1 -> 0
- net SDI: track 45.1 -> 0.00 mm, vias 1 -> 0
- net SCK: track 42.4 -> 0.00 mm, vias 1 -> 0
- net 5V: track 40.5 -> 1.66 mm, vias 1 -> 0
- net A1: track 80.0 -> 43.5 mm, vias 0 -> 2
- net DIRECTION: track 9.67 -> 45.1 mm, vias 0 -> 4
- net SDO: track 41.1 -> 14.0 mm, vias 1 -> 2
- net GND: track 5.51 -> 32.0 mm, vias 18 -> 64
- net /pusher/M_UART: track 0.00 -> 26.5 mm, vias 0 -> 2
- net A2: track 71.0 -> 49.9 mm, vias 1 -> 2
- net /pusher/Vref: track 0.00 -> 21.0 mm, vias 0 -> 2
- net Tx: track 0.00 -> 20.6 mm
- net Rx: track 0.00 -> 20.4 mm
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- added copper zone on B.Cu, net +24V
- added copper zone on F.Cu, net +24V
- added copper zone on F.Cu, net +3V3
- added copper zone on In1.Cu, net GND
- added copper zone on In2.Cu, net GND
Other:
- copper layers 2 -> 4
- board text removed: "3.3V"
- board text removed: "CS"
- board text removed: "DI"
- board text removed: "EN"
- board text removed: "SPI"
- board text removed: "STEP"
