File: motordriver/klepcontroller.kicad_sch (KiCad schematic)
At the start: 27 parts, among them J1 Motor, J2 GPIOs, J3 SPI, J4 Motor, J5 Motor, J6 Power, P1 USB_C_Plug_USB2.0, U1 TMC2660, U2 ESP32-S3-WROOM-2, U3 TPS62177DQC

Commit message: save
Parts:
- removed C17: 10nF, digikey-footprints:0603, symbol klepcontroller-rescue:C-device
- removed R5, R6: 100m, digikey-footprints:0603, symbol klepcontroller-rescue:R-device
- removed U1: TMC2660, Housings_QFP:PQFP-44_10x10mm_Pitch0.8mm, symbol klepcontroller-rescue:TMC2660-DriverMotor
- added D1: SS14, symbol Device:D
- added R1: 10k, symbol Device:R
- added R9: 5k1, digikey-footprints:0603, symbol klepcontroller-rescue:R-Device
- added U1: TMC2209-LA, Package_DFN_QFN:VQFN-28-1EP_5x5mm_P0.5mm_EP3.7x3.7mm_ThermalVias, symbol Driver_Motor:TMC2209-LA
- C1: value 470nF -> 2.2uF
- C12, C7: value 10uF -> 100nF
- C19, C20: value 10uF -> 47uF
- C8: value 10nF -> 22nF
- R7: value 10R -> 10k
- R8: value 10R -> 5k1
Connections:
- net +24V: now also C2.1, C6.2, D1.1 (K), U1.22 (VS), U1.28 (VS); no longer C2.2, C6.1, P1.A4 (VBUS), P1.A9 (VBUS), P1.B4 (VBUS), P1.B9 (VBUS)
- net +3V3: now also C4.1, J3.1, L1.2, R7.1, U2.2 (3V3), U3.10 (VOS), U3.8 (~{SLEEP}), R1.1, U1.15 (VCC_IO)
- net 5V: now also C1.1, U1.8 (5VOUT); no longer C1.2, C4.1, J3.2, L1.2, U3.10 (VOS), U3.8 (~{SLEEP})
- net A1: now also U1.24 (OA1)
- net A2: now also U1.21 (OA2)
- net B1: now also U1.26 (OB1)
- net B2: now also U1.1 (OB2)
- net CS: no longer U2.35 (MTMS/IO42)
- net DIRECTION: now also U2.31 (IO38), U1.19 (DIR)
- net ENABLE: now also R7.2, U2.33 (MTDO/IO40), U1.2 (~{EN}), U1.20 (STDBY)
- net GND: now also C1.2, C2.2, J3.5, R8.1, U2.1 (GND), U2.40 (GND), U2.41 (GND), R9.1, U1.10 (MS2/AD1), U1.18 (GND), U1.23 (BRA), U1.25 (NC), U1.27 (BRB), U1.29 (GND), U1.3 (GND), U1.9 (MS1/AD0); no longer C1.1, C2.1, C8.1, P1.A5 (CC), P1.B5 (VCONN)
- net SCK: now also U2.10 (IO17); no longer J3.3, U2.32 (MTCK/IO39)
- net SDO: now also U2.11 (IO18); no longer J3.1, U2.33 (MTDO/IO40)
- net STEP: now also U2.12 (IO8), U1.16 (STEP)
- net at C8.2: now also U1.4 (CPO); no longer R7.2
- net at R8.2: now also P1.A5 (CC)
- net GPIO0: now reaches U2.27 (IO0)
- net GPIO0: now also J3.4
- net at U2.3 (EN): now also R1.2
- net Rx: now reaches U2.36 (RXD0/IO44)
- net Rx: now also J3.3
- net Tx: now reaches U2.37 (TXD0/IO43)
- net Tx: now also J3.2
- net SDI: no longer names the net of U2.34 (MTDI/IO41)
- net SDI: no longer J3.4
- new net: C8.1, U1.5 (CPI)
- new net: C6.1, U1.6 (VCP)
- new net: P1.B5 (VCONN), R9.2
- new net +5V: D1.2 (A), P1.A4 (VBUS), P1.A9 (VBUS), P1.B4 (VBUS), P1.B9 (VBUS)
Other:
- moved on the sheet: C1, C2, C6, C8, R7
